File: IOT-Mess-BoardESP/IOT-Mess-BoardB/IOT-Mess-BoardB.kicad_pcb (KiCad board)
At the start: 2 copper layers, 30.4 x 65 mm, 33 parts, among them J1 Conn_01x05_Pin, J3 Conn_01x05_Pin, J5 Conn_01x24_Pin, J6 USB_C_Receptacle_USB2.0_16P, SW1 RotaryEncoder, SW10 SW_Push, SW11 SW_Push, U1 ESP-12F, U3 ESP32-S3-WROOM-1, U4 ME6211C33M5, U5 ESP32-C3-WROOM-02

Commit message: did some works.
Parts:
- moved D2 47.8 mm to (131.1, 116.5)
- moved R8 47.8 mm to (131.1, 116.5)
Changed lines of the file:
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@@
 	(footprint "Resistor_SMD:R_0603_1608Metric"
 		(layer "F.Cu")
-		(at 87.106996 97.707721 90)
+		(at 131.08 116.505 90)
 		(descr "Resistor SMD 0603 (1608 Metric), square (rectangular) end terminal, IPC-7351 nominal, (Body size source: IPC-SM-782 page 72, https://www.pcb-3d.com/wordpress/wp-content/uploads/ipc-sm-782a_amendment_1_and_2.pdf), generated with kicad-footprint-generator")
 		(tags "resistor")
@@
 	(footprint "LED_SMD:LED_0603_1608Metric"
 		(layer "B.Cu")
-		(at 87.106996 97.707721 -90)
+		(at 131.08 116.505 -90)
 		(descr "LED SMD 0603 (1608 Metric), square (rectangular) end terminal, IPC-7351 nominal, (Body size source: http://www.tortai-tech.com/upload/download/2011102023233369053.pdf), generated with kicad-footprint-generator")
 		(tags "LED")
@@
 		(layer "Edge.Cuts")
 	)
+	(dimension
+		(type orthogonal)
+		(layer "User.1")
+		(pts
+			(xy 93.306996 57.307721) (xy 93.306997 122.30772)
+		)
+		(height -7.976996)
+		(orientation 1)
+		(format
+			(prefix "")
+			(suffix "")
+			(units 3)
+			(units_format 0)
+			(precision 4)
+			(suppress_zeroes yes)
+		)
+		(style
+			(thickness 0.1)
+			(arrow_length 1.27)
+			(text_position_mode 0)
+			(arrow_direction outward)
+			(extension_height 0.58642)
+			(extension_offset 0.5)
+			(keep_text_aligned yes)
+		)
+		(gr_text "65"
+			(at 84.18 89.807721 90)
+			(layer "User.1")
+			(effects
+				(font
+					(size 1 1)
+					(thickness 0.15)
+				)
+			)
+		)
+	)
+	(dimension
+		(type orthogonal)
+		(layer "User.1")
+		(pts
+			(xy 93.306997 122.30772) (xy 123.706995 122.30772)
+		)
+		(height 8.23228)
+		(orientation 0)
+		(format
+			(prefix "")
+			(suffix "")
+			(units 3)
+			(units_format 0)
+			(precision 4)
+			(suppress_zeroes yes)
+		)
+		(style
+			(thickness 0.1)
+			(arrow_length 1.27)
+			(text_position_mode 0)
+			(arrow_direction outward)
+			(extension_height 0.58642)
+			(extension_offset 0.5)
+			(keep_text_aligned yes)
+		)
+		(gr_text "30.4"
+			(at 108.506996 129.39 0)
+			(layer "User.1")
+			(effects
+				(font
+					(size 1 1)
+					(thickness 0.15)
+				)
+			)
+		)
+	)
 	(segment
