File: IOT-Mess-CH_P20/IOT-Mess-P20.kicad_pcb (KiCad board)
At the start: 2 copper layers, 21.4 x 49.5 mm, 31 parts, among them J10 Jumper_2, J11 Jumper_2, J16 Jumper, J3 Jumper_2, J4 Jumper_2, J5 Conn_01x15_Pin, J6 Conn_01x15_Pin, J7 Jumper, J8 Jumper_2, J9 Jumper, K1 Crystal, SW11 SW_Push, U10 USB_C_Receptacle_USB2.0_16P, U6 ME6211C33M5

Commit message: did some works.
Other:
- board text added: "IOT_Mess CH_P20 V1.0"
- board text removed: "CH32V_Mess P20 V1.0"
Changed lines of the file:
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@@
 		)
 	)
-	(gr_text "CH32V_Mess\nP20 V1.0\n"
+	(gr_text "IOT_Mess\nCH_P20 V1.0\n"
 		(at 112.875 75.125 0)
 		(layer "B.SilkS")

Commit message: did some works.
Connections:
- C4 pad 1: +3.3V -> Net-(J3-A)
- J3 pad 1: +3.3V -> Net-(J3-A)
- J3 pad 2: VCC -> +3.3V
- J5 pad 1: ANT -> P_1
- J5 pad 10: P_9 -> P_10
- J5 pad 11: P_10 -> 5V
- J5 pad 14: VCC -> +3.3V
- J5 pad 2: P_1 -> P_2
- J5 pad 3: P_2 -> P_3
- J5 pad 4: P_3 -> P_4
- J5 pad 5: P_4 -> P_5
- J5 pad 6: P_5 -> P_6
- J5 pad 7: P_6 -> P_7
- J5 pad 8: P_7 -> P_8
- J5 pad 9: P_8 -> P_9
- J7 pad 2: VCC -> +3.3V
- R5 pad 1: VCC -> +3.3V
- U6 pad 5: +3.3V -> Net-(J3-A)
- U8 pad 2: P_13 -> P_12
- U8 pad 3: P_14 -> P_13
- U8 pad 4: P_15 -> P_14
- U8 pad 5: P_18 -> P_16
- U8 pad 6: P_19 -> P_17
- U8 pad 7: P_20 -> P_18
Routing:
- net VCC: track 24.5 -> 0.00 mm, vias 1 -> 0
- net +3.3V: track 12.3 -> 26.1 mm
- net Net-(J3-A): track 0.00 -> 12.3 mm, vias 0 -> 1
- net 5V: track 13.9 -> 24.2 mm
- net ANT: track 6.63 -> 1.69 mm
- net P_8: track 26.1 -> 22.7 mm
- net P_7: track 30.1 -> 27.1 mm
- net P_16: track 32.0 -> 34.7 mm
- net P_17: track 29.1 -> 31.8 mm
- net P_10: track 31.0 -> 28.5 mm
- net P_18: track 27.0 -> 28.7 mm
- net P_3: track 25.7 -> 24.0 mm
- net P_14: track 23.0 -> 24.4 mm
- net P_2: track 26.4 -> 25.0 mm
- net P_19: track 29.4 -> 30.6 mm
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
Commit message: did some works.
Parts:
- removed the G*** at (113.3, 67.9)
- added G***: LOGO, IOT-Mess-Footprints:catIcon8x8, B.Cu at (112.5, 76.0)
Connections:
- J3 pad 2: +3.3V -> 5V
- J5 pad 14: +3.3V -> 5V
- J7 pad 2: +3.3V -> 5V
- R5 pad 1: +3.3V -> 5V
Routing:
- net 5V: track 24.2 -> 53.1 mm, vias 1 -> 2
- net +3.3V: track 26.1 -> 0.00 mm, vias 1 -> 0
- net P_15: track 24.2 -> 23.7 mm
- net P_0: vias 4 -> 0
Other:
- board text added: "1"
- board text added: "10"
- board text added: "11"
- board text added: "12"
- board text added: "13"
- board text added: "14"
- board text added: "15"
- board text added: "16"
- board text added: "17"
- board text added: "18"
- board text added: "19"
- board text added: "2"
- board text added: "20"
- board text added: "3"
- board text added: "4"
- board text added: "5"
- board text added: "5V"
- board text added: "6"
- board text added: "7"
- board text added: "8"
- board text added: "9"
- board text added: "G"
- board text added: "IOT_Mess CH_P20 V1.0 7/5/25"
- board text added: "X0"
- board text removed: "GND"
- board text removed: "IOT_Mess CH_P20 V1.0"
- board text removed: "P1"
- board text removed: "P10"
- board text removed: "P11"
- board text removed: "P12"
- board text removed: "P13"
- board text removed: "P14"
- board text removed: "P15"
- board text removed: "P16"
- board text removed: "P17"
- board text removed: "P18"
- board text removed: "P19"
- board text removed: "P2"
- board text removed: "P20"
- board text removed: "P3"
- board text removed: "P4"
- board text removed: "P5"
- board text removed: "P6"
- board text removed: "P7"
- board text removed: "P8"
- board text removed: "P9"
- board text removed: "VCC"
- board text removed: "X"
- board text removed: "XO"
