File: IOT-Mess-CH_P20/IOT-Mess-P20.kicad_sch (KiCad schematic)
At the start: 33 parts, among them J10 Jumper_2, J11 Jumper_2, J16 Jumper, J3 Jumper_2, J4 Jumper_2, J5 Conn_01x15_Pin, J6 Conn_01x15_Pin, J7 Jumper, J8 Jumper_2, J9 Jumper, K1 Crystal, SW11 SW_Push, U10 USB_C_Receptacle_USB2.0_16P, U6 ME6211C33M5

Commit message: did some works.
Parts:
- removed TP1, TP2: TestPoint, symbol Connector:TestPoint
Connections:
- net VCC is gone; now on net +3.3V: J3.2 (B), J5.14 (Pin_14), J7.2 (C), R5.1
- net +3.3V: no longer C4.1, J3.1 (A), U6.5 (V_{OUT})
- net 5V: now also J5.11 (Pin_11)
- net ANT: no longer J5.1 (Pin_1)
- net P_1: now also J5.1 (Pin_1); no longer J5.2 (Pin_2)
- net P_10: now also J5.10 (Pin_10); no longer J5.11 (Pin_11)
- net P_12: now also U8.2 (PC2/SCL)
- net P_13: now also U8.3 (PC3); no longer U8.2 (PC2/SCL)
- net P_14: now also U8.4 (PC4/A2); no longer U8.3 (PC3)
- net P_15: no longer U8.4 (PC4/A2)
- net P_16: now also U8.5 (PC6/MOSI)
- net P_17: now also U8.6 (PC7/MISO)
- net P_18: now also U8.7 (PD1/SWIO); no longer U8.5 (PC6/MOSI)
- net P_19: no longer U8.6 (PC7/MISO)
- net P_2: now also J5.2 (Pin_2); no longer J5.3 (Pin_3)
- net P_20: no longer U8.7 (PD1/SWIO)
- net P_3: now also J5.3 (Pin_3); no longer J5.4 (Pin_4)
- net P_4: now also J5.4 (Pin_4); no longer J5.5 (Pin_5)
- net P_5: now also J5.5 (Pin_5); no longer J5.6 (Pin_6)
- net P_6: now also J5.6 (Pin_6); no longer J5.7 (Pin_7)
- net P_7: now also J5.7 (Pin_7); no longer J5.8 (Pin_8)
- net P_8: now also J5.8 (Pin_8); no longer J5.9 (Pin_9)
- net P_9: now also J5.9 (Pin_9); no longer J5.10 (Pin_10)
- new net: C4.1, J3.1 (A), U6.5 (V_{OUT})
Other:
- moved on the sheet: D1, J6, R5

Commit message: did some works.
Parts:
- removed TP3: TestPoint, symbol Connector:TestPoint
Connections:
- net 5V is gone; now on net +3.3V: C2.1, C5.1, D2.1 (K), J4.2 (B), J5.11 (Pin_11), U6.1 (V_{IN}), U6.3 (CE)
- net GND: now also U3.21 (GND); no longer U3.0 (GND)
Other:
- moved on the sheet: AE1
Changed lines of the file:
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@@
 	)
 	(junction
+		(at 185.42 205.74)
+		(diameter 0)
+		(color 0 0 0 0)
+	)
+	(junction
 		(at 81.28 49.53)
 		(diameter 0)
@@
 	(wire
 		(pts
-			(xy 137.16 43.18) (xy 137.16 46.99)
-		)
-		(stroke
-			(width 0)
-			(type default)
-		)
-	)
-	(wire
-		(pts
 			(xy 214.63 114.3) (xy 220.98 114.3)
 		)
@@
 	(wire
 		(pts
+			(xy 185.42 205.74) (xy 185.42 215.9)
+		)
+		(stroke
+			(width 0)
+			(type default)
+		)
+	)
+	(wire
+		(pts
 			(xy 326.39 114.3) (xy 332.74 114.3)
 		)
@@
 	(wire
 		(pts
-			(xy 185.42 210.82) (xy 185.42 215.9)
+			(xy 185.42 201.93) (xy 185.42 205.74)
 		)
 		(stroke
@@
 	(wire
 		(pts
-			(xy 128.27 46.99) (xy 128.27 43.18)
+			(xy 137.16 46.99) (xy 137.16 41.91)
 		)
 		(stroke
@@
 	(wire
 		(pts
-			(xy 128.27 46.99) (xy 137.16 46.99)
+			(xy 165.1 119.38) (xy 158.75 119.38)
 		)
 		(stroke
@@
 	(wire
 		(pts
-			(xy 165.1 119.38) (xy 158.75 119.38)
+			(xy 78.74 127) (xy 78.74 120.65)
 		)
 		(stroke
@@
 	(wire
 		(pts
-			(xy 78.74 127) (xy 78.74 120.65)
+			(xy 158.75 124.46) (xy 165.1 124.46)
 		)
 		(stroke
@@
 	(wire
 		(pts
-			(xy 158.75 124.46) (xy 165.1 124.46)
+			(xy 191.77 205.74) (xy 185.42 205.74)
 		)
 		(stroke
@@
 		)
 	)
+	(global_label "5V"
+		(shape input)
+		(at 191.77 205.74 0)
+		(fields_autoplaced yes)
+		(effects
+			(font
+				(size 1.27 1.27)
+				(color 255 0 0 1)
+			)
+			(justify left)
+		)
+		(property "Intersheetrefs" "${INTERSHEET_REFS}"
+			(at 197.0533 205.74 0)
+			(effects
+				(font
+					(size 1.27 1.27)
+				)
+				(justify left)
+				(hide yes)
+			)
+		)
+	)
 	(global_label "P_4"
 		(shape input)
@@
 	(symbol
 		(lib_id "Device:Antenna")
-		(at 128.27 38.1 0)
+		(at 137.16 36.83 0)
 		(unit 1)
 		(exclude_from_sim no)
@@
 		(dnp no)
 		(property "Reference" "AE1"
-			(at 122.174 36.068 0)
+			(at 131.064 34.798 0)
 			(effects
 				(font
@@
 		)
 		(property "Value" "Antenna"
-			(at 119.38 38.354 0)
+			(at 128.27 37.084 0)
 			(effects
 				(font
@@
 		)
 		(property "Footprint" "RF_Antenna:Texas_SWRA117D_2.4GHz_Right"
-			(at 128.27 38.1 0)
+			(at 137.16 36.83 0)
 			(effects
 				(font
@@
 		)
 		(property "Datasheet" "~"
-			(at 128.27 38.1 0)
+			(at 137.16 36.83 0)
 			(effects
 				(font
@@
 		)
 		(property "Description" "Antenna"
-			(at 128.27 38.1 0)
+			(at 137.16 36.83 0)
 			(effects
 				(font
@@
 			)
 		)
-		(property "Description" ""
+		(property "Description" "Power symbol creates a global label with name \"GND\" , ground"
 			(at 215.9 223.52 0)
 			(effects
@@
 	)
 	(symbol
-		(lib_id "Connector:TestPoint")
-		(at 137.16 43.18 0)
-		(mirror y)
-		(unit 1)
-		(exclude_from_sim no)
-		(in_bom yes)
-		(on_board yes)
-		(dnp no)
-		(property "Reference" "TP3"
-			(at 141.732 39.878 0)
-			(effects
-				(font
-					(size 1.27 1.27)
-				)
-				(justify left)
-			)
-		)
-		(property "Value" "TestPoint"
-			(at 144.272 37.338 0)
-			(effects
-				(font
-					(size 1.27 1.27)
-				)
-				(justify left)
-			)
-		)
-		(property "Footprint" ""
-			(at 132.08 43.18 0)
-			(effects
-				(font
-					(size 1.27 1.27)
-				)
-				(hide yes)
-			)
-		)
-		(property "Datasheet" "~"
-			(at 132.08 43.18 0)
-			(effects
-				(font
-					(size 1.27 1.27)
-				)
-				(hide yes)
-			)
-		)
-		(property "Description" "test point"
-			(at 137.16 43.18 0)
-			(effects
-				(font
-					(size 1.27 1.27)
-				)
-				(hide yes)
-			)
-		)
-		(pin "1"
-		)
-		(instances
-			(project "IOT-Mess-P20"
-				(path "/ab2cc265-7ef1-48af-b7c5-4cd6db1bae75"
-					(reference "TP3")
-					(unit 1)
-				)
-			)
-		)
-	)
-	(symbol
 		(lib_id "Connector:Conn_01x15_Pin")
 		(at 360.68 213.36 0)
@@
 			)
 		)
-		(property "Description" ""
+		(property "Description" "Light emitting diode"
+			(at 207.01 215.9 0)
+			(effects
+				(font
+					(size 1.27 1.27)
+				)
+				(hide yes)
+			)
+		)
+		(property "Sim.Pins" "1=K 2=A"
 			(at 207.01 215.9 0)
 			(effects
@@
 	(symbol
 		(lib_id "power:+3.3V")
-		(at 185.42 210.82 0)
+		(at 185.42 201.93 0)
 		(unit 1)
 		(exclude_from_sim no)
@@
 		(fields_autoplaced yes)
 		(property "Reference" "#PWR01"
-			(at 185.42 214.63 0)
+			(at 185.42 205.74 0)
 			(effects
 				(font
@@
 		)
 		(property "Value" "+3.3V"
-			(at 185.42 205.74 0)
+			(at 185.42 196.85 0)
 			(effects
 				(font
@@
 		)
 		(property "Footprint" ""
-			(at 185.42 210.82 0)
+			(at 185.42 201.93 0)
 			(effects
 				(font
@@
 		)
 		(property "Datasheet" ""
-			(at 185.42 210.82 0)
+			(at 185.42 201.93 0)
 			(effects
 				(font
@@
 		)
 		(property "Description" "Power symbol creates a global label with name \"+3.3V\""
-			(at 185.42 210.82 0)
+			(at 185.42 201.93 0)
 			(effects
 				(font
@@
 		(pin "20"
 		)
-		(pin "0"
+		(pin "21"
 		)
 		(pin "2"
