File: IOT-Mess-CH_P48/IOT-Mess-P48.kicad_pcb (KiCad board)
At the start: 2 copper layers, 29.1 x 49.8 mm, 28 parts, among them J1 Conn_02x19_Odd_Even, J10 Jumper, J11 Jumper, J12 Jumper, J14 Jumper, J2 Conn_02x19_Odd_Even, J3 Jumper_2, J6 Jumper, J7 Jumper, J8 Jumper, K1 Crystal, K32 Crystal, SW11 SW_Push, U10 USB_C_Receptacle_USB2.0_16P, U3 CH32L103C8T6, U6 ME6211C33M5

Commit message: did some works.
Routing:
- added copper zone on B.Cu, net GND
- added copper zone on F.Cu, net GND
Changed lines of the file:
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@@
 		)
 		(property "Datasheet" ""
-			(at 0 0 -90)
+			(at 0 0 270)
 			(unlocked yes)
 			(layer "B.Fab")
@@
 		)
 		(property "Description" "Solder Jumper, 3-pole, open"
-			(at 0 0 -90)
+			(at 0 0 270)
 			(unlocked yes)
 			(layer "B.Fab")
@@
 		)
 		(property "Datasheet" ""
-			(at 0 0 -90)
+			(at 0 0 270)
 			(unlocked yes)
 			(layer "B.Fab")
@@
 		)
 		(property "Description" "Solder Jumper, 3-pole, open"
-			(at 0 0 -90)
+			(at 0 0 270)
 			(unlocked yes)
 			(layer "B.Fab")
@@
 		)
 		(property "Datasheet" ""
-			(at 0 0 -90)
+			(at 0 0 270)
 			(unlocked yes)
 			(layer "B.Fab")
@@
 		)
 		(property "Description" "Solder Jumper, 3-pole, open"
-			(at 0 0 -90)
+			(at 0 0 270)
 			(unlocked yes)
 			(layer "B.Fab")
@@
 		(net 61)
 	)
+	(zone
+		(net 2)
+		(net_name "GND")
+		(layers "F.Cu" "B.Cu")
+		(hatch edge 0.5)
+		(connect_pads
+			(clearance 0.5)
+		)
+		(min_thickness 0.25)
+		(filled_areas_thickness no)
+		(fill yes
+			(thermal_gap 0.5)
+			(thermal_bridge_width 0.5)
+		)
+		(polygon
+			(pts
+				(xy 189.55 73.29) (xy 218.58 73.3) (xy 218.59 123.07) (xy 189.55 123.05)
+			)
+		)
+	)
 	(embedded_fonts no)

Commit message: did some works.
Parts:
- removed D3: SS14, Diode_SMD:D_SMA
- removed J8: Jumper, IOT-Mess-Footprints:Jumper-3_P1.3mm_Open_RoundedPad1.0x1.5mm
- added D2: 1N5819WS, Diode_SMD:D_SOD-323, F.Cu at (196.6, 111.2)
- added J4: Jumper_2, IOT-Mess-Footprints:Jumpper-triangle, F.Cu at (196.7, 113.7)
- J12: moved to F.Cu
- moved J11 7.86 mm to (204.4, 105.1)
- moved J7 7.80 mm to (194.1, 101.6), turned to -135 degrees
- moved J6 7.71 mm to (213.4, 100.2), turned to 135 degrees
- moved J3 4.85 mm to (210.0, 112.7)
- moved J14 4.64 mm to (204.4, 107.8), turned to 180 degrees
- moved J12 0.95 mm to (197.9, 108.2)
- moved C8 0.29 mm to (201.4, 75.2)
- moved C9 0.29 mm to (198.2, 75.2)
- moved K32 0.29 mm to (200.3, 78.4)
Routing:
- net VCC: track 0.00 -> 36.6 mm, vias 0 -> 4
- net P_3: track 22.4 -> 53.7 mm
- net Net-(J10-C): track 2.85 -> 25.8 mm, vias 0 -> 2
- net P_35: track 20.0 -> 41.0 mm
- net P_33: track 20.1 -> 36.2 mm, vias 1 -> 2
- net P_7: track 29.2 -> 42.3 mm
- net P_48: track 21.5 -> 33.8 mm, vias 1 -> 2
- net Net-(D3-A): track 8.07 -> 0.00 mm, vias 1 -> 0
- net P_36: track 20.2 -> 28.0 mm
- net P_8: track 23.6 -> 31.0 mm, vias 1 -> 2
- net P_47: track 24.6 -> 31.2 mm
- net Net-(D2-A): track 9.21 -> 15.7 mm, vias 0 -> 2
- net P_23: track 39.5 -> 44.4 mm, vias 1 -> 2
- net +3.3V: track 2.47 -> 7.25 mm
- net P_18: track 52.9 -> 57.6 mm
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Other:
- board size 29.1 x 49.8 mm -> 30.1 x 49.8 mm

Commit message: did some works.
Parts:
- added J5: Conn_01x05_Pin, Connector_PinHeader_2.54mm:PinHeader_1x05_P2.54mm_Vertical, F.Cu at (193.9, 110.9)
- moved D2 1.01 mm to (197.7, 111.1)
- moved J4 1.01 mm to (197.7, 113.7)
- moved C2 0.15 mm to (202.4, 112.6)
- moved C4 0.15 mm to (206.5, 109.7)
- moved C5 0.15 mm to (205.7, 112.6)
- moved U6 0.15 mm to (203.0, 109.5)
Connections:
- J14 pad 2: VCC -> +3.3V
- J3 pad 1: +3.3V -> Net-(J3-A)
- J3 pad 2: VCC -> +3.3V
- J6 pad 2: VCC -> +3.3V
- J7 pad 2: VCC -> +3.3V
- U6 pad 5: +3.3V -> Net-(J3-A)
Routing:
- net +3.3V: track 7.25 -> 57.7 mm, vias 0 -> 6
- net VCC: track 36.6 -> 0.00 mm, vias 4 -> 0
- net D+: track 2.87 -> 16.0 mm, vias 0 -> 2
- net D-: track 2.99 -> 15.0 mm
- net Net-(J3-A): track 0.00 -> 7.21 mm
- net Net-(D2-A): track 15.7 -> 17.9 mm
- net 5V: track 16.4 -> 18.3 mm
- net P_46: track 26.4 -> 27.8 mm
- net P_41: track 31.6 -> 32.6 mm
- net P_42: track 34.2 -> 35.1 mm
- net P_44: track 31.6 -> 32.5 mm
- net P_45: track 29.0 -> 29.9 mm
- net P_43: track 34.2 -> 35.1 mm
- net P_48: track 33.8 -> 34.4 mm
- net P_40: vias 1 -> 2

Commit message: did some works.
Parts:
- added G***: LOGO, IOT-Mess-Footprints:catIcon8x8, B.Cu at (204.0, 80.5)
Routing:
- net +3.3V: track 57.7 -> 54.4 mm
Other:
- board text added: "1"
- board text added: "10 9"
- board text added: "11 12"
- board text added: "12 11"
- board text added: "13 14"
- board text added: "14 13"
- board text added: "15 16"
- board text added: "16 15"
- board text added: "17 18"
- board text added: "18 17"
- board text added: "19 20"
- board text added: "2"
- board text added: "20 19"
- board text added: "21 22"
- board text added: "22 21"
- board text added: "23 24"
- board text added: "24 23"
- board text added: "25 26"
- board text added: "26 25"
- board text added: "27 28"
- board text added: "28 27"
- board text added: "29"
- board text added: "3"
- board text added: "30"
- board text added: "31"
- board text added: "32"
- board text added: "33"
- board text added: "34"
- board text added: "35"
- board text added: "36"
- board text added: "37"
- board text added: "38"
- board text added: "39"
- board text added: "3V 45"
- board text added: "4"
- board text added: "40"
- board text added: "41"
- board text added: "42"
- board text added: "43 D+"
- board text added: "44 D-"
- board text added: "45 3V"
- board text added: "46 G"
- board text added: "47 5V"
- board text added: "48"
- board text added: "5"
- board text added: "5V 47"
- board text added: "6"
- board text added: "7"
- board text added: "8"
- board text added: "9 10"
- board text added: "D+ 43"
- board text added: "D- 44"
- board text added: "G 46"
- board text added: "IOT_Mess CH_P48 V1.0 7/5/25"
