File: IOT-Mess-CH_P48/IOT-Mess-P48.kicad_sch (KiCad schematic)
At the start: 29 parts, among them J1 Conn_02x19_Odd_Even, J10 Jumper, J11 Jumper, J12 Jumper, J14 Jumper, J2 Conn_02x19_Odd_Even, J3 Jumper_2, J6 Jumper, J7 Jumper, J8 Jumper, K1 Crystal, K32 Crystal, SW11 SW_Push, U10 USB_C_Receptacle_USB2.0_16P, U3 CH32L103C8T6, U6 ME6211C33M5

Commit message: did some works.
Parts:
- removed D3: SS14, Diode_SMD:D_SMA, symbol Diode:SS14
- removed F1: Fuse_Small, symbol Device:Fuse_Small
- removed J8: Jumper, IOT-Mess-Footprints:Jumper-3_P1.3mm_Open_RoundedPad1.0x1.5mm, symbol Jumper:SolderJumper_3_Open
- added D2: 1N5819WS, Diode_SMD:D_SOD-323, symbol Diode:1N5819WS
- added J4: Jumper_2, IOT-Mess-Footprints:Jumpper-triangle, symbol Jumper:Jumper_2_Small_Open
Connections:
- net VCC is gone; now on net +3.3V: J14.2 (C), J3.2 (B), J6.2 (C), J7.2 (C)
- net +3.3V: no longer J3.1 (A), U6.5 (V_{OUT})
- net 5V: now also D2.1 (K), J4.2 (B)
- net at U10.A4 (VBUS), U10.A9 (VBUS), U10.B4 (VBUS)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: now also D2.2 (A), J4.1 (A)
- new net: J3.1 (A), U6.5 (V_{OUT})
Other:
- moved on the sheet: C2, C4, C5, J3, U6

Commit message: did some works.
Parts:
- added J5: Conn_01x05_Pin, Connector_PinHeader_2.54mm:PinHeader_1x05_P2.54mm_Vertical, symbol Connector:Conn_01x05_Pin
Connections:
- net +3.3V: now also J5.3V (Pin_3)
- net 5V: now also J5.5V (Pin_1)
- net D+: now also J5.D+
- net D-: now also J5.D- (Pin_4)
- net GND: now also J5.G (Pin_2)
Other:
- moved on the sheet: U1

Commit message: did some works.
Connections:
- net +3.3V: now also J5.3 (Pin_3); no longer J5.3V (Pin_3)
- net 5V: now also J5.1 (Pin_1); no longer J5.5V (Pin_1)
- net D+: now also J5.5 (Pin_5); no longer J5.D+
- net D-: now also J5.4 (Pin_4); no longer J5.D- (Pin_4)
- net GND: now also J5.2 (Pin_2); no longer J5.G (Pin_2)
Changed lines of the file:
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@@
 	(wire
 		(pts
+			(xy 173.99 217.17) (xy 162.56 217.17)
+		)
+		(stroke
+			(width 0)
+			(type default)
+		)
+	)
+	(wire
+		(pts
 			(xy 227.33 63.5) (xy 227.33 69.85)
 		)
@@
 	(wire
 		(pts
+			(xy 173.99 212.09) (xy 173.99 217.17)
+		)
+		(stroke
+			(width 0)
+			(type default)
+		)
+	)
+	(wire
+		(pts
 			(xy 162.56 212.09) (xy 162.56 217.17)
 		)
@@
 	)
 	(symbol
+		(lib_id "power:PWR_FLAG")
+		(at 173.99 212.09 0)
+		(unit 1)
+		(exclude_from_sim no)
+		(in_bom yes)
+		(on_board yes)
+		(dnp no)
+		(fields_autoplaced yes)
+		(property "Reference" "#FLG06"
+			(at 173.99 210.185 0)
+			(effects
+				(font
+					(size 1.27 1.27)
+				)
+				(hide yes)
+			)
+		)
+		(property "Value" "PWR_FLAG"
+			(at 173.99 207.01 0)
+			(effects
+				(font
+					(size 1.27 1.27)
+				)
+			)
+		)
+		(property "Footprint" ""
+			(at 173.99 212.09 0)
+			(effects
+				(font
+					(size 1.27 1.27)
+				)
+				(hide yes)
+			)
+		)
+		(property "Datasheet" "~"
+			(at 173.99 212.09 0)
+			(effects
+				(font
+					(size 1.27 1.27)
+				)
+				(hide yes)
+			)
+		)
+		(property "Description" "Special symbol for telling ERC where power comes from"
+			(at 173.99 212.09 0)
+			(effects
+				(font
+					(size 1.27 1.27)
+				)
+				(hide yes)
+			)
+		)
+		(pin "1"
+		)
+		(instances
+			(project "IOT-Mess-P48"
+				(path "/e8b1b29c-6130-44f1-99c5-074e206e80b8"
+					(reference "#FLG06")
+					(unit 1)
+				)
+			)
+		)
+	)
+	(symbol
 		(lib_id "Connector_Generic:Conn_02x19_Odd_Even")
 		(at 365.76 217.17 0)
@@
 			)
 		)
-		(pin "D+"
+		(pin "3"
 		)
-		(pin "D-"
+		(pin "5"
 		)
-		(pin "3V"
+		(pin "1"
 		)
-		(pin "5V"
+		(pin "2"
 		)
-		(pin "G"
+		(pin "4"
 		)
 		(instances
