File: IOT-Mess-ESP32/IOT-Mess-ESP32.kicad_pcb (KiCad board)
At the start: 2 copper layers, 29.1 x 49.5 mm, 28 parts, among them J1 Conn_01x19_Pin, J10 Jumper, J2 Conn_01x19_Pin, J3 Jumper_2, J4 Jumper_2, J5 Conn_01x06_Pin, J7 Jumper, J8 Jumper, J9 Jumper, SW10 SW_Push, SW11 SW_Push, U10 USB_C_Receptacle_USB2.0_16P, U2 ESP32-C6-MINI-1, U4 ESP32-S2-WROVER, U6 ME6211C33M5

Commit message: did some works.
Parts:
- added G***: LOGO, catIcon.preety:catIcon8x8, B.Cu at (103.0, 112.3)
- moved J1 79.2 mm to (93.2, 78.6)
- moved C4 79.2 mm to (106.1, 112.4)
- moved C5 79.2 mm to (113.1, 112.4)
- moved C9 79.2 mm to (111.2, 116.1)
- moved D1 79.2 mm to (97.3, 113.8)
- moved J5 79.2 mm to (112.3, 107.5)
- moved J7 79.2 mm to (101.8, 102.5)
- moved R9 79.2 mm to (98.9, 111.3)
- moved SW11 79.2 mm to (97.7, 120.8)
- moved U10 79.2 mm to (105.8, 123.6)
- moved U4 79.2 mm to (106.0, 90.4)
- moved C10 79.2 mm to (100.5, 116.2)
- moved C2 79.2 mm to (114.9, 112.4)
- moved D2 79.2 mm to (105.9, 116.0)
- moved D4 79.2 mm to (102.1, 111.3)
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Routing:
- net VCC: track 0.00 -> 9.45 mm, vias 0 -> 1
- net Net-(D2-K): track 15.1 -> 18.9 mm
- net P2: track 89.6 -> 91.8 mm, vias 7 -> 9
- net 5V: track 19.7 -> 20.1 mm, vias 2 -> 3
Other:
- board size 29.1 x 49.5 mm -> 29 x 49.5 mm
- board text added: "3.3V"
- board text added: "5V"
- board text added: "D+"
- board text added: "D-"
- board text added: "GND"
- board text added: "IOT_Mess ESP32 V1.0"
- board text added: "LED"
- board text added: "P1"
- board text added: "P10"
- board text added: "P11"
- board text added: "P12"
- board text added: "P13"
- board text added: "P14"
- board text added: "P15"
- board text added: "P17"
- board text added: "P18"
- board text added: "P19"
- board text added: "P2"
- board text added: "P20"
- board text added: "P21"
- board text added: "P22"
- board text added: "P23"
- board text added: "P24"
- board text added: "P25"
- board text added: "P27"
- board text added: "P28"
- board text added: "P29"
- board text added: "P3"
- board text added: "P30"
- board text added: "P31"
- board text added: "P32"
- board text added: "P33"
- board text added: "P34"
- board text added: "P35"
- board text added: "P36"
- board text added: "P37"
- board text added: "P38"
- board text added: "P39"
- board text added: "P4"
- board text added: "P40"
- board text added: "P5"
- board text added: "P6"
- board text added: "P7"
- board text added: "P8"
- board text added: "P9"

Commit message: did some works.
Parts:
- turned J3 to 90 degrees
Connections:
- J3 pad 1: P2 -> Net-(J3-A)
- J3 pad 2: VCC -> P2
- R5 pad 1: VCC -> P2
- U6 pad 5: P2 -> Net-(J3-A)
Routing:
- net VCC: track 9.45 -> 0.00 mm, vias 1 -> 0
- net Net-(J3-A): track 0.00 -> 3.65 mm, vias 0 -> 1
- net P2: track 91.8 -> 94.8 mm, vias 9 -> 10
Changed lines of the file:
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@@
 	(net 5 "P3")
 	(net 6 "Net-(D1-A)")
-	(net 7 "VCC")
+	(net 7 "Net-(J3-A)")
 	(net 8 "LED22")
 	(net 9 "D-")
@@
 			(layers "F.Cu" "F.Mask" "F.Paste")
 			(roundrect_rratio 0.25)
-			(net 3 "P2")
+			(net 7 "Net-(J3-A)")
 			(pinfunction "V_{OUT}")
 			(pintype "power_out")
@@
 			(layers "F.Cu" "F.Mask" "F.Paste")
 			(roundrect_rratio 0.25)
-			(net 7 "VCC")
+			(net 3 "P2")
 			(pintype "passive")
 		)
@@
 			(pintype "bidirectional")
 		)
-		(zone
-			(net 0)
-			(net_name "")
-			(layers "F.Cu" "B.Cu")
-			(name "antenna keepout")
-			(hatch edge 0.508)
-			(connect_pads
-				(clearance 0)
-			)
-			(min_thickness 0.254)
-			(filled_areas_thickness no)
-			(keepout
-				(tracks not_allowed)
-				(vias not_allowed)
-				(pads not_allowed)
-				(copperpour not_allowed)
-				(footprints not_allowed)
-			)
-			(placement
-				(enabled no)
-				(sheetname "")
-			)
-			(fill
-				(thermal_gap 0.508)
-				(thermal_bridge_width 0.508)
-			)
-			(polygon
-				(pts
-					(xy 114.929 76.720002) (xy 96.929 76.720002) (xy 96.929 70.770002) (xy 114.929 70.770002)
-				)
-			)
-		)
 		(embedded_fonts no)
 		(model "C:/Users/uni/Documents/Hardware/IOT-Mess-Hardware/3D-Models/ESP32-WROOM-32--3DModel-STEP-1.STEP"
@@
 	(footprint "IOT-Mess-Footprints:Jumpper-triangle"
 		(layer "B.Cu")
-		(at 109.63 112.615001 -90)
+		(at 109.63 112.615001 90)
 		(descr "SMD Solder Jumper, 1x1.5mm Triangular Pads, 0.3mm gap, open")
 		(tags "solder jumper open")
@@
 		)
 		(property "Datasheet" ""
-			(at 0 0 90)
+			(at 0 0 270)
 			(unlocked yes)
 			(layer "B.Fab")
@@
 		)
 		(property "Description" "Jumper, 2-pole, small symbol, open"
-			(at 0 0 90)
+			(at 0 0 270)
 			(unlocked yes)
 			(layer "B.Fab")
@@
 		)
 		(fp_line
-			(start -1.4 0.7)
-			(end 1.4 0.7)
+			(start 1.4 -0.7)
+			(end -1.4 -0.7)
 			(stroke
 				(width 0.12)
@@
 		)
 		(fp_line
-			(start 1.4 0.7)
-			(end 1.4 -0.7)
+			(start -1.4 -0.7)
+			(end -1.4 0.7)
 			(stroke
 				(width 0.12)
@@
 		)
 		(fp_line
-			(start -1.4 -0.7)
-			(end -1.4 0.7)
+			(start 1.4 0.7)
+			(end 1.4 -0.7)
 			(stroke
 				(width 0.12)
@@
 		)
 		(fp_line
-			(start 1.4 -0.7)
-			(end -1.4 -0.7)
+			(start -1.4 0.7)
+			(end 1.4 0.7)
 			(stroke
 				(width 0.12)
@@
 		)
 		(fp_line
-			(start -1.65 0.8)
-			(end 1.65 0.8)
+			(start 1.65 -0.8)
+			(end -1.65 -0.8)
 			(stroke
 				(width 0.05)
@@
 		)
 		(fp_line
-			(start -1.65 0.8)
-			(end -1.65 -0.8)
+			(start 1.65 -0.8)
+			(end 1.65 0.8)
 			(stroke
 				(width 0.05)
@@
 		)
 		(fp_line
-			(start 1.65 -0.8)
-			(end 1.65 0.8)
+			(start -1.65 0.8)
+			(end -1.65 -0.8)
 			(stroke
 				(width 0.05)
@@
 		)
 		(fp_line
-			(start 1.65 -0.8)
-			(end -1.65 -0.8)
+			(start -1.65 0.8)
+			(end 1.65 0.8)
 			(stroke
 				(width 0.05)
@@
 		)
 		(pad "1" smd custom
-			(at -0.724999 0 270)
+			(at -0.724999 0 90)
 			(size 0.3 0.3)
 			(layers "B.Cu" "B.Mask")
-			(net 3 "P2")
+			(net 7 "Net-(J3-A)")
 			(pinfunction "A")
 			(pintype "passive")
@@
 		)
 		(pad "2" smd custom
-			(at 0.724999 0 270)
+			(at 0.724999 0 90)
 			(size 0.3 0.3)
 			(layers "B.Cu" "B.Mask")
-			(net 7 "VCC")
+			(net 3 "P2")
 			(pinfunction "B")
 			(pintype "passive")
@@
 			(layers "B.Cu" "B.Mask" "B.Paste")
 			(net 36 "P33")
-			(pinfunction "IO08")
+			(pinfunction "IO08/SDA")
 			(pintype "bidirectional")
 		)
@@
 			(layers "B.Cu" "B.Mask" "B.Paste")
 			(net 30 "P32")
-			(pinfunction "IO09")
+			(pinfunction "IO09/SCL")
 			(pintype "bidirectional")
 		)
@@
 			(layers "B.Cu" "B.Mask" "B.Paste")
 			(net 35 "P30")
-			(pinfunction "IO11")
+			(pinfunction "IO11/MOSI")
 			(pintype "bidirectional")
 		)
@@
 			(layers "B.Cu" "B.Mask" "B.Paste")
 			(net 29 "P29")
-			(pinfunction "IO12")
+			(pinfunction "IO12/CLK")
 			(pintype "bidirectional")
 		)
@@
 			(layers "B.Cu" "B.Mask" "B.Paste")
 			(net 26 "P28")
-			(pinfunction "IO13")
+			(pinfunction "IO13/MISO")
 			(pintype "bidirectional")
 		)
@@
 			(layers "B.Cu" "B.Mask" "B.Paste")
 			(net 23 "P14")
-			(pinfunction "IO35")
+			(pinfunction "IO35/MOSI")
 			(pintype "bidirectional")
 		)
@@
 			(layers "B.Cu" "B.Mask" "B.Paste")
 			(net 22 "P13")
-			(pinfunction "IO36")
+			(pinfunction "IO36/CLK")
 			(pintype "bidirectional")
 		)
@@
 			(layers "B.Cu" "B.Mask" "B.Paste")
 			(net 25 "P12")
-			(pinfunction "IO37")
+			(pinfunction "IO37/MISO")
 			(pintype "bidirectional")
 		)
@@
 	)
 	(segment
-		(start 107.485499 112.126501)
-		(end 107.485499 109.303503)
+		(start 97.439 115.230002)
+		(end 96.514 116.155002)
 		(width 0.2)
 		(layer "F.Cu")
@@
 	)
 	(segment
-		(start 97.439 115.230002)
-		(end 96.514 116.155002)
+		(start 102.539 81.450002)
+		(end 102.529 81.460002)
 		(width 0.2)
 		(layer "F.Cu")
@@
 	)
 	(segment
-		(start 102.539 81.450002)
-		(end 102.529 81.460002)
+		(start 103.15 113.37)
+		(end 102.759998 113.760002)
+		(width 0.2)
+		(layer "F.Cu")
+		(net 3)
+	)
+	(segment
+		(start 107.454003 111.8)
+		(end 106.099 113.155003)
+		(width 0.2)
+		(layer "F.Cu")
+		(net 3)
+	)
+	(segment
+		(start 102.759998 113.760002)
+		(end 101.354 113.760002)
 		(width 0.2)
 		(layer "F.Cu")
@@
 	)
 	(segment
-		(start 108.448999 113.090001)
-		(end 107.485499 112.126501)
+		(start 110.07 84.24)
+		(end 110.07 81.72)
 		(width 0.2)
 		(layer "F.Cu")
@@
 	)
 	(segment
-		(start 110.07 84.24)
-		(end 110.07 81.72)
+		(start 97.179 79.530002)
+		(end 97.697 79.530002)
 		(width 0.2)
 		(layer "F.Cu")
@@
 	)
 	(segment
-		(start 97.179 79.530002)
-		(end 97.697 79.530002)
+		(start 107.485499 111.8)
+		(end 107.485499 109.303503)
 		(width 0.2)
 		(layer "F.Cu")
@@
 	)
 	(segment
+		(start 103.15 112.68)
+		(end 103.15 113.37)
+		(width 0.2)
+		(layer "F.Cu")
+		(net 3)
+	)
+	(segment
+		(start 103.21 112.62)
+		(end 103.15 112.68)
+		(width 0.2)
+		(layer "F.Cu")
+		(net 3)
+	)
+	(segment
 		(start 93.229 81.100002)
 		(end 94.799 79.530002)
@@
 	)
 	(segment
+		(start 107.485499 111.8)
+		(end 107.454003 111.8)
+		(width 0.2)
+		(layer "F.Cu")
+		(net 3)
+	)
+	(segment
 		(start 114.529 116.960002)
 		(end 114.529 116.585002)
@@
 		(net 3)
 	)
-	(segment
-		(start 108.449001 113.090002)
-		(end 106.164001 113.090002)
-		(width 0.2)
-		(layer "F.Cu")
-		(net 3)
-	)
 	(via
 		(at 113.25 109.7)
@@
 	)
 	(via
+		(at 103.21 112.62)
+		(size 0.6)
+		(drill 0.3)
+		(layers "F.Cu" "B.Cu")
+		(net 3)
+	)
+	(via
 		(at 104.878 113.300002)
 		(size 0.6)
@@
 	)
 	(segment
-		(start 107.609 109.260002)
-		(end 107.569 109.220002)
-		(width 0.2)
-		(layer "B.Cu")
-		(net 3)
-	)
-	(segment
 		(start 113.389998 109.759998)
 		(end 114.4 110.77)
@@
 	)
 	(segment
-		(start 110.77 110.750002)
-		(end 110.77 109.220002)
-		(width 0.2)
-		(layer "B.Cu")
-		(net 3)
-	)
-	(segment
 		(start 112.770002 109.220002)
 		(end 110.77 109.220002)
@@
 	)
 	(segment
+		(start 109.63 111.890002)
+		(end 109.63 111.281002)
+		(width 0.2)
+		(layer "B.Cu")
+		(net 3)
+	)
+	(segment
 		(start 114.4 110.77)
 		(end 114.4 116.831002)
@@
 	)
 	(segment
-		(start 109.63 111.890002)
-		(end 110.77 110.750002)
+		(start 104.197998 112.62)
+		(end 104.878 113.300002)
 		(width 0.2)
 		(layer "B.Cu")
@@
 	)
 	(segment
+		(start 103.21 112.62)
+		(end 104.197998 112.62)
+		(width 0.2)
+		(layer "B.Cu")
+		(net 3)
+	)
+	(segment
+		(start 109.63 111.281002)
+		(end 107.569 109.220002)
+		(width 0.2)
+		(layer "B.Cu")
+		(net 3)
+	)
+	(segment
 		(start 109.929 88.29)
 		(end 109.929 91.370002)
@@
 	)
 	(segment
-		(start 103.15 113.37)
-		(end 102.759998 113.760002)
-		(width 0.2)
-		(layer "F.Cu")
-		(net 7)
-	)
-	(segment
-		(start 102.759998 113.760002)
-		(end 101.354 113.760002)
-		(width 0.2)
-		(layer "F.Cu")
-		(net 7)
-	)
-	(segment
-		(start 103.15 112.68)
-		(end 103.15 113.37)
+		(start 107.5 113.9)
+		(end 107.639 113.9)
 		(width 0.2)
 		(layer "F.Cu")
@@
 	)
 	(segment
-		(start 103.21 112.62)
-		(end 103.15 112.68)
+		(start 107.639 113.9)
+		(end 108.448999 113.090001)
 		(width 0.2)
 		(layer "F.Cu")
@@
 	)
 	(via
-		(at 103.21 112.62)
+		(at 107.5 113.9)
 		(size 0.6)
 		(drill 0.3)
@@
 	)
 	(segment
-		(start 108.91 112.62)
-		(end 109.63 113.34)
+		(start 109.07 113.9)
+		(end 107.5 113.9)
 		(width 0.2)
 		(layer "B.Cu")
@@
 	)
 	(segment
-		(start 103.21 112.62)
-		(end 108.91 112.62)
+		(start 109.63 113.34)
+		(end 109.07 113.9)
 		(width 0.2)
 		(layer "B.Cu")
@@
 			"77f62475-7d0d-4fdd-b07b-b1b5cac67f31" "851e3314-e08d-4aca-8f6c-6e38de5a96d9"
 			"8a7c116d-4e5d-4887-8209-1413465551ee" "a8424079-3ad3-4b8d-992d-3e56e6e6af6a"
-			"c0f806cc-e8d2-4b49-bad2-86c02b9a018b" "fbf5f902-b4c3-491d-bc7b-f5faca34f5c3"
+			"c0f806cc-e8d2-4b49-bad2-86c02b9a018b"
 		)
 	)

Commit message: did some works.
Parts:
- removed the G*** at (103.0, 112.3)
- added G***: LOGO, IOT-Mess-Footprints:catIcon8x8, B.Cu at (103.5, 112.5)
Connections:
- net LED22 renamed Net-(J5-Pin_6)
Other:
- board text added: "1"
- board text added: "10"
- board text added: "11"
- board text added: "12"
- board text added: "13"
- board text added: "14"
- board text added: "15"
- board text added: "17"
- board text added: "18"
- board text added: "19"
- board text added: "2"
- board text added: "20"
- board text added: "21"
- board text added: "22"
- board text added: "23"
- board text added: "24"
- board text added: "25"
- board text added: "27"
- board text added: "28"
- board text added: "29"
- board text added: "3"
- board text added: "30"
- board text added: "31"
- board text added: "32"
- board text added: "33"
- board text added: "34"
- board text added: "35"
- board text added: "36"
- board text added: "37"
- board text added: "38"
- board text added: "39"
- board text added: "4"
- board text added: "40"
- board text added: "5"
- board text added: "6"
- board text added: "7"
- board text added: "8"
- board text added: "9"
- board text added: "G"
- board text added: "IOT_Mess ESP32 V1.0 7/5/25"
- board text removed: "GND"
- board text removed: "IOT_Mess ESP32 V1.0"
- board text removed: "P1"
- board text removed: "P10"
- board text removed: "P11"
- board text removed: "P12"
- board text removed: "P13"
- board text removed: "P14"
- board text removed: "P15"
- board text removed: "P17"
- board text removed: "P18"
- board text removed: "P19"
- board text removed: "P2"
- board text removed: "P20"
- board text removed: "P21"
- board text removed: "P22"
- board text removed: "P23"
- board text removed: "P24"
- board text removed: "P25"
- board text removed: "P27"
- board text removed: "P28"
- board text removed: "P29"
- board text removed: "P3"
- board text removed: "P30"
- board text removed: "P31"
- board text removed: "P32"
- board text removed: "P33"
- board text removed: "P34"
- board text removed: "P35"
- board text removed: "P36"
- board text removed: "P37"
- board text removed: "P38"
- board text removed: "P39"
- board text removed: "P4"
- board text removed: "P40"
- board text removed: "P5"
- board text removed: "P6"
- board text removed: "P7"
- board text removed: "P8"
- board text removed: "P9"
