File: IOT-Mess-ESP_P16/IOT-Mess-ESP_P16.kicad_pcb (KiCad board)
At the start: 2 copper layers, 28.9 x 32.4 mm, 24 parts, among them J1 Conn_01x09_Pin, J2 Conn_01x09_Pin, J3 Jumper_2, J4 Jumper_2, J5 Jumper_2, J6 Jumper_2, SW10 SW_Push, SW11 SW_Push, U1 ESP-12F, U10 USB_C_Receptacle_USB2.0_16P, U5 ESP32-C3-WROOM-02, U6 ME6211C33M5

Commit message: did some works.
Parts:
- J1: value Conn_01x09_Pin -> Conn_01x10_Pin; footprint Connector_PinHeader_2.54mm:PinHeader_1x09_P2.54mm_Vertical -> Connector_PinHeader_2.54mm:PinHeader_1x10_P2.54mm_Vertical
- moved D2 5.25 mm to (129.4, 98.7), turned to 0 degrees
- moved C9 4.87 mm to (126.5, 103.9), turned to 90 degrees
- moved R16 0.89 mm to (126.5, 107.2), turned to -90 degrees
- turned J3 to 180 degrees
Connections:
- C4 pad 1: Net-(J3-A) -> P1
- J3 pad 1: Net-(J3-A) -> P1
- J3 pad 2: P1 -> Net-(J3-B)
- U1 pad 16: unconnected-(U1-GPIO15/SS-Pad16) -> P13
- U6 pad 5: Net-(J3-A) -> Net-(J3-B)
Routing:
- net Net-(J3-A): track 23.2 -> 0.00 mm
- net 5V: track 15.4 -> 24.9 mm
- net Net-(J3-B): track 0.00 -> 8.13 mm
- net Net-(D2-A): track 16.9 -> 24.2 mm
- net P13: track 19.6 -> 26.3 mm
- net P1: track 75.5 -> 81.2 mm
- net P12: track 16.4 -> 18.6 mm
- net P2: track 58.7 -> 60.2 mm
- net BOOT: track 39.4 -> 40.8 mm
- net P14: track 17.4 -> 16.9 mm
- net P9: vias 0 -> 1
Other:
- board size 28.9 x 32.4 mm -> 29.4 x 32.4 mm

Commit message: did some works.
Parts:
- removed the G*** at (144.6, 110.2)
- added G***: LOGO, IOT-Mess-Footprints:catIcon8x8, B.Cu at (144.7, 110.0)
- moved J4 0.71 mm to (126.5, 102.4)
Routing:
- net 5V: track 24.9 -> 25.7 mm
- net Net-(D2-A): track 24.2 -> 24.9 mm
Other:
- board text added: "1"
- board text added: "10"
- board text added: "11"
- board text added: "12"
- board text added: "13"
- board text added: "14"
- board text added: "15"
- board text added: "16"
- board text added: "17"
- board text added: "18"
- board text added: "2"
- board text added: "3"
- board text added: "4"
- board text added: "5"
- board text added: "5V"
- board text added: "6"
- board text added: "7"
- board text added: "8"
- board text added: "9"
- board text added: "IOT_Mess ESP_P16 V1.0 7/5/25"
- board text removed: "IOT_Mess ESP_P16 V1.0"
- board text removed: "P1"
- board text removed: "P10"
- board text removed: "P11"
- board text removed: "P12"
- board text removed: "P13"
- board text removed: "P14"
- board text removed: "P15"
- board text removed: "P16"
- board text removed: "P17"
- board text removed: "P18"
- board text removed: "P2"
- board text removed: "P3"
- board text removed: "P4"
- board text removed: "P5"
- board text removed: "P6"
- board text removed: "P7"
- board text removed: "P8"
- board text removed: "P9"
