File: IOT-Mess-ESP_P16/IOT-Mess-ESP_P16.kicad_sch (KiCad schematic)
At the start: 14 parts, among them J3 Jumper_2, J4 Jumper_2, U10 USB_C_Receptacle_USB2.0_16P, U6 ME6211C33M5

Commit message: did some works.
Parts:
- removed R2, R3: 5.1K, Resistor_SMD:R_0603_1608Metric, symbol Device:R
- added C10, C9: .1u, Capacitor_SMD:C_0603_1608Metric, symbol Device:C
- added J1, J2: Conn_01x09_Pin, Connector_PinHeader_2.54mm:PinHeader_1x09_P2.54mm_Vertical, symbol Connector:Conn_01x09_Pin
- added J5, J6: Jumper_2, IOT-Mess-Footprints:Jumpper-triangle, symbol Jumper:Jumper_2_Small_Open
- added R10, R15, R16: 10K, Resistor_SMD:R_0603_1608Metric, symbol Device:R
- added SW10, SW11: SW_Push, Button_Switch_SMD:SW_SPST_PTS810, symbol Switch:SW_Push
- added U1: ESP-12F, RF_Module:ESP-12E, symbol RF_Module:ESP-12F
- added U5: ESP32-C3-WROOM-02, RF_Module:ESP32-C3-WROOM-02, symbol Espressif:ESP32-C3-WROOM-02
Connections:
- net VCC is gone; now on net +3.3V: J3.2 (B), R5.1, TP1.1
- net +3.3V: now also J1.1 (Pin_1), R10.2, R15.2, R16.2, U1.8 (VCC), U5.1 (3V3); no longer C4.1, J3.1 (A), U6.5 (V_{OUT})
- net D+: now also J6.2 (B)
- net D-: now also J5.2 (B)
- net GND: now also C10.2, C9.2, J1.9 (Pin_9), SW10.2, SW11.2, U1.15 (GND), U5.19 (GND), U5.9 (GND)
- net CC1: no longer names the net of U10.A5 (CC1)
- net CC2: no longer names the net of U10.B5 (CC2)
- new net: R10.1, U1.3 (EN)
- new net: C4.1, J3.1 (A), U6.5 (V_{OUT})
- new net BOOT: C9.1, J1.8 (Pin_8), R16.1, SW10.1, U1.18 (GPIO0), U5.8 (GPIO9/SCL)
- new net P10: J2.9 (Pin_9), U1.12 (GPIO10), U5.10 (GPIO10)
- new net P11: J2.8 (Pin_8), U5.11 (GPIO20/U0RXD)
- new net P12: J2.7 (Pin_7), U1.7 (GPIO13/MOSI), U5.12 (GPIO21/U0TXD)
- new net P13: J2.6 (Pin_6), J5.1 (A), U5.13 (GPIO18/USB_D-)
- new net P14: J2.5 (Pin_5), J6.1 (A), U5.14 (GPIO19/USB_D+)
- new net P15: J2.4 (Pin_4), U1.6 (GPIO12/MISO), U5.15 (GPIO3/ADC1_CH3)
- new net P16: J2.3 (Pin_3), U1.5 (GPIO14/SCK), U5.16 (GPIO2/ADC1_CH2)
- new net P17: J2.2 (Pin_2), U1.4 (GPIO16), U5.17 (GPIO1/ADC1_CH1/XTAL_32K_N)
- new net P18: J2.1 (Pin_1), U1.2 (ADC), U5.18 (GPIO0/ADC1_CH0/XTAL_32K_P)
- new net P2: C10.1, J1.2 (Pin_2), R15.1, SW11.1, U1.1 (~{RST}), U5.2 (EN/CHIP_PU)
- new net P3: J1.3 (Pin_3), U1.22 (GPIO1/TXD), U5.3 (GPIO4/SCK)
- new net P4: J1.4 (Pin_4), U1.21 (GPIO3/RXD), U5.4 (GPIO5/MISO)
- new net P5: J1.5 (Pin_5), U1.20 (GPIO5/SCL), U5.5 (GPIO6/MOSI)
- new net P6: J1.6 (Pin_6), U1.19 (GPIO4/SDA), U5.6 (GPIO7/SS)
- new net P7: J1.7 (Pin_7), U1.17 (GPIO2), U5.7 (GPIO8/SDA)
- no-connect marks 2 -> 9
Other:
- moved on the sheet: C2, C4, C5, D1, D2, J3, J4, R5, TP1, TP2, U6

Commit message: did some works.
Parts:
- removed J1: Conn_01x09_Pin, Connector_PinHeader_2.54mm:PinHeader_1x09_P2.54mm_Vertical, symbol Connector:Conn_01x09_Pin
- removed TP1, TP2: TestPoint, symbol Connector:TestPoint
- added J1: Conn_01x10_Pin, Connector_PinHeader_2.54mm:PinHeader_1x10_P2.54mm_Vertical, symbol Connector:Conn_01x10_Pin
Connections:
- net +3.3V: now also C4.1, J3.1 (A), J1.1 (Pin_1); no longer J3.2 (B)
- net 5V: now also J1.10 (Pin_10)
- net BOOT: now also J1.8 (Pin_8)
- net GND: now also J1.9 (Pin_9)
- net P13: now also U1.16 (GPIO15/SS)
- net P2: now also J1.2 (Pin_2)
- net P3: now also J1.3 (Pin_3)
- net P4: now also J1.4 (Pin_4)
- net P5: now also J1.5 (Pin_5)
- net P6: now also J1.6 (Pin_6)
- net P7: now also J1.7 (Pin_7)
- new net: J3.2 (B), U6.5 (V_{OUT})
- no-connect marks 9 -> 10
Other:
- moved on the sheet: C4, D1, J3, R5

Commit message: did some works.
Parts:
- U5: footprint RF_Module:ESP32-C3-WROOM-02 -> PCM_Espressif:ESP32-C3-WROOM-02
Connections:
- no-connect marks 10 -> 9
Changed lines of the file:
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@@
 	)
 	(junction
+		(at 152.4 209.55)
+		(diameter 0)
+		(color 0 0 0 0)
+	)
+	(junction
 		(at 125.73 232.41)
 		(diameter 0)
@@
 	)
 	(no_connect
-		(at 185.42 116.84)
-	)
-	(no_connect
 		(at 124.46 110.49)
 	)
@@
 	(wire
 		(pts
+			(xy 161.29 204.47) (xy 161.29 209.55)
+		)
+		(stroke
+			(width 0)
+			(type default)
+		)
+	)
+	(wire
+		(pts
 			(xy 288.29 168.91) (xy 294.64 168.91)
 		)
@@
 	(wire
 		(pts
+			(xy 152.4 209.55) (xy 152.4 204.47)
+		)
+		(stroke
+			(width 0)
+			(type default)
+		)
+	)
+	(wire
+		(pts
 			(xy 294.64 160.02) (xy 294.64 158.75)
 		)
@@
 	(wire
 		(pts
-			(xy 152.4 214.63) (xy 152.4 209.55)
+			(xy 152.4 209.55) (xy 152.4 214.63)
 		)
 		(stroke
@@
 	(wire
 		(pts
+			(xy 161.29 209.55) (xy 152.4 209.55)
+		)
+		(stroke
+			(width 0)
+			(type default)
+		)
+	)
+	(wire
+		(pts
 			(xy 158.75 214.63) (xy 152.4 214.63)
 		)
@@
 	)
 	(symbol
+		(lib_id "power:PWR_FLAG")
+		(at 161.29 204.47 0)
+		(unit 1)
+		(exclude_from_sim no)
+		(in_bom yes)
+		(on_board yes)
+		(dnp no)
+		(property "Reference" "#FLG06"
+			(at 161.29 202.565 0)
+			(effects
+				(font
+					(size 1.27 1.27)
+				)
+				(hide yes)
+			)
+		)
+		(property "Value" "PWR_FLAG"
+			(at 161.29 199.39 0)
+			(effects
+				(font
+					(size 1.27 1.27)
+				)
+			)
+		)
+		(property "Footprint" ""
+			(at 161.29 204.47 0)
+			(effects
+				(font
+					(size 1.27 1.27)
+				)
+				(hide yes)
+			)
+		)
+		(property "Datasheet" "~"
+			(at 161.29 204.47 0)
+			(effects
+				(font
+					(size 1.27 1.27)
+				)
+				(hide yes)
+			)
+		)
+		(property "Description" "Special symbol for telling ERC where power comes from"
+			(at 161.29 204.47 0)
+			(effects
+				(font
+					(size 1.27 1.27)
+				)
+				(hide yes)
+			)
+		)
+		(pin "1"
+		)
+		(instances
+			(project "IOT-Mess-ESP_P16"
+				(path "/015ef37e-b488-4fc9-8cfc-c186768bee82"
+					(reference "#FLG06")
+					(unit 1)
+				)
+			)
+		)
+	)
+	(symbol
 		(lib_id "Device:R")
 		(at 115.57 87.63 270)
@@
 			)
 		)
-		(property "Description" ""
+		(property "Description" "Power symbol creates a global label with name \"GND\" , ground"
 			(at 182.88 222.25 0)
 			(effects
@@
 			)
 		)
-		(property "Description" ""
+		(property "Description" "Light emitting diode"
+			(at 173.99 214.63 0)
+			(effects
+				(font
+					(size 1.27 1.27)
+				)
+				(hide yes)
+			)
+		)
+		(property "Sim.Pins" "1=K 2=A"
 			(at 173.99 214.63 0)
 			(effects
@@
 	(symbol
 		(lib_id "power:+3.3V")
-		(at 152.4 209.55 0)
+		(at 152.4 204.47 0)
 		(unit 1)
 		(exclude_from_sim no)
@@
 		(dnp no)
 		(property "Reference" "#PWR026"
-			(at 152.4 213.36 0)
+			(at 152.4 208.28 0)
 			(effects
 				(font
@@
 		)
 		(property "Value" "+3.3V"
-			(at 152.4 205.486 0)
+			(at 152.4 200.406 0)
 			(effects
 				(font
@@
 		)
 		(property "Footprint" ""
-			(at 152.4 209.55 0)
+			(at 152.4 204.47 0)
 			(effects
 				(font
@@
 		)
 		(property "Datasheet" ""
-			(at 152.4 209.55 0)
+			(at 152.4 204.47 0)
 			(effects
 				(font
@@
 		)
 		(property "Description" "Power symbol creates a global label with name \"+3.3V\""
-			(at 152.4 209.55 0)
+			(at 152.4 204.47 0)
 			(effects
 				(font
@@
 			)
 		)
-		(property "Footprint" "RF_Module:ESP32-C3-WROOM-02"
+		(property "Footprint" "PCM_Espressif:ESP32-C3-WROOM-02"
 			(at 242.57 128.27 0)
 			(effects
