File: IOT-Mess-Sens/IOT-Mess-Base.kicad_pcb (KiCad board)
At the start: 2 copper layers, 24.5 x 24.5 mm, 34 parts, among them J1 Conn_01x09_Pin, J2 TP_4056, J3 R_DELAY, Q1 AO3400A, Q2 AO3401A, Q3 AO3400A, Q4 AO3401A, Q5 AO3400A, SW2 SW_Push, SW3 SW_Push, U1 INA219AxD, U12 APDS-9960, U13 SHT31-DIS, U17 BH1750FVI-TR, U2 SHT4x, U3 INA219AxDCN, U8 TPL5110

Commit message: did some works.
Connections:
- net DRIVE renamed EN
- net V- renamed Vb
- net Vi+ renamed Va
Changed lines of the file:
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@@
 	(net 2 "GND")
 	(net 3 "+3.3V")
-	(net 4 "Vi+")
+	(net 4 "EN")
 	(net 5 "ADDR")
 	(net 6 "SCL_0")
@@
 	(net 10 "unconnected-(U13-~{RESET}-Pad6)")
 	(net 11 "unconnected-(U13-ALERT-Pad3)")
-	(net 12 "DRIVE")
+	(net 12 "Va")
 	(net 13 "Net-(Q2-G)")
 	(net 14 "DONE")
@@
 	(net 18 "Net-(Q1-D)")
 	(net 19 "unconnected-(J2-Pin_3-Pad3)")
-	(net 20 "V-")
+	(net 20 "Vb")
 	(net 21 "PWR")
 	(footprint "Package_TO_SOT_SMD:SOT-23-8"
@@
 			(layers "F.Cu" "F.Mask" "F.Paste")
 			(roundrect_rratio 0.25)
-			(net 4 "Vi+")
+			(net 12 "Va")
 			(pinfunction "IN+")
 			(pintype "input")
@@
 			(layers "F.Cu" "F.Mask" "F.Paste")
 			(roundrect_rratio 0.25)
-			(net 20 "V-")
+			(net 20 "Vb")
 			(pinfunction "IN-")
 			(pintype "input")
@@
 			(layers "F.Cu" "F.Mask" "F.Paste")
 			(roundrect_rratio 0.25)
-			(net 20 "V-")
+			(net 20 "Vb")
 			(pinfunction "IN-")
 			(pintype "input")
@@
 			(layers "F.Cu" "F.Mask" "F.Paste")
 			(roundrect_rratio 0.25)
-			(net 4 "Vi+")
+			(net 12 "Va")
 			(pinfunction "IN+")
 			(pintype "input")
@@
 			(layers "F.Cu" "F.Mask" "F.Paste")
 			(roundrect_rratio 0.25)
-			(net 12 "DRIVE")
+			(net 4 "EN")
 			(pinfunction "G")
 			(pintype "input")
@@
 			(layers "F.Cu" "F.Mask" "F.Paste")
 			(roundrect_rratio 0.25)
-			(net 12 "DRIVE")
+			(net 4 "EN")
 			(pintype "passive")
 		)
@@
 			(layers "*.Cu" "*.Mask")
 			(remove_unused_layers no)
-			(net 4 "Vi+")
+			(net 12 "Va")
 			(pinfunction "Pin_1")
 			(pintype "passive")
@@
 			(layers "*.Cu" "*.Mask")
 			(remove_unused_layers no)
-			(net 4 "Vi+")
+			(net 12 "Va")
 			(pinfunction "Pin_2")
 			(pintype "passive")
@@
 			(layers "*.Cu" "*.Mask")
 			(remove_unused_layers no)
-			(net 12 "DRIVE")
+			(net 4 "EN")
 			(pinfunction "Pin_6")
 			(pintype "passive")
@@
 			(layers "F.Cu" "F.Mask" "F.Paste")
 			(roundrect_rratio 0.25)
-			(net 20 "V-")
+			(net 20 "Vb")
 			(pinfunction "S")
 			(pintype "passive")
@@
 			(layers "F.Cu" "F.Mask" "F.Paste")
 			(roundrect_rratio 0.25)
-			(net 20 "V-")
+			(net 20 "Vb")
 			(pintype "passive")
 		)
@@
 			(layers "F.Cu" "F.Mask" "F.Paste")
 			(roundrect_rratio 0.25)
-			(net 20 "V-")
+			(net 20 "Vb")
 			(pinfunction "S")
 			(pintype "passive")
@@
 			(layers "F.Cu" "F.Mask" "F.Paste")
 			(roundrect_rratio 0.25)
-			(net 20 "V-")
+			(net 20 "Vb")
 			(pinfunction "VDD")
 			(pintype "bidirectional")
@@
 			(layers "F.Cu" "F.Mask" "F.Paste")
 			(roundrect_rratio 0.25)
-			(net 20 "V-")
+			(net 20 "Vb")
 			(pinfunction "EN/ONE_SHOT")
 			(pintype "input")
@@
 			(size 1.05 0.65)
 			(layers "B.Cu" "B.Mask" "B.Paste")
-			(net 20 "V-")
+			(net 20 "Vb")
 			(pinfunction "1")
 			(pintype "passive")
@@
 			(size 1.05 0.65)
 			(layers "B.Cu" "B.Mask" "B.Paste")
-			(net 20 "V-")
+			(net 20 "Vb")
 			(pinfunction "1")
 			(pintype "passive")
@@
 			(layers "B.Cu" "B.Mask" "B.Paste")
 			(roundrect_rratio 0.204082)
-			(net 20 "V-")
+			(net 20 "Vb")
 			(pintype "passive")
 		)
@@
 			(layers "B.Cu" "B.Mask" "B.Paste")
 			(roundrect_rratio 0.204082)
-			(net 4 "Vi+")
+			(net 12 "Va")
 			(pintype "passive")
 		)
@@
 			(size 1.05 0.65)
 			(layers "B.Cu" "B.Mask" "B.Paste")
-			(net 20 "V-")
+			(net 20 "Vb")
 			(pinfunction "1")
 			(pintype "passive")
@@
 			(size 1.05 0.65)
 			(layers "B.Cu" "B.Mask" "B.Paste")
-			(net 20 "V-")
+			(net 20 "Vb")
 			(pinfunction "1")
 			(pintype "passive")
@@
 	)
 	(segment
-		(start 98.407502 83.942498)
-		(end 99.345499 84.880495)
+		(start 86.225 80.7)
+		(end 86.225 82.799999)
 		(width 0.2)
 		(layer "F.Cu")
@@
 	)
 	(segment
-		(start 85.785 72.96)
-		(end 89.084999 72.96)
+		(start 85.829468 82.924999)
+		(end 83.364467 85.39)
 		(width 0.2)
 		(layer "F.Cu")
@@
 	)
 	(segment
-		(start 97.524018 83.059014)
-		(end 98.407502 83.942498)
+		(start 86.35 82.924999)
+		(end 85.829468 82.924999)
 		(width 0.2)
 		(layer "F.Cu")
@@
 	)
 	(segment
-		(start 99.345499 84.919014)
-		(end 99.345499 88.424501)
+		(start 83.364467 85.39)
+		(end 80.9 85.39)
 		(width 0.2)
 		(layer "F.Cu")
@@
 	)
 	(segment
-		(start 99.345499 88.424501)
-		(end 98.162501 89.607499)
+		(start 86.225 82.799999)
+		(end 86.35 82.924999)
 		(width 0.2)
 		(layer "F.Cu")
 		(net 4)
 	)
-	(via
-		(at 98.407502 83.942498)
-		(size 0.6)
-		(drill 0.3)
-		(layers "F.Cu" "B.Cu")
-		(net 4)
-	)
-	(segment
-		(start 96.2025 75.01)
-		(end 98.29 75.01)
-		(width 0.2)
-		(layer "B.Cu")
-		(net 4)
-	)
-	(segment
-		(start 94.1525 72.96)
-		(end 95.63125 74.43875)
-		(width 0.2)
-		(layer "B.Cu")
-		(net 4)
-	)
-	(segment
-		(start 100.0625 83.1375)
-		(end 99.257502 83.942498)
-		(width 0.2)
-		(layer "B.Cu")
-		(net 4)
-	)
-	(segment
-		(start 100.0625 78.87)
-		(end 100.0625 83.1375)
-		(width 0.2)
-		(layer "B.Cu")
-		(net 4)
-	)
-	(segment
-		(start 98.29 75.01)
-		(end 98.29 76.59)
-		(width 0.2)
-		(layer "B.Cu")
-		(net 4)
-	)
-	(segment
-		(start 89.084999 72.96)
-		(end 94.1525 72.96)
-		(width 0.2)
-		(layer "B.Cu")
-		(net 4)
-	)
-	(segment
-		(start 99.257502 83.942498)
-		(end 98.407502 83.942498)
-		(width 0.2)
-		(layer "B.Cu")
-		(net 4)
-	)
-	(segment
-		(start 95.63125 74.43875)
-		(end 96.2025 75.01)
-		(width 0.2)
-		(layer "B.Cu")
-		(net 4)
-	)
-	(segment
-		(start 98.29 76.59)
-		(end 100.04 78.34)
-		(width 0.2)
-		(layer "B.Cu")
-		(net 4)
-	)
 	(segment
 		(start 95.249018 82.409013)
@@
 	)
 	(segment
-		(start 86.225 80.7)
-		(end 86.225 82.799999)
+		(start 98.407502 83.942498)
+		(end 99.345499 84.880495)
 		(width 0.2)
 		(layer "F.Cu")
@@
 	)
 	(segment
-		(start 85.829468 82.924999)
-		(end 83.364467 85.39)
+		(start 85.785 72.96)
+		(end 89.084999 72.96)
 		(width 0.2)
 		(layer "F.Cu")
@@
 	)
 	(segment
-		(start 86.35 82.924999)
-		(end 85.829468 82.924999)
+		(start 97.524018 83.059014)
+		(end 98.407502 83.942498)
 		(width 0.2)
 		(layer "F.Cu")
@@
 	)
 	(segment
-		(start 83.364467 85.39)
-		(end 80.9 85.39)
+		(start 99.345499 84.919014)
+		(end 99.345499 88.424501)
 		(width 0.2)
 		(layer "F.Cu")
@@
 	)
 	(segment
-		(start 86.225 82.799999)
-		(end 86.35 82.924999)
+		(start 99.345499 88.424501)
+		(end 98.162501 89.607499)
 		(width 0.2)
 		(layer "F.Cu")
 		(net 12)
 	)
+	(via
+		(at 98.407502 83.942498)
+		(size 0.6)
+		(drill 0.3)
+		(layers "F.Cu" "B.Cu")
+		(net 12)
+	)
+	(segment
+		(start 96.2025 75.01)
+		(end 98.29 75.01)
+		(width 0.2)
+		(layer "B.Cu")
+		(net 12)
+	)
+	(segment
+		(start 94.1525 72.96)
+		(end 95.63125 74.43875)
+		(width 0.2)
+		(layer "B.Cu")
+		(net 12)
+	)
+	(segment
+		(start 100.0625 83.1375)
+		(end 99.257502 83.942498)
+		(width 0.2)
+		(layer "B.Cu")
+		(net 12)
+	)
+	(segment
+		(start 100.0625 78.87)
+		(end 100.0625 83.1375)
+		(width 0.2)
+		(layer "B.Cu")
+		(net 12)
+	)
+	(segment
+		(start 98.29 75.01)
+		(end 98.29 76.59)
+		(width 0.2)
+		(layer "B.Cu")
+		(net 12)
+	)
+	(segment
+		(start 89.084999 72.96)
+		(end 94.1525 72.96)
+		(width 0.2)
+		(layer "B.Cu")
+		(net 12)
+	)
+	(segment
+		(start 99.257502 83.942498)
+		(end 98.407502 83.942498)
+		(width 0.2)
+		(layer "B.Cu")
+		(net 12)
+	)
+	(segment
+		(start 95.63125 74.43875)
+		(end 96.2025 75.01)
+		(width 0.2)
+		(layer "B.Cu")
+		(net 12)
+	)
+	(segment
+		(start 98.29 76.59)
+		(end 100.04 78.34)
+		(width 0.2)
+		(layer "B.Cu")
+		(net 12)
+	)

Commit message: did some works.
Parts:
- moved R15 3.93 mm to (98.5, 82.0), turned to 90 degrees
Routing:
- net SDA_0: track 54.0 -> 57.6 mm
- net Vb: track 58.9 -> 61.7 mm
- net +3.3V: track 70.6 -> 71.7 mm, vias 5 -> 4
- net SCL_0: track 50.0 -> 50.8 mm
Other:
- board text added: "3V"
- board text added: "G"
- board text added: "IOT-Mess SENS V1.0 7/5/25"
- board text removed: "3.3"
- board text removed: "GND"
- board text removed: "IOT-Mess SENS V1.0"
