File: IOT-Mess-Sens/IOT-Mess-Base.kicad_sch (KiCad schematic)
At the start: 34 parts, among them J1 Conn_01x09_Pin, J2 TP_4056, J3 R_DELAY, Q1 AO3400A, Q2 AO3401A, Q3 AO3400A, Q4 AO3401A, Q5 AO3400A, SW2 SW_Push, SW3 SW_Push, U1 INA219AxD, U12 APDS-9960, U13 SHT31-DIS, U17 BH1750FVI-TR, U2 SHT4x, U3 INA219AxDCN, U8 TPL5110

Commit message: did some works.
Connections:
- net DRIVE renamed EN
- net V- renamed Vb
- net Vi+ renamed Va
Other:
- moved on the sheet: C6, J2, J3, JP4, JP5, Q1, Q2, Q3, Q4, Q5, R1, R15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

Commit message: did some works.
Other:
- moved on the sheet: C7
