File: Version2/IOT-Mess-BaseSmall/IOT-Mess-BaseSmall.kicad_sch (KiCad schematic)
At the start: 5 parts, among them J1 ESP_P16 / ESP12, J2 ESP_P16 / C3, J22 Lolin32, J3 ESP_P40, J6 CH582

Commit message: added jumper boards.
Parts:
- removed J2: ESP_P16 / C3, IOT-Mess-Footprints:ESP_P16, symbol IOT-Mess:ESP_P16
- removed J22: Lolin32, IOT-Mess-Footprints:Lolin32-Adapter, symbol Connector_Generic:Conn_02x11_Top_Bottom
- added J1, J2, J5, J6, J7, J8, J9: Conn_02x34_Odd_Even, Connector_PinSocket_2.54mm:PinSocket_2x34_P2.54mm_Vertical, symbol Connector_Generic:Conn_02x34_Odd_Even
- added J11: Milk-V Duo, IOT-Mess-Footprints:Milk-V Duo, symbol Connector_Generic:Conn_02x20_Counter_Clockwise
- added J13: SuperMini_ESP32-H2, IOT-Mess-Footprints:SuperMiniH2, symbol IOT-Mess:SuperMini_ESP32-H2
- added J14: Lolin32-Lite, IOT-Mess-Footprints:Lolin32-Lite, symbol IOT-Mess:Lolin32-Lite
- added J15, J18: Conn_02x19_Odd_Even, Connector_PinHeader_2.54mm:PinHeader_2x19_P2.54mm_Vertical, symbol Connector_Generic:Conn_02x19_Odd_Even
- added J17: CH_P20, IOT-Mess-Footprints:CH_P20, symbol IOT-Mess:CH_P20
- added J20, J3, J4: Conn_01x34_Pin, Connector_PinHeader_2.54mm:PinHeader_1x34_P2.54mm_Vertical, symbol Connector:Conn_01x34_Pin
- renumbered J3 to J10, J1 to J12, J6 to J16
Connections:
- net C10: now also J2.19 (Pin_19), J2.20 (Pin_20); no longer J10.P36 (Pin_24)
- net C11: now also J2.21 (Pin_21), J2.22 (Pin_22); no longer J10.P37 (Pin_23)
- net C23: now also J2.45 (Pin_45), J2.46 (Pin_46); no longer J10.P38 (Pin_22)
- net C24: now also J2.47 (Pin_47), J2.48 (Pin_48); no longer J10.P27 (Pin_33)
- net C25: now also J2.49 (Pin_49), J2.50 (Pin_50); no longer J12.P14 (Pin_16)
- net C29: now also J2.57 (Pin_57), J2.58 (Pin_58); no longer J16.A5 (Pin_2)
- net C3: now also J2.5 (Pin_5), J2.6 (Pin_6); no longer J12.P4 (Pin_4)
- net C30: now also J2.59 (Pin_59), J2.60 (Pin_60); no longer J16.A11 (Pin_7)
- net C31: now also J2.61 (Pin_61), J2.62 (Pin_62); no longer J16.A10 (Pin_8)
- net C32: now also J2.63 (Pin_63), J2.64 (Pin_64); no longer J10.P3 (Pin_3)
- net C33: now also J2.65 (Pin_65), J2.66 (Pin_66); no longer J10.P4 (Pin_4)
- net C34: now also J2.67 (Pin_67), J2.68 (Pin_68); no longer J10.P5 (Pin_5)
- net C4: now also J2.7 (Pin_7), J2.8 (Pin_8); no longer J12.P3 (Pin_3)
- net C5: now also J2.10 (Pin_10), J2.9 (Pin_9); no longer J12.P2 (Pin_2)
- net C6: now also J2.11 (Pin_11), J2.12 (Pin_12); no longer J16.B10 (Pin_17)
- net C7: now also J2.13 (Pin_13), J2.14 (Pin_14); no longer J16.B7 (Pin_16)
- net C8: now also J2.15 (Pin_15), J2.16 (Pin_16); no longer J16.B4 (Pin_15)
- net C9: now also J2.17 (Pin_17), J2.18 (Pin_18); no longer J10.P35 (Pin_25)
- removed net +3.3V: J10.P2 (Pin_2), J12.P1 (Pin_1), J16.3V3 (Pin_9)
- net 5V: no longer names the net of J16.5V (Pin_11)
- net 5V: no longer J12.5V (Pin_10)
- net ADC_SW: no longer names the net of J16.B11 (Pin_18)
- net ADC_SW: no longer J10.P34 (Pin_26)
- net ADC_X: no longer names the net of J10.P28 (Pin_32)
- net ADC_Y: no longer names the net of J10.P12 (Pin_12)
- net C35: no longer names the net of J10.P6 (Pin_6)
- net C36: no longer names the net of J10.P7 (Pin_7)
- net C37: no longer names the net of J12.P11 (Pin_13)
- net C38: no longer names the net of J12.P10 (Pin_12)
- net C40: no longer names the net of J10.P15 (Pin_15)
- net C41: no longer names the net of J10.P20 (Pin_19)
- net C45: no longer names the net of J10.P21 (Pin_38)
- net C46: no longer names the net of J10.P22 (Pin_37)
- net C47: no longer names the net of J10.P23 (Pin_36)
- net C48: no longer names the net of J10.P25 (Pin_34)
- removed net CS: J10.P31 (Pin_29), J12.P17 (Pin_19), J16.A12 (Pin_6)
- net CS_1: no longer names the net of J16.A4 (Pin_1)
- net CS_1: no longer J10.P24 (Pin_35)
- removed net DC: J10.P29 (Pin_31), J12.P7 (Pin_7), J16.B9 (Pin_23)
- removed net DONE: J10.P19 (Pin_18), J12.P13 (Pin_15), J16.B23 (Pin_14)
- removed net DRIVE: J10.P18 (Pin_17), J12.P18 (Pin_20), J16.B22 (Pin_13)
- removed net GND: J10.P1 (Pin_1), J10.P40 (Pin_20), J12.P9 (Pin_9), J16.G1 (Pin_10), J16.G2 (Pin_12)
- removed net MISO: J10.P33 (Pin_27), J12.P15 (Pin_17), J16.A15 (Pin_3)
- net MISO2: no longer names the net of J16.B15 (Pin_22)
- net MISO2: no longer J10.P14 (Pin_14)
- removed net MOSI: J10.P39 (Pin_21), J12.P12 (Pin_14), J16.A14 (Pin_4)
- net MOSI2: no longer names the net of J16.B14 (Pin_21)
- net MOSI2: no longer J10.P17 (Pin_16)
- removed net RST1: J10.P30 (Pin_30), J12.P8 (Pin_8), J16.B8 (Pin_24)
- removed net SCK: J10.P32 (Pin_28), J12.P16 (Pin_18), J16.A13 (Pin_5)
- net SCK2: no longer names the net of J10.P13 (Pin_13)
- removed net SCL: J10.P11 (Pin_11), J12.P5 (Pin_5), J16.B13 (Pin_20)
- net SCL2: no longer names the net of J10.P9 (Pin_9)
- removed net SDA: J10.P10 (Pin_10), J12.P6 (Pin_6), J16.B12 (Pin_19)
- net SDA2: no longer names the net of J10.P8 (Pin_8)
- new net A1: J1.1 (Pin_1), J1.2 (Pin_2)
- new net A10: J1.19 (Pin_19), J1.20 (Pin_20)
- new net A11: J1.21 (Pin_21), J1.22 (Pin_22)
- new net A12: J1.23 (Pin_23), J1.24 (Pin_24)
- new net A13: J1.25 (Pin_25), J1.26 (Pin_26)
- new net A14: J1.27 (Pin_27), J1.28 (Pin_28)
- new net A15: J1.29 (Pin_29), J1.30 (Pin_30)
- new net A16: J1.31 (Pin_31), J1.32 (Pin_32)
- new net A17: J1.33 (Pin_33), J1.34 (Pin_34)
- new net A18: J1.35 (Pin_35), J1.36 (Pin_36)
- new net A19: J1.37 (Pin_37), J1.38 (Pin_38)
- new net A2: J1.3 (Pin_3), J1.4 (Pin_4)
- new net A20: J1.39 (Pin_39), J1.40 (Pin_40)
- new net A21: J1.41 (Pin_41), J1.42 (Pin_42)
- new net A22: J1.43 (Pin_43), J1.44 (Pin_44)
- new net A23: J1.45 (Pin_45), J1.46 (Pin_46)
- new net A24: J1.47 (Pin_47), J1.48 (Pin_48)
- new net A25: J1.49 (Pin_49), J1.50 (Pin_50)
- new net A26: J1.51 (Pin_51), J1.52 (Pin_52)
- new net A27: J1.53 (Pin_53), J1.54 (Pin_54)
- new net A28: J1.55 (Pin_55), J1.56 (Pin_56)
- new net A29: J1.57 (Pin_57), J1.58 (Pin_58)
- new net A3: J1.5 (Pin_5), J1.6 (Pin_6)
- new net A30: J1.59 (Pin_59), J1.60 (Pin_60)
- new net A31: J1.61 (Pin_61), J1.62 (Pin_62)
- new net A32: J1.63 (Pin_63), J1.64 (Pin_64)
- new net A33: J1.65 (Pin_65), J1.66 (Pin_66)
- new net A34: J1.67 (Pin_67), J1.68 (Pin_68)
- new net A4: J1.7 (Pin_7), J1.8 (Pin_8)
- new net A5: J1.10 (Pin_10), J1.9 (Pin_9)
- new net A6: J1.11 (Pin_11), J1.12 (Pin_12)
- new net A7: J1.13 (Pin_13), J1.14 (Pin_14)
- new net A8: J1.15 (Pin_15), J1.16 (Pin_16)
- new net A9: J1.17 (Pin_17), J1.18 (Pin_18)
- new net B1: J3.1 (Pin_1), J5.1 (Pin_1), J5.2 (Pin_2), J7.1 (Pin_1), J7.2 (Pin_2)
- new net B10: J3.10 (Pin_10), J5.19 (Pin_19), J5.20 (Pin_20), J7.19 (Pin_19), J7.20 (Pin_20)
- new net B11: J3.11 (Pin_11), J5.21 (Pin_21), J5.22 (Pin_22), J7.21 (Pin_21), J7.22 (Pin_22)
- new net B12: J3.12 (Pin_12), J5.23 (Pin_23), J5.24 (Pin_24), J7.23 (Pin_23), J7.24 (Pin_24)
- new net B13: J3.13 (Pin_13), J5.25 (Pin_25), J5.26 (Pin_26), J7.25 (Pin_25), J7.26 (Pin_26)
- new net B14: J3.14 (Pin_14), J5.27 (Pin_27), J5.28 (Pin_28), J7.27 (Pin_27), J7.28 (Pin_28)
- new net B15: J3.15 (Pin_15), J5.29 (Pin_29), J5.30 (Pin_30), J7.29 (Pin_29), J7.30 (Pin_30)
- new net B16: J3.16 (Pin_16), J5.31 (Pin_31), J5.32 (Pin_32), J7.31 (Pin_31), J7.32 (Pin_32)
- new net B17: J3.17 (Pin_17), J5.33 (Pin_33), J5.34 (Pin_34), J7.33 (Pin_33), J7.34 (Pin_34)
- new net B18: J3.18 (Pin_18), J5.35 (Pin_35), J5.36 (Pin_36), J7.35 (Pin_35), J7.36 (Pin_36)
- new net B19: J3.19 (Pin_19), J5.37 (Pin_37), J5.38 (Pin_38), J7.37 (Pin_37), J7.38 (Pin_38)
- new net B2: J3.2 (Pin_2), J5.3 (Pin_3), J5.4 (Pin_4), J7.3 (Pin_3), J7.4 (Pin_4)
- new net B20: J3.20 (Pin_20), J5.39 (Pin_39), J5.40 (Pin_40), J7.39 (Pin_39), J7.40 (Pin_40)
- new net B21: J3.21 (Pin_21), J5.41 (Pin_41), J5.42 (Pin_42), J7.41 (Pin_41), J7.42 (Pin_42)
- new net B22: J3.22 (Pin_22), J5.43 (Pin_43), J5.44 (Pin_44), J7.43 (Pin_43), J7.44 (Pin_44)
- new net B23: J3.23 (Pin_23), J5.45 (Pin_45), J5.46 (Pin_46), J7.45 (Pin_45), J7.46 (Pin_46)
- new net B24: J3.24 (Pin_24), J5.47 (Pin_47), J5.48 (Pin_48), J7.47 (Pin_47), J7.48 (Pin_48)
- new net B25: J3.25 (Pin_25), J5.49 (Pin_49), J5.50 (Pin_50), J7.49 (Pin_49), J7.50 (Pin_50)
- new net B26: J3.26 (Pin_26), J5.51 (Pin_51), J5.52 (Pin_52), J7.51 (Pin_51), J7.52 (Pin_52)
- new net B27: J3.27 (Pin_27), J5.53 (Pin_53), J5.54 (Pin_54), J7.53 (Pin_53), J7.54 (Pin_54)
- new net B28: J3.28 (Pin_28), J5.55 (Pin_55), J5.56 (Pin_56), J7.55 (Pin_55), J7.56 (Pin_56)
- new net B29: J3.29 (Pin_29), J5.57 (Pin_57), J5.58 (Pin_58), J7.57 (Pin_57), J7.58 (Pin_58)
- new net B3: J3.3 (Pin_3), J5.5 (Pin_5), J5.6 (Pin_6), J7.5 (Pin_5), J7.6 (Pin_6)
- new net B30: J3.30 (Pin_30), J5.59 (Pin_59), J5.60 (Pin_60), J7.59 (Pin_59), J7.60 (Pin_60)
- new net B31: J3.31 (Pin_31), J5.61 (Pin_61), J5.62 (Pin_62), J7.61 (Pin_61), J7.62 (Pin_62)
- new net B32: J3.32 (Pin_32), J5.63 (Pin_63), J5.64 (Pin_64), J7.63 (Pin_63), J7.64 (Pin_64)
- new net B33: J3.33 (Pin_33), J5.65 (Pin_65), J5.66 (Pin_66), J7.65 (Pin_65), J7.66 (Pin_66)
- new net B34: J3.34 (Pin_34), J5.67 (Pin_67), J5.68 (Pin_68), J7.67 (Pin_67), J7.68 (Pin_68)
- new net B4: J3.4 (Pin_4), J5.7 (Pin_7), J5.8 (Pin_8), J7.7 (Pin_7), J7.8 (Pin_8)
- new net B5: J3.5 (Pin_5), J5.10 (Pin_10), J5.9 (Pin_9), J7.10 (Pin_10), J7.9 (Pin_9)
- new net B6: J3.6 (Pin_6), J5.11 (Pin_11), J5.12 (Pin_12), J7.11 (Pin_11), J7.12 (Pin_12)
- new net B7: J3.7 (Pin_7), J5.13 (Pin_13), J5.14 (Pin_14), J7.13 (Pin_13), J7.14 (Pin_14)
- new net B8: J3.8 (Pin_8), J5.15 (Pin_15), J5.16 (Pin_16), J7.15 (Pin_15), J7.16 (Pin_16)
- new net B9: J3.9 (Pin_9), J5.17 (Pin_17), J5.18 (Pin_18), J7.17 (Pin_17), J7.18 (Pin_18)
- new net C1: J2.1 (Pin_1), J2.2 (Pin_2)
- new net C12: J2.23 (Pin_23), J2.24 (Pin_24)
- new net C13: J2.25 (Pin_25), J2.26 (Pin_26)
- new net C14: J2.27 (Pin_27), J2.28 (Pin_28)
- new net C15: J2.29 (Pin_29), J2.30 (Pin_30)
- new net C16: J2.31 (Pin_31), J2.32 (Pin_32)
- new net C17: J2.33 (Pin_33), J2.34 (Pin_34)
- new net C18: J2.35 (Pin_35), J2.36 (Pin_36)
- new net C19: J2.37 (Pin_37), J2.38 (Pin_38)
- new net C2: J2.3 (Pin_3), J2.4 (Pin_4)
- new net C20: J2.39 (Pin_39), J2.40 (Pin_40)
- new net C21: J2.41 (Pin_41), J2.42 (Pin_42)
- new net C22: J2.43 (Pin_43), J2.44 (Pin_44)
- new net C26: J2.51 (Pin_51), J2.52 (Pin_52)
- new net C27: J2.53 (Pin_53), J2.54 (Pin_54)
- new net C28: J2.55 (Pin_55), J2.56 (Pin_56)
- new net D1: J4.1 (Pin_1), J6.1 (Pin_1), J6.2 (Pin_2), J8.1 (Pin_1), J8.2 (Pin_2)
- new net D10: J4.10 (Pin_10), J6.19 (Pin_19), J6.20 (Pin_20), J8.19 (Pin_19), J8.20 (Pin_20)
- new net D11: J4.11 (Pin_11), J6.21 (Pin_21), J6.22 (Pin_22), J8.21 (Pin_21), J8.22 (Pin_22)
- new net D12: J4.12 (Pin_12), J6.23 (Pin_23), J6.24 (Pin_24), J8.23 (Pin_23), J8.24 (Pin_24)
- new net D13: J4.13 (Pin_13), J6.25 (Pin_25), J6.26 (Pin_26), J8.25 (Pin_25), J8.26 (Pin_26)
- new net D14: J4.14 (Pin_14), J6.27 (Pin_27), J6.28 (Pin_28), J8.27 (Pin_27), J8.28 (Pin_28)
- new net D15: J4.15 (Pin_15), J6.29 (Pin_29), J6.30 (Pin_30), J8.29 (Pin_29), J8.30 (Pin_30)
- new net D16: J4.16 (Pin_16), J6.31 (Pin_31), J6.32 (Pin_32), J8.31 (Pin_31), J8.32 (Pin_32)
- new net D17: J4.17 (Pin_17), J6.33 (Pin_33), J6.34 (Pin_34), J8.33 (Pin_33), J8.34 (Pin_34)
- new net D18: J4.18 (Pin_18), J6.35 (Pin_35), J6.36 (Pin_36), J8.35 (Pin_35), J8.36 (Pin_36)
- new net D19: J4.19 (Pin_19), J6.37 (Pin_37), J6.38 (Pin_38), J8.37 (Pin_37), J8.38 (Pin_38)
- new net D2: J4.2 (Pin_2), J6.3 (Pin_3), J6.4 (Pin_4), J8.3 (Pin_3), J8.4 (Pin_4)
- new net D20: J4.20 (Pin_20), J6.39 (Pin_39), J6.40 (Pin_40), J8.39 (Pin_39), J8.40 (Pin_40)
- new net D21: J4.21 (Pin_21), J6.41 (Pin_41), J6.42 (Pin_42), J8.41 (Pin_41), J8.42 (Pin_42)
- new net D22: J4.22 (Pin_22), J6.43 (Pin_43), J6.44 (Pin_44), J8.43 (Pin_43), J8.44 (Pin_44)
- new net D23: J4.23 (Pin_23), J6.45 (Pin_45), J6.46 (Pin_46), J8.45 (Pin_45), J8.46 (Pin_46)
- new net D24: J4.24 (Pin_24), J6.47 (Pin_47), J6.48 (Pin_48), J8.47 (Pin_47), J8.48 (Pin_48)
- new net D25: J4.25 (Pin_25), J6.49 (Pin_49), J6.50 (Pin_50), J8.49 (Pin_49), J8.50 (Pin_50)
- new net D26: J4.26 (Pin_26), J6.51 (Pin_51), J6.52 (Pin_52), J8.51 (Pin_51), J8.52 (Pin_52)
- new net D27: J4.27 (Pin_27), J6.53 (Pin_53), J6.54 (Pin_54), J8.53 (Pin_53), J8.54 (Pin_54)
- new net D28: J4.28 (Pin_28), J6.55 (Pin_55), J6.56 (Pin_56), J8.55 (Pin_55), J8.56 (Pin_56)
- new net D29: J4.29 (Pin_29), J6.57 (Pin_57), J6.58 (Pin_58), J8.57 (Pin_57), J8.58 (Pin_58)
- new net D3: J4.3 (Pin_3), J6.5 (Pin_5), J6.6 (Pin_6), J8.5 (Pin_5), J8.6 (Pin_6)
- new net D30: J4.30 (Pin_30), J6.59 (Pin_59), J6.60 (Pin_60), J8.59 (Pin_59), J8.60 (Pin_60)
- new net D31: J4.31 (Pin_31), J6.61 (Pin_61), J6.62 (Pin_62), J8.61 (Pin_61), J8.62 (Pin_62)
- new net D32: J4.32 (Pin_32), J6.63 (Pin_63), J6.64 (Pin_64), J8.63 (Pin_63), J8.64 (Pin_64)
- new net D33: J4.33 (Pin_33), J6.65 (Pin_65), J6.66 (Pin_66), J8.65 (Pin_65), J8.66 (Pin_66)
- new net D34: J4.34 (Pin_34), J6.67 (Pin_67), J6.68 (Pin_68), J8.67 (Pin_67), J8.68 (Pin_68)
- new net D4: J4.4 (Pin_4), J6.7 (Pin_7), J6.8 (Pin_8), J8.7 (Pin_7), J8.8 (Pin_8)
- new net D5: J4.5 (Pin_5), J6.10 (Pin_10), J6.9 (Pin_9), J8.10 (Pin_10), J8.9 (Pin_9)
- new net D6: J4.6 (Pin_6), J6.11 (Pin_11), J6.12 (Pin_12), J8.11 (Pin_11), J8.12 (Pin_12)
- new net D7: J4.7 (Pin_7), J6.13 (Pin_13), J6.14 (Pin_14), J8.13 (Pin_13), J8.14 (Pin_14)
- new net D8: J4.8 (Pin_8), J6.15 (Pin_15), J6.16 (Pin_16), J8.15 (Pin_15), J8.16 (Pin_16)
- new net D9: J4.9 (Pin_9), J6.17 (Pin_17), J6.18 (Pin_18), J8.17 (Pin_17), J8.18 (Pin_18)
- new net E1: J15.1 (Pin_1), J15.2 (Pin_2)
- new net E10: J15.19 (Pin_19), J15.20 (Pin_20)
- new net E11: J15.21 (Pin_21), J15.22 (Pin_22)
- new net E12: J15.23 (Pin_23), J15.24 (Pin_24)
- new net E13: J15.25 (Pin_25), J15.26 (Pin_26)
- new net E14: J15.27 (Pin_27), J15.28 (Pin_28)
- new net E15: J15.29 (Pin_29), J15.30 (Pin_30)
- new net E16: J15.31 (Pin_31), J15.32 (Pin_32)
- new net E17: J15.33 (Pin_33), J15.34 (Pin_34)
- new net E18: J15.35 (Pin_35), J15.36 (Pin_36)
- new net E19: J15.37 (Pin_37), J15.38 (Pin_38)
- new net E2: J15.3 (Pin_3), J15.4 (Pin_4)
- new net E3: J15.5 (Pin_5), J15.6 (Pin_6)
- new net E4: J15.7 (Pin_7), J15.8 (Pin_8)
- new net E5: J15.10 (Pin_10), J15.9 (Pin_9)
- new net E6: J15.11 (Pin_11), J15.12 (Pin_12)
- new net E7: J15.13 (Pin_13), J15.14 (Pin_14)
- new net E8: J15.15 (Pin_15), J15.16 (Pin_16)
- new net E9: J15.17 (Pin_17), J15.18 (Pin_18)
- new net F1: J18.1 (Pin_1), J18.2 (Pin_2)
- new net F10: J18.19 (Pin_19), J18.20 (Pin_20)
- new net F11: J18.21 (Pin_21), J18.22 (Pin_22)
- new net F12: J18.23 (Pin_23), J18.24 (Pin_24)
- new net F13: J18.25 (Pin_25), J18.26 (Pin_26)
- new net F14: J18.27 (Pin_27), J18.28 (Pin_28)
- new net F15: J18.29 (Pin_29), J18.30 (Pin_30)
- new net F16: J18.31 (Pin_31), J18.32 (Pin_32)
- new net F17: J18.33 (Pin_33), J18.34 (Pin_34)
- new net F18: J18.35 (Pin_35), J18.36 (Pin_36)
- new net F19: J18.37 (Pin_37), J18.38 (Pin_38)
- new net F2: J18.3 (Pin_3), J18.4 (Pin_4)
- new net F3: J18.5 (Pin_5), J18.6 (Pin_6)
- new net F4: J18.7 (Pin_7), J18.8 (Pin_8)
- new net F5: J18.10 (Pin_10), J18.9 (Pin_9)
- new net F6: J18.11 (Pin_11), J18.12 (Pin_12)
- new net F7: J18.13 (Pin_13), J18.14 (Pin_14)
- new net F8: J18.15 (Pin_15), J18.16 (Pin_16)
- new net F9: J18.17 (Pin_17), J18.18 (Pin_18)
- no-connect marks 0 -> 102
Other:
- moved on the sheet: J10, J12, J16
