File: Version1/IOT-Mess-CH_P48/IOT-Mess-P48.kicad_pcb (KiCad board)
At the start: 2 copper layers, 30.1 x 49.5 mm, 30 parts, among them J1 Conn_02x19_Odd_Even, J10 Jumper, J11 Jumper, J12 Jumper, J14 Jumper, J2 Conn_02x19_Odd_Even, J3 Jumper_2, J4 Jumper_2, J5 Conn_01x05_Pin, J6 Jumper, J7 Jumper, K1 Crystal, K32 Crystal, SW11 SW_Push, U10 USB_C_Receptacle_USB2.0_16P, U3 CH32L103C8T6, U6 ME6211C33M5

Commit message: updated.
Parts:
- removed D2: 1N5819WS, Diode_SMD:D_SOD-323
- removed J4: Jumper_2, IOT-Mess-Footprints:Jumpper-triangle
Connections:
- U10 pad A4: Net-(D2-A) -> 5V
- U10 pad A9: Net-(D2-A) -> 5V
- U10 pad B4: Net-(D2-A) -> 5V
- U10 pad B9: Net-(D2-A) -> 5V
Routing:
- net 5V: track 23.6 -> 39.3 mm, vias 1 -> 4
- net Net-(D2-A): track 15.7 -> 0.00 mm, vias 3 -> 0
