File: Version2/PWR-Switching/PWR-Switching.kicad_pcb (KiCad board)
At the start: 2 copper layers, 24.5 x 49.5 mm, 37 parts, among them J1 SUPER CAP, J2 MCU, J3 TP4056, J4 TP4056, J5 Conn_01x12_Pin, J6 MT3608, J7 Conn_02x03_Counter_Clockwise, J8 SOLAR_PWR, Q1 AO3400A, Q2 AO3400A, Q3 AO3400A, Q4 AO3401A, Q5 AO3401A, Q6 AO3401A, Q7 AO3401A, Q9 AO3401A

Commit message: updated.
Parts:
- removed D8: LED, LED_SMD:LED_0603_1608Metric
- removed the R11 at (142.0, 122.4)
- added C1: 100uF, Capacitor_SMD:C_0603_1608Metric, F.Cu at (143.7, 89.5)
- added C3: 10u, Capacitor_SMD:C_0603_1608Metric, F.Cu at (164.2, 85.0)
- added C4: 1u, Capacitor_SMD:C_0603_1608Metric, F.Cu at (142.6, 84.3)
- added D3: LED, LED_SMD:LED_0603_1608Metric, F.Cu at (167.5, 91.5)
- added G***: LOGO, IOT-Mess-Footprints:catIcon8x8, B.Cu at (141.2, 100.9)
- added J10: Jumper_2, IOT-Mess-Footprints:Jumpper-triangle, F.Cu at (159.2, 91.7)
- added J4: Jumper, IOT-Mess-Footprints:Jumper-3_P1.3mm_Open_RoundedPad1.0x1.5mm, B.Cu at (147.3, 84.8)
- added R12: R, Resistor_SMD:R_0603_1608Metric, F.Cu at (167.5, 94.0)
- added U5: ME6211C33M5, Package_TO_SOT_SMD:SOT-23-5, F.Cu at (159.6, 83.5)
- added U6: XC6206PxxxMR, Package_TO_SOT_SMD:SOT-23-3, F.Cu at (159.6, 88.2)
- C5: value 20F -> 1u
- J5: renamed from J7; value Conn_02x03_Counter_Clockwise -> Boost Converter
- L1: value L -> 22uH; footprint Inductor_SMD:L_Taiyo-Yuden_NR-60xx_HandSoldering -> IOT-Mess-Footprints:Inductor_4x4_5x5mm
- moved C5 39.0 mm to (164.2, 87.5), turned to 0 degrees
- moved J5 16.6 mm to (148.8, 88.8)
- moved P3 6.47 mm to (138.3, 90.2), turned to -90 degrees
- moved L1 3.53 mm to (146.4, 78.8), turned to 180 degrees
- moved R11 3.29 mm to (138.3, 87.0), turned to -90 degrees
- moved Q7 1.35 mm to (141.7, 97.1)
- moved R8 1.27 mm to (140.9, 92.6)
- moved R3 1.27 mm to (149.3, 92.7)
- moved Q8 1.27 mm to (144.4, 92.7)
- moved J9 0.56 mm to (129.8, 78.1)
- moved R7 0.29 mm to (138.3, 94.1)
- renumbered D6 to D1, D1 to D2, J8 to J1, J6 to J2, J5 to J3, J3 to J6, J4 to J7, J1 to J8, J2 to J9, D7 to P1, D3 to P2, D5 to P3, Q7 to Q1, Q6 to Q2, Q9 to Q3, Q5 to Q4, Q4 to Q5, Q1 to Q6, Q2 to Q7, Q3 to Q8, R5 to R10, R12 to R11, R3 to R2, R7 to R3, R13 to R4, R10 to R5, R2 to R6, R4 to R7, R6 to R9, D4 to S1
Connections:
- C5 pad 1: Vcc -> Net-(J10-A)
- D1 pad 1: SOLAR_RA -> Net-(D1-K)
- J3 pad 11: P1 -> Net-(D1-K)
- J3 pad 12: SOLAR_RA -> P1
- J5 pad 1: unconnected-(J7-Pin_1-Pad1) -> Net-(J4-C)
- J5 pad 2: unconnected-(J7-Pin_2-Pad2) -> P2
- J5 pad 4: unconnected-(J7-Pin_4-Pad4) (its old number) -> GND
- J5 pad 5: unconnected-(J7-Pin_5-Pad5) (its old number) -> GND
- J5 pad 6: unconnected-(J7-Pin_6-Pad6) -> Net-(J5-Pin_6)
- J6 pad 4: B+ -> unconnected-(J6-Pin_4-Pad4)
- J6 pad 5: B- -> unconnected-(J6-Pin_5-Pad5)
- L1 pad 1: unconnected-(L1-Pad1) -> Net-(J5-Pin_6)
- L1 pad 2: unconnected-(L1-Pad2) -> P1
Routing:
- net P1: track 30.6 -> 73.1 mm, vias 0 -> 1
- net P2: track 8.77 -> 47.9 mm, vias 0 -> 3
- net P2_SW: track 28.2 -> 45.3 mm, vias 1 -> 2
- net Net-(J9-Pin_5): track 2.54 -> 15.3 mm, vias 0 -> 1
- net Net-(J5-Pin_6): track 0.00 -> 9.94 mm
- net SOLAR_RA: track 5.78 -> 0.00 mm
- net Net-(D1-K): track 0.00 -> 4.83 mm
- net Net-(J4-C): track 0.00 -> 3.10 mm, vias 0 -> 1
- net GND: track 2.80 -> 0.00 mm
- net Vcc: track 25.9 -> 23.5 mm, vias 9 -> 8
- net P3_SW: track 57.1 -> 58.9 mm
- net Net-(D8-K): track 1.74 -> 0.00 mm
- net P1_SW: track 46.8 -> 48.4 mm
- net Net-(Q7-D): track 2.45 -> 3.12 mm
- net Net-(J6-Pin_1): track 25.8 -> 25.2 mm
Other:
- board text added: "3S"
- board text added: "Ca"
- board text added: "Cb"
- board text added: "G"
- board text added: "IOT_Mess PWR-Switch V1.2 8/12/25"
- board text added: "S1"
- board text added: "S2"
- board text added: "S2i"
- board text added: "S3"
- board text added: "SS"
- board text added: "Sa"
- board text added: "Sb"
- board text added: "Ta"
- board text added: "Tb"
- board text added: "Vc"
- board text added: "Vcc"

Commit message: did some works.
Parts:
- removed C5: 1u, Capacitor_SMD:C_0603_1608Metric
- removed the D2 at (145.4, 106.1)
- removed Q3: AO3401A, Package_TO_SOT_SMD:SOT-23
- removed Q6, Q7, Q8: AO3400A, Package_TO_SOT_SMD:SOT-23
- removed R12, R9: R, Resistor_SMD:R_0603_1608Metric
- removed the R2 at (146.0, 95.7)
- removed the R4 at (149.2, 110.2)
- removed the R8 at (140.9, 92.6)
- removed the S1 at (150.0, 97.0)
- added C3: 1u, Capacitor_SMD:C_0603_1608Metric, F.Cu at (142.2, 120.6)
- added D1: MBR0520, Diode_SMD:D_SOD-123, B.Cu at (140.8, 109.0)
- added D4: MBR0520, Diode_SMD:D_SOD-123, F.Cu at (138.8, 101.2)
- added EN2: Jumper_2, IOT-Mess-Footprints:Jumpper-triangle, F.Cu at (138.0, 118.8)
- added J8: Switch Inv, Connector_PinSocket_1.00mm:PinSocket_1x02_P1.00mm_Vertical, F.Cu at (144.1, 100.5)
- added P2: LED, LED_SMD:LED_0603_1608Metric, F.Cu at (141.0, 86.6)
- added R6: R, Resistor_SMD:R_0603_1608Metric, F.Cu at (144.0, 86.6)
- added U3: SN74LVC2G14DBV, Package_TO_SOT_SMD:SOT-23-6, F.Cu at (147.9, 96.3)
- added V1: AO3401A, Package_TO_SOT_SMD:SOT-23, F.Cu at (144.8, 104.4)
- added V2: AO3401A, Package_TO_SOT_SMD:SOT-23, F.Cu at (143.6, 90.6)
- C4: value 1u -> 10uF
- D3: value LED -> MBR0520; footprint LED_SMD:LED_0603_1608Metric -> Diode_SMD:D_SOD-123
- J3: value Conn_01x12_Pin -> Conn_01x11_Pin; footprint Connector_PinHeader_2.54mm:PinHeader_1x12_P2.54mm_Vertical -> Connector_PinHeader_2.54mm:PinHeader_1x11_P2.54mm_Vertical
- J9: footprint Connector_PinHeader_2.54mm:PinHeader_1x06_P2.54mm_Vertical -> Connector_PinHeader_2.54mm:PinHeader_1x07_P2.54mm_Vertical
- moved L1 40.7 mm to (147.1, 119.5), turned to 0 degrees
- moved C1 39.3 mm to (142.2, 117.6), turned to -90 degrees
- moved U2 37.2 mm to (139.1, 114.5), turned to 90 degrees
- moved EN1 36.6 mm to (139.0, 120.5), turned to 90 degrees
- moved J4 34.9 mm to (134.8, 120.7), turned to -90 degrees
- moved C4 30.4 mm to (145.4, 114.6), turned to 0 degrees
- moved D3 30.1 mm to (137.8, 96.6), turned to -90 degrees
- moved S1 29.6 mm to (148.7, 81.5)
- moved U1 27.0 mm to (143.2, 109.6)
- moved EN3 26.7 mm to (138.8, 109.0), turned to 180 degrees
- moved C2 25.5 mm to (148.4, 114.6)
- moved R8 20.7 mm to (144.0, 81.2), turned to 180 degrees
- moved P1 18.6 mm to (147.8, 88.6)
- moved J6 18.5 mm to (148.2, 77.0), turned to -90 degrees
- moved R5 18.3 mm to (147.8, 85.6)
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- renumbered C3 to C1, C1 to C2, D1 to D2, P2 to D5, J4 to EN1, J10 to EN3, J5 to J4, J8 to J5, R6 to R2, R7 to R3, R3 to R4, R11 to R7, R10 to R8, Q1 to S1, Q2 to S2, Q4 to SR1, Q5 to SR2, U6 to U1, U5 to U2
Connections:
- C4 pad 1: LDO_EN -> P1
- D2 pad 1: Net-(D1-K) (its old number) -> Net-(D2-K)
- D3 pad 1: GND -> Net-(D3-K)
- D3 pad 2: Net-(D3-A) -> TP_RB
- D5 pad 2: P1_SW -> SW1
- J3 pad 1: Vcc -> TP_RA
- J3 pad 10: CAP_RB -> Vcc
- J3 pad 11: Net-(D1-K) (its old number) -> GND
- J3 pad 2: GND -> TP_RB
- J3 pad 3: P1_SW -> CAP_RA
- J3 pad 4: P2_SW -> CAP_RB
- J3 pad 5: P3_SW -> Net-(D2-K)
- J3 pad 6: SRC_SW- -> P1
- J3 pad 7: TP_RA -> Vcc
- J3 pad 8: TP_RB -> GND
- J3 pad 9: CAP_RA -> unconnected-(J3-Pin_9-Pad9)
- J9 pad 1: Vcc -> +3.3V
- J9 pad 3: SRC_SW- -> unconnected-(J9-Pin_3-Pad3)
- J9 pad 4: P1_SW -> SW1
- J9 pad 5: Net-(J9-Pin_5) -> SW2
- J9 pad 6: P3_SW -> X+
- P1 pad 2: P3_SW -> X+
- P3 pad 2: Net-(J9-Pin_5) -> SW2
- R1 pad 1: Vcc -> GND
- R1 pad 2: /SRC_SW+ -> X+
- R2 pad 2: SRC_SW- -> Y+
- R3 pad 2: P1_SW -> SW1
- R4 pad 1: Vcc -> +3.3V
- R4 pad 2: P2_SW -> SW2
- S1 pad 1: P1_SW -> SW1
- S2 pad 1: P2_SW -> SW2
- SR1 pad 1: SRC_SW- -> Y+
- SR1 pad 2: TP_RB -> Net-(D3-K)
- SR1 pad 3: Vcc -> Net-(SR1-D)
- SR2 pad 1: /SRC_SW+ -> Y-
- SR2 pad 2: CAP_RB -> Net-(D4-K)
- SR2 pad 3: Net-(D2-A) (its old number) -> Net-(SR1-D)
- U2 pad 3: LDO_EN -> Net-(EN2-A)
Routing:
- net P3_SW: track 58.9 -> 0.00 mm, vias 2 -> 0
- net SRC_SW-: track 55.5 -> 0.00 mm, vias 1 -> 0
- net P1_SW: track 48.4 -> 0.00 mm, vias 2 -> 0
- net P2_SW: track 45.3 -> 0.00 mm, vias 2 -> 0
- net Vcc: track 23.5 -> 63.2 mm, vias 8 -> 6
- net SW2: track 0.00 -> 35.6 mm, vias 0 -> 2
- net Y+: track 0.00 -> 28.6 mm, vias 0 -> 3
- net X+: track 0.00 -> 28.6 mm, vias 0 -> 2
- net SW1: track 0.00 -> 23.3 mm, vias 0 -> 2
- net Net-(J6-Pin_1): track 25.2 -> 3.71 mm, vias 1 -> 0
- net Net-(J9-Pin_5): track 15.3 -> 0.00 mm, vias 1 -> 0
- net /SRC_SW+: track 12.6 -> 0.00 mm
- net Net-(D1-K): track 0.00 -> 11.1 mm, vias 0 -> 1
- net Net-(D4-K): track 0.00 -> 10.0 mm, vias 0 -> 2
- net Net-(SR1-D): track 0.00 -> 9.26 mm
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- added copper zone on B.Cu, net +3.3V
- removed copper zone on B.Cu, net Vcc
Other:
- board text added: "3V"
- board text added: "B+"
- board text added: "B-"
- board text added: "IN"
- board text added: "P1"
- board text added: "P2"
- board text added: "PW"
- board text added: "PWi"
- board text added: "X+"
- board text added: "Y+"
- board text added: "x"
- board text removed: "3S"
- board text removed: "S2i"
- board text removed: "S3"
- board text removed: "SS"
- board text removed: "Sa"
- board text removed: "Sb"
- board text removed: "Vcc"
