File: Version2/PWR-Switching/PWR-Switching.kicad_sch (KiCad schematic)
At the start: 41 parts, among them J1 SUPER CAP, J10 Jumper_2, J2 MCU, J3 TP4056, J4 TP4056, J5 Conn_01x12_Pin, J6 MT3608, J7 Boost Converter, J8 SOLAR_PWR, J9 Jumper_2, Q1 AO3400A, Q2 AO3400A, Q3 AO3400A, Q4 AO3401A, Q5 AO3401A, Q6 AO3401A, Q7 AO3401A, Q9 AO3401A

Commit message: updated.
Parts:
- removed D8: LED, LED_SMD:LED_0603_1608Metric, symbol Device:LED
- removed J9: Jumper_2, IOT-Mess-Footprints:Jumpper-triangle, symbol Jumper:Jumper_2_Small_Open
- removed R11: R, Resistor_SMD:R_0603_1608Metric, symbol Device:R
- added C3: 10u, Capacitor_SMD:C_0603_1608Metric, symbol Device:C
- added D3: LED, LED_SMD:LED_0603_1608Metric, symbol Device:LED
- added J4: Jumper, IOT-Mess-Footprints:Jumper-3_P1.3mm_Open_RoundedPad1.0x1.5mm, symbol Jumper:SolderJumper_3_Open
- added R12: R, Resistor_SMD:R_0603_1608Metric, symbol Device:R
- added U5: ME6211C33M5, Package_TO_SOT_SMD:SOT-23-5, symbol Regulator_Linear:ME6211C33M5
- added U6: XC6206PxxxMR, Package_TO_SOT_SMD:SOT-23-3, symbol Regulator_Linear:XC6206PxxxMR
- C4: value 10uF -> 1u
- C5: value 20F -> 1u
- L1: footprint Inductor_SMD:L_Taiyo-Yuden_NR-60xx_HandSoldering -> IOT-Mess-Footprints:Inductor_4x4_5x5mm
- renumbered D6 to D1, D1 to D2, J8 to J1, J6 to J2, J5 to J3, J7 to J5, J3 to J6, J4 to J7, J1 to J8, J2 to J9, D7 to P1, D3 to P2, D5 to P3, Q7 to Q1, Q6 to Q2, Q9 to Q3, Q5 to Q4, Q4 to Q5, Q1 to Q6, Q2 to Q7, Q3 to Q8, R5 to R10, R12 to R11, R3 to R2, R7 to R3, R13 to R4, R10 to R5, R2 to R6, R4 to R7, R6 to R9, D4 to S1
Connections:
- net GND: now also C3.2, D3.1 (K), U5.2 (V_{SS}), U6.1 (GND)
- net P1: now also J3.12 (Pin_12), J4.3 (B); no longer J3.11 (Pin_11)
- net P2: now also J4.1 (A); no longer J10.1 (A)
- net Vcc: now also C3.1, U5.1 (V_{IN}), U6.3 (VI); no longer C5.1
- net at J5.1 (Pin_1): now also J4.2 (C); no longer J10.2 (B)
- net B+: no longer names the net of J6.4 (Pin_4)
- net B-: no longer names the net of J6.5 (Pin_5)
- net SOLAR_RA: no longer names the net of D1.1 (K)
- net SOLAR_RA: now also J3.11 (Pin_11); no longer J3.12 (Pin_12)
- new net: C5.1, J10.1 (A), U5.5 (V_{OUT}), U6.2 (VO)
- new net: D3.2 (A), R12.2
- new net +3.3V: J10.2 (B), R12.1
- new net LDO_EN: C4.1, U5.3 (CE)
- no-connect marks 6 -> 8
Other:
- note added: "B+/B-"
- note added: "SOLAR_RA"
- note added: "SOLAR_RB"
- moved on the sheet: C1, C2, D1, J1, J2, J3, J5, L1

Commit message: did some works.
Parts:
- removed C5: 1u, Capacitor_SMD:C_0603_1608Metric, symbol Device:C
- removed D2: MBR0520, Diode_SMD:D_SOD-123, symbol Diode:MBR0520
- removed D3, S1: LED, LED_SMD:LED_0603_1608Metric, symbol Device:LED
- removed J3: Conn_01x12_Pin, Connector_PinHeader_2.54mm:PinHeader_1x12_P2.54mm_Vertical, symbol Connector:Conn_01x12_Pin
- removed J9: MCU, Connector_PinHeader_2.54mm:PinHeader_1x06_P2.54mm_Vertical, symbol Connector:Conn_01x06_Pin
- removed Q3: AO3401A, Package_TO_SOT_SMD:SOT-23, symbol Transistor_FET:AO3401A
- removed Q6, Q7, Q8: AO3400A, Package_TO_SOT_SMD:SOT-23, symbol Transistor_FET:AO3400A
- removed R12, R2, R4, R8, R9: R, Resistor_SMD:R_0603_1608Metric, symbol Device:R
- added C3: 1u, Capacitor_SMD:C_0603_1608Metric, symbol Device:C
- added D1, D3, D4: MBR0520, Diode_SMD:D_SOD-123, symbol Diode:MBR0520
- added EN2: Jumper_2, IOT-Mess-Footprints:Jumpper-triangle, symbol Jumper:Jumper_2_Small_Open
- added J3: Conn_01x11_Pin, Connector_PinHeader_2.54mm:PinHeader_1x11_P2.54mm_Vertical, symbol Connector:Conn_01x11_Pin
- added J8: Switch Inv, Connector_PinSocket_1.00mm:PinSocket_1x02_P1.00mm_Vertical, symbol Connector:Conn_01x02_Pin
- added J9: MCU, Connector_PinHeader_2.54mm:PinHeader_1x07_P2.54mm_Vertical, symbol Connector:Conn_01x07_Pin
- added P2: LED, LED_SMD:LED_0603_1608Metric, symbol Device:LED
- added R6: R, Resistor_SMD:R_0603_1608Metric, symbol Device:R
- added U3: SN74LVC2G14DBV, Package_TO_SOT_SMD:SOT-23-6, symbol 74xGxx:SN74LVC2G14DBV
- added V1, V2: AO3401A, Package_TO_SOT_SMD:SOT-23, symbol Transistor_FET:AO3401A
- C4: value 1u -> 10uF
- renumbered C3 to C1, C1 to C2, D1 to D2, P2 to D5, J4 to EN1, J10 to EN3, J5 to J4, J8 to J5, R6 to R2, R7 to R3, R3 to R4, R11 to R7, R10 to R8, Q1 to S1, Q2 to S2, Q4 to SR1, Q5 to SR2, U6 to U1, U5 to U2
Connections:
- net P2_SW is gone; now on net SW2: R4.2, S2.1 (G)
- net +3.3V: now also R4.1, J9.1 (Pin_1), U3.5 (V_{CC})
- net CAP_RA: now also J3.3 (Pin_3)
- net CAP_RB: now also D4.2 (A), J3.4 (Pin_4); no longer SR2.2 (S)
- net GND: now also R1.1, C3.2, J3.11 (Pin_11), J3.8 (Pin_8), J9.2 (Pin_2), R6.1, U3.2 (GND)
- net P1: now also J3.6 (Pin_6)
- net P2: now also V1.3 (D)
- net TP_RA: now also J3.1 (Pin_1)
- net TP_RB: now also D3.2 (A), J3.2 (Pin_2); no longer SR1.2 (S)
- net Vcc: now also D1.2 (A), EN2.2 (B), J3.10 (Pin_10), J3.7 (Pin_7), V1.2 (S), V2.3 (D); no longer R1.1, R4.1, SR1.3 (D)
- net SW2: now reaches P3.2 (A)
- net SW2: now also J9.5 (Pin_5)
- net at EN3.1 (A), U1.2 (VO), U2.5 (V_{OUT}): now also D1.1 (K)
- net at SR2.3 (D): now also SR1.3 (D), V2.2 (S)
- net at D2.1 (K): now also J3.5 (Pin_5)
- net LDO_EN: no longer names the net of U2.3 (CE)
- net LDO_EN: now also C3.1, EN2.1 (A); no longer C4.1
- net P1_SW renamed SW1
- net SW1: now also J9.4 (Pin_4)
- net P3_SW renamed X+
- net X+: now also R1.2, J9.6 (Pin_6), U3.1 (1A), V2.1 (G)
- net SRC_SW+ renamed Y-
- net Y-: now also J8.2 (Pin_2), U3.4 (2Y); no longer R1.2
- net SRC_SW- renamed Y+
- net Y+: now also J9.7 (Pin_7), P2.2 (A), U3.3 (2A)
- new net: D3.1 (K), SR1.2 (S)
- new net: D4.1 (K), SR2.2 (S)
- new net: P2.1 (K), R6.2
- new net X-: J8.1 (Pin_1), U3.6 (1Y), V1.1 (G)
- no-connect marks 8 -> 10
Other:
- note added: "LDO Circuit"
- note added: "P1: Solar Output P2: Boost Converter Output"
- note added: "PFET (INV - OFF)"
- note added: "Power Path Circuit"
- note added: "SA controls Switch between Direct P2 OR from Lipo/Cap Circuits"
- note added: "SB controls Switch between Lipo OR Cap Circuit"
- note removed: "Direct Source Circuit"
- note removed: "NFET (PD - OFF)"
- moved on the sheet: C1, C2, C4, D2, D5, EN1, EN3, J1, J2, J4, J5, J6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
