File: Version2/LED-Matrix/LED-Matrix.kicad_sch (KiCad schematic)
At the start: 345 parts, among them U1 74HC595, U2 74HC595, U3 74HC595

Commit message: updates.
Parts:
- added J1: Conn_02x19_Odd_Even, Connector_PinHeader_2.54mm:PinHeader_2x18_P2.54mm_Vertical, symbol Connector_Generic:Conn_02x19_Odd_Even
Connections:
- net A_0: now also J1.1 (Pin_1)
- net A_1: now also J1.3 (Pin_3)
- net A_2: now also J1.5 (Pin_5)
- net A_3: now also J1.7 (Pin_7)
- net A_4: now also J1.9 (Pin_9)
- net A_5: now also J1.11 (Pin_11)
- net A_6: now also J1.13 (Pin_13)
- net A_7: now also J1.15 (Pin_15)
- net B_0: now also J1.2 (Pin_2)
- net B_1: now also J1.4 (Pin_4)
- net B_2: now also J1.6 (Pin_6)
- net B_3: now also J1.8 (Pin_8)
- net B_4: now also J1.10 (Pin_10)
- net B_5: now also J1.12 (Pin_12)
- net B_6: now also J1.14 (Pin_14)
- net B_7: now also J1.16 (Pin_16)
- net C_0: now also J1.24 (Pin_24)
- net C_1: now also J1.26 (Pin_26)
- net C_2: now also J1.28 (Pin_28)
- net C_3: now also J1.30 (Pin_30)
- net C_4: now also J1.32 (Pin_32)
- net C_5: now also J1.34 (Pin_34)
- net C_6: now also J1.36 (Pin_36)
- net C_7: now also J1.38 (Pin_38)
- net CLCK: now reaches U3.11 (SRCLK)
- net CLCK: now also U1.11 (SRCLK), U2.11 (SRCLK)
- net LATCH: now reaches U3.12 (RCLK)
- net LATCH: now also U1.12 (RCLK), U2.12 (RCLK)
- net EN_C: now reaches U3.13 (~{OE})
- net DATA: now reaches U3.14 (SER)
- net DATA: now also U1.14 (SER), U2.14 (SER)
- net VCC: now reaches U3.16 (VCC)
- net VCC: now also U1.16 (VCC), U2.16 (VCC)
- net GND: now reaches U3.8 (GND)
- net GND: now also U1.8 (GND), U2.8 (GND)
- net EN_B: now reaches U2.13 (~{OE})
- net EN_A: now reaches U1.13 (~{OE})
- no-connect marks 0 -> 20
Other:
- moved on the sheet: D1, D10, D100, D101, D102, D103, D104, D105, D106, D107, D108, D109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

Commit message: did some works.
Parts:
- removed U2, U3: 74HC595, symbol 74xx:74HC595
Connections:
- no-connect marks 20 -> 16
Other:
- moved on the sheet: U1

Commit message: update.
Parts:
- removed U1: 74HC595, symbol 74xx:74HC595
- J1: footprint Connector_PinHeader_2.54mm:PinHeader_2x18_P2.54mm_Vertical -> Connector_PinHeader_2.54mm:PinHeader_2x19_P2.54mm_Vertical
Connections:
- net C_0: now also J1.23 (Pin_23)
- net C_1: now also J1.25 (Pin_25)
- net C_2: now also J1.27 (Pin_27)
- net C_3: now also J1.29 (Pin_29)
- net C_4: now also J1.31 (Pin_31)
- net C_5: now also J1.33 (Pin_33)
- net C_6: now also J1.35 (Pin_35)
- net C_7: now also J1.37 (Pin_37)
- net B_0 renamed R_0
- net B_1 renamed R_1
- net B_2 renamed R_2
- net B_3 renamed R_3
- net B_4 renamed R_4
- net B_5 renamed R_5
- net B_6 renamed R_6
- net B_7 renamed R_7
- no-connect marks 16 -> 6
Other:
- moved on the sheet: J1
