File: Version2/LED-Matrix/LED-Matrix.kicad_pcb (KiCad board)
At the start: 2 copper layers, 342 parts

Commit message: updates.
Parts:
- added G***: LOGO, IOT-Mess-Footprints:catIcon8x8, B.Cu at (154.0, 134.4)
- added J1: Conn_02x19_Odd_Even, Connector_PinHeader_2.54mm:PinHeader_2x18_P2.54mm_Vertical, F.Cu at (175.7, 49.0)
- moved D71 0.46 mm to (134.9, 69.8)
- moved D72 0.46 mm to (132.3, 69.8)
- moved D55 0.46 mm to (176.2, 69.8)
- moved D56 0.46 mm to (173.6, 69.8)
- moved D57 0.46 mm to (171.0, 69.8)
- moved D58 0.46 mm to (168.4, 69.8)
- moved D59 0.46 mm to (165.8, 69.8)
- moved D60 0.46 mm to (163.2, 69.8)
- moved D61 0.46 mm to (160.6, 69.8)
- moved D62 0.46 mm to (158.0, 69.8)
- moved D63 0.46 mm to (155.5, 69.8)
- moved D64 0.46 mm to (152.9, 69.8)
- moved D65 0.46 mm to (150.3, 69.8)
- moved D66 0.46 mm to (147.7, 69.8)
- moved D67 0.46 mm to (145.1, 69.8)
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Routing:
- net A_1: track 75.5 -> 147.7 mm, vias 0 -> 2
- net A_5: track 229.6 -> 295.9 mm, vias 12 -> 17
- net A_2: track 115.7 -> 168.1 mm, vias 2 -> 4
- net C_4: track 188.3 -> 240.4 mm, vias 12 -> 14
- net C_6: track 252.2 -> 303.8 mm
- net A_4: track 168.7 -> 217.0 mm
- net C_5: track 225.3 -> 273.6 mm
- net B_3: track 155.0 -> 198.5 mm, vias 8 -> 10
- net C_7: track 265.0 -> 308.1 mm, vias 15 -> 14
- net A_6: track 207.3 -> 247.9 mm, vias 13 -> 17
- net B_4: track 209.4 -> 247.9 mm, vias 9 -> 10
- net B_6: track 223.7 -> 257.8 mm
- net A_7: track 189.0 -> 220.3 mm
- net B_7: track 230.6 -> 257.7 mm, vias 14 -> 18
- net C_3: track 160.5 -> 184.6 mm, vias 10 -> 11
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Other:
- board outline added: 49.5 x 100 mm
- board text added: "A0"
- board text added: "A1"
- board text added: "A2"
- board text added: "A3"
- board text added: "A4"
- board text added: "A5"
- board text added: "A6"
- board text added: "A7"
- board text added: "B0"
- board text added: "B1"
- board text added: "B2"
- board text added: "B3"
- board text added: "B4"
- board text added: "B5"
- board text added: "B6"
- board text added: "B7"
- board text added: "C0"
- board text added: "C1"
- board text added: "C2"
- board text added: "C3"
- board text added: "C4"
- board text added: "C5"
- board text added: "C6"
- board text added: "IOT_Mess Charlieplexing LEDs V1.2 8/12/25"
- board text added: "x"

Commit message: update.
Parts:
- J1: footprint Connector_PinHeader_2.54mm:PinHeader_2x18_P2.54mm_Vertical -> Connector_PinHeader_2.54mm:PinHeader_2x19_P2.54mm_Vertical
- moved J1 1.24 mm to (176.9, 49.0)
Connections:
- net B_0 renamed R_0
- net B_1 renamed R_1
- net B_2 renamed R_2
- net B_3 renamed R_3
- net B_4 renamed R_4
- net B_5 renamed R_5
- net B_6 renamed R_6
- net B_7 renamed R_7
- J1 pad 23: unconnected-(J1-Pin_23-Pad23) -> C_0
- J1 pad 25: unconnected-(J1-Pin_25-Pad25) -> C_1
- J1 pad 27: unconnected-(J1-Pin_27-Pad27) -> C_2
- J1 pad 29: unconnected-(J1-Pin_29-Pad29) -> C_3
- J1 pad 31: unconnected-(J1-Pin_31-Pad31) -> C_4
- J1 pad 33: unconnected-(J1-Pin_33-Pad33) -> C_5
- J1 pad 35: unconnected-(J1-Pin_35-Pad35) -> C_6
Routing:
- net A_1: track 147.7 -> 109.0 mm, vias 2 -> 1
- net C_7: track 308.1 -> 337.1 mm, vias 14 -> 15
- net A_2: track 168.1 -> 161.2 mm
- net C_6: track 303.8 -> 306.9 mm
- net C_5: track 273.6 -> 276.7 mm
- net C_3: track 184.6 -> 187.5 mm
- net R_3: track 198.5 -> 196.1 mm, vias 10 -> 9
- net C_0: track 113.0 -> 115.1 mm
- net C_2: track 181.1 -> 183.2 mm
- net A_5: track 295.9 -> 294.3 mm, vias 17 -> 16
- net A_4: track 217.0 -> 218.7 mm
- net C_4: track 240.4 -> 238.8 mm
- net R_2: track 155.4 -> 156.7 mm
- net C_1: track 146.7 -> 147.7 mm
- net R_1: track 116.3 -> 117.2 mm
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Other:
- board text added: "C7"
- board text added: "R0"
- board text added: "R1"
- board text added: "R2"
- board text added: "R3"
- board text added: "R4"
- board text added: "R5"
- board text added: "R6"
- board text added: "R7"
- board text removed: "B0"
- board text removed: "B1"
- board text removed: "B2"
- board text removed: "B3"
- board text removed: "B4"
- board text removed: "B5"
- board text removed: "B6"
- board text removed: "B7"

Commit message: update stuff.
Parts:
- moved G*** 1.79 mm to (153.8, 132.6)
Other:
- board text added: "IOT_Mess Charlieplexing2 V2.0 8/19/25"
- board text removed: "IOT_Mess Charlieplexing LEDs V1.2 8/12/25"
Changed lines of the file:
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@@
 	(footprint "IOT-Mess-Footprints:catIcon8x8"
 		(layer "B.Cu")
-		(at 153.956458 134.382904 180)
+		(at 153.8 132.6 180)
 		(property "Reference" "G***"
 			(at 0 0 0)
@@
 		)
 	)
-	(gr_text "IOT_Mess Charlieplexing LEDs\nV1.2 8/12/25"
-		(at 152.980001 143.275 0)
+	(gr_text "IOT_Mess Charlieplexing2\nV2.0 8/19/25"
+		(at 152.980001 141.492096 0)
 		(layer "B.SilkS")
 		(effects
