File: Version1/IOT-Mess-ESP32/IOT-Mess-ESP32.kicad_pcb (KiCad board)
At the start: 2 copper layers, 29 x 49.5 mm, 27 parts, among them J1 Conn_01x19_Pin, J10 Jumper, J2 Conn_01x19_Pin, J3 Jumper_2, J4 Jumper_2, J5 Conn_01x06_Pin, J7 Jumper, J8 Jumper, J9 Jumper, SW10 SW_Push, SW11 SW_Push, U10 USB_C_Receptacle_USB2.0_16P, U2 ESP32-C6-MINI-1, U4 ESP32-S2-WROVER, U6 ME6211C33M5

Commit message: updated.
Parts:
- removed D2: 1N5819WS, Diode_SMD:D_SOD-323
- removed J4: Jumper_2, IOT-Mess-Footprints:Jumpper-triangle
- added U3: XC6206PxxxMR, Package_TO_SOT_SMD:SOT-23-3, F.Cu at (104.9, 114.0)
- moved J3 7.83 mm to (101.8, 112.7)
- moved G*** 5.16 mm to (108.7, 112.4)
- moved C9 3.17 mm to (114.4, 116.2), turned to 0 degrees
- moved R16 3.00 mm to (111.4, 116.2), turned to 180 degrees
- moved C4 2.15 mm to (104.9, 110.6), turned to 180 degrees
- moved SW11 1.22 mm to (97.7, 122.0)
- moved SW10 1.11 mm to (114.1, 121.9)
- moved D1 0.24 mm to (100.3, 113.5)
- moved C10 0.23 mm to (100.3, 116.2)
- turned J10 to 90 degrees
Connections:
- C4 pad 1: P2 -> Net-(J3-A)
- U10 pad A4: Net-(D2-K) -> 5V
- U10 pad A9: Net-(D2-K) -> 5V
- U10 pad B4: Net-(D2-K) -> 5V
- U10 pad B9: Net-(D2-K) -> 5V
Routing:
- net P2: track 92.0 -> 35.3 mm, vias 9 -> 3
- net Net-(D2-K): track 17.1 -> 0.00 mm, vias 3 -> 0
- net Net-(J3-A): track 3.65 -> 13.6 mm
- net 5V: track 21.5 -> 30.8 mm, vias 3 -> 2
- net BOOT: track 53.1 -> 60.9 mm
- net P15: track 40.7 -> 33.0 mm
- net P18: track 48.2 -> 43.3 mm
- net P31: track 30.7 -> 35.1 mm
- net P12: track 27.2 -> 23.1 mm
- net P20: track 48.0 -> 44.3 mm
- net P1: track 27.5 -> 24.1 mm
- net P29: track 31.9 -> 28.7 mm, vias 0 -> 2
- net P30: track 34.1 -> 37.1 mm, vias 1 -> 3
- net P35: track 16.2 -> 13.4 mm, vias 0 -> 1
- net P28: track 34.4 -> 37.1 mm
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- added copper zone on B.Cu, net P2
- removed copper zone on B.Cu, net P1
Other:
- board size 29 x 49.5 mm -> 29.6 x 49.5 mm

Commit message: did some works.
Other:
- board text added: "3V"
- board text added: "x"
- board text removed: "3.3V"
- board text removed: "LED"
Changed lines of the file:
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@@
 		(tags "LED")
 		(property "Reference" "D1"
-			(at 0 -1.43 0)
+			(at -0.9 1.3 0)
 			(layer "F.SilkS")
 			(effects
@@
 		(tags "capacitor")
 		(property "Reference" "C10"
-			(at 0 1.344998 0)
+			(at 0.7 1.444998 0)
 			(layer "F.SilkS")
 			(effects
@@
 		(tags "solder jumper open")
 		(property "Reference" "J10"
-			(at -3.494561 0 90)
+			(at 2.994561 -0.018756 90)
 			(layer "F.SilkS")
 			(effects
@@
 		(tags "capacitor")
 		(property "Reference" "C4"
-			(at 0 -1.43 0)
+			(at 0 1.2 0)
 			(layer "F.SilkS")
 			(effects
@@
 		(tags "resistor")
 		(property "Reference" "R15"
-			(at 0 -1.43 0)
+			(at -0.461 -1.43 0)
 			(layer "F.SilkS")
 			(effects
@@
 		(tags "SOT TO_SOT_SMD")
 		(property "Reference" "U6"
-			(at 0 -2.4 0)
+			(at 0 2.540002 0)
 			(layer "F.SilkS")
 			(effects
@@
 		(tags "resistor")
 		(property "Reference" "R5"
-			(at 0 1.200003 0)
+			(at 1.061082 -1.3 0)
 			(layer "F.SilkS")
 			(effects
@@
 		(tags "SOT TO_SOT_SMD")
 		(property "Reference" "U3"
-			(at 0 -2.4 90)
+			(at 2.4 -0.1 180)
 			(layer "F.SilkS")
 			(effects
@@
 		)
 	)
-	(gr_text "5V"
-		(at 112.340769 104.865769 90)
-		(layer "F.SilkS")
-		(effects
-			(font
-				(size 1 1)
-				(thickness 0.15)
-			)
-		)
-	)
 	(gr_text "3"
 		(at 95.466377 83.395692 0)
@@
 		)
 	)
-	(gr_text "3.3V"
-		(at 107.290769 105.435769 90)
+	(gr_text "5V"
+		(at 112.2 105.2 90)
 		(layer "F.SilkS")
 		(effects
@@
 		)
 	)
-	(gr_text "D+"
-		(at 104.600769 104.955769 90)
-		(layer "F.SilkS")
-		(effects
-			(font
-				(size 1 1)
-				(thickness 0.15)
-			)
-		)
-	)
 	(gr_text "33"
 		(at 116.435 96.357928 0)
@@
 		)
 	)
-	(gr_text "LED"
-		(at 99.650769 105.175769 90)
+	(gr_text "x"
+		(at 99.479998 105.230001 90)
 		(layer "F.SilkS")
 		(effects
@@
 		)
 	)
-	(gr_text "36"
-		(at 116.445 88.767928 0)
+	(gr_text "D+"
+		(at 104.56 105.2 90)
 		(layer "F.SilkS")
 		(effects
@@
 		)
 	)
-	(gr_text "18"
-		(at 95.466377 119.055692 0)
+	(gr_text "36"
+		(at 116.445 88.767928 0)
 		(layer "F.SilkS")
 		(effects
@@
 		)
 	)
-	(gr_text "14"
-		(at 95.466378 111.38569 0)
+	(gr_text "3V"
+		(at 107.139999 105.200001 90)
 		(layer "F.SilkS")
 		(effects
@@
 		)
 	)
-	(gr_text "39"
-		(at 116.445 81.177929 0)
+	(gr_text "18"
+		(at 95.466377 119.055692 0)
 		(layer "F.SilkS")
 		(effects
@@
 		)
 	)
-	(gr_text "35"
-		(at 116.445001 91.317929 0)
+	(gr_text "14"
+		(at 95.466378 111.38569 0)
 		(layer "F.SilkS")
 		(effects
@@
 		)
 	)
-	(gr_text "G"
-		(at 109.810769 105.365769 90)
+	(gr_text "39"
+		(at 116.445 81.177929 0)
 		(layer "F.SilkS")
 		(effects
@@
 		)
 	)
-	(gr_text "D-"
-		(at 102.120769 104.955769 90)
+	(gr_text "35"
+		(at 116.445001 91.317929 0)
 		(layer "F.SilkS")
 		(effects
@@
 		)
 	)
+	(gr_text "G"
+		(at 109.649999 105.200001 90)
+		(layer "F.SilkS")
+		(effects
+			(font
+				(size 1 1)
+				(thickness 0.15)
+			)
+		)
+	)
 	(gr_text "10"
 		(at 95.466377 101.245691 0)
@@
 		)
 	)
+	(gr_text "D-"
+		(at 102.06 105.2 90)
+		(layer "F.SilkS")
+		(effects
+			(font
+				(size 1 1)
+				(thickness 0.15)
+			)
+		)
+	)
 	(gr_text "27"
 		(at 116.445001 111.667929 0)
@@
 		)
 	)
-	(gr_text "G"
-		(at 109.78 105.07 90)
-		(layer "B.SilkS")
-		(effects
-			(font
-				(size 1 1)
-				(thickness 0.15)
-			)
-			(justify mirror)
-		)
-	)
 	(gr_text "29"
 		(at 116.471465 106.607127 0)
@@
 		)
 	)
-	(gr_text "D+"
-		(at 104.57 105.48 90)
-		(layer "B.SilkS")
-		(effects
-			(font
-				(size 1 1)
-				(thickness 0.15)
-			)
-			(justify mirror)
-		)
-	)
 	(gr_text "10"
 		(at 95.400622 101.236234 0)
@@
 		)
 	)
-	(gr_text "D-"
-		(at 102.09 105.48 90)
+	(gr_text "30"
+		(at 116.471465 104.047128 0)
 		(layer "B.SilkS")
 		(effects
@@
 		)
 	)
-	(gr_text "30"
-		(at 116.471465 104.047128 0)
+	(gr_text "11"
+		(at 95.400622 103.756234 0)
 		(layer "B.SilkS")
 		(effects
@@
 		)
 	)
-	(gr_text "11"
-		(at 95.400622 103.756234 0)
+	(gr_text "22"
+		(at 116.481464 121.827126 0)
 		(layer "B.SilkS")
 		(effects
@@
 		)
 	)
-	(gr_text "22"
-		(at 116.481464 121.827126 0)
+	(gr_text "G"
+		(at 109.709999 105.199999 90)
 		(layer "B.SilkS")
 		(effects
@@
 		)
 	)
-	(gr_text "LED"
-		(at 99.62 105.26 90)
-		(layer "B.SilkS")
-		(effects
-			(font
-				(size 1 1)
-				(thickness 0.15)
-			)
-			(justify mirror)
-		)
-	)
 	(gr_text "7"
 		(at 95.410622 93.516234 0)
@@
 	)
 	(gr_text "5V"
-		(at 112.31 105.57 90)
+		(at 112.26 105.2 90)
 		(layer "B.SilkS")
 		(effects
@@
 		)
 	)
-	(gr_text "3.3V"
-		(at 107.26 105 90)
+	(gr_text "36"
+		(at 116.471465 88.767127 0)
 		(layer "B.SilkS")
 		(effects
@@
 		)
 	)
-	(gr_text "36"
-		(at 116.471465 88.767127 0)
+	(gr_text "3V"
+		(at 107.199999 105.199999 90)
 		(layer "B.SilkS")
 		(effects
@@
 		)
 	)
+	(gr_text "D-"
+		(at 102.12 105.2 90)
+		(layer "B.SilkS")
+		(effects
+			(font
+				(size 1 1)
+				(thickness 0.15)
+			)
+			(justify mirror)
+		)
+	)
 	(gr_text "12"
 		(at 95.40062 106.316233 0)
@@
 		)
 	)
+	(gr_text "x"
+		(at 99.539998 105.169999 90)
+		(layer "B.SilkS")
+		(effects
+			(font
+				(size 1 1)
+				(thickness 0.15)
+			)
+			(justify mirror)
+		)
+	)
 	(gr_text "13"
 		(at 95.40062 108.826233 0)
@@
 		)
 	)
+	(gr_text "D+"
+		(at 104.62 105.2 90)
+		(layer "B.SilkS")
+		(effects
+			(font
+				(size 1 1)
+				(thickness 0.15)
+			)
+			(justify mirror)
+		)
+	)
 	(gr_text "IOT_Mess ESP32 V1.0\n7/5/25"
 		(at 106 119.2 0)
@@
 	)
 	(group ""
+		(members "1ea30b50-2980-45f1-b051-4b9d54d956a7" "39cf85b8-40f8-46f7-956c-832bae126d42"
+			"46f34ba9-3392-439c-bbc6-31a28c2b23b0" "4a7c8223-f58b-4f18-a575-b580d50ff448"
+			"cedd495f-5860-4f75-b5fe-8695a7adcf97" "dadea013-0c36-4721-bd72-5a7f9982ef19"
+		)
+	)
+	(group ""
 		(members "09be2f69-bed6-4867-ad83-8910105b6e4f" "1fa842ac-02ef-4382-8eeb-2fb6086d3366"
 			"2bd700bd-fe3d-46cb-ad39-a7e9ac78eade" "3a25d167-2cd8-4ddc-8c46-9fa56e3ed10a"
@@
 		)
 	)
+	(group ""
+		(members "5b4c63f5-c40f-42db-a841-5963af39c4ff" "c7b3732d-944f-47c8-a280-131bc4eb056b"
+			"c97afa2f-5036-4f78-acae-55ed2c447baf" "d48d7c9a-b455-40b9-88b4-dac4d795522e"
+			"f2d9cb90-ecb7-4537-a874-c2e14076d50a" "fcd92fdf-6320-4904-8369-590e0c0a0744"
+		)
+	)

Commit message: update stuff.
Connections:
- C4 pad 1: Net-(J3-A) -> P2
Routing:
- net P2: track 35.3 -> 39.1 mm
- net Net-(J3-A): track 13.6 -> 9.87 mm
Other:
- board size 29.6 x 49.5 mm -> 29.6 x 49 mm
- board text added: "IOT_Mess ESP32 V2.0 8/19/25"
- board text removed: "IOT_Mess ESP32 V1.0 7/5/25"
