File: Version1/IOT-Mess-ESP32/IOT-Mess-ESP32.kicad_sch (KiCad schematic)
At the start: 26 parts, among them J1 Conn_01x19_Pin, J10 Jumper, J2 Conn_01x19_Pin, J3 Jumper_2, J4 Jumper_2, J5 Conn_01x06_Pin, J7 Jumper, J8 Jumper, J9 Jumper, SW10 SW_Push, SW11 SW_Push, U10 USB_C_Receptacle_USB2.0_16P, U2 ESP32-C6-MINI-1, U4 ESP32-S2-WROVER, U6 ME6211C33M5

Commit message: updated.
Parts:
- removed D2: 1N5819WS, Diode_SMD:D_SOD-323, symbol Diode:1N5819WS
- removed J4: Jumper_2, IOT-Mess-Footprints:Jumpper-triangle, symbol Jumper:Jumper_2_Small_Open
- added U3: XC6206PxxxMR, Package_TO_SOT_SMD:SOT-23-3, symbol Regulator_Linear:XC6206PxxxMR
Connections:
- net +3.3V: no longer C4.1
- net 5V: now also U10.A4 (VBUS), U10.A9 (VBUS), U10.B4 (VBUS), U10.B9 (VBUS), U3.3 (VI)
- net GND: now also U3.1 (GND)
- net at J3.1 (A), U6.5 (V_{OUT}): now also C4.1, U3.2 (VO)
Other:
- moved on the sheet: C2, C4, C5, D1, J3, R5, U10, U6

Commit message: update stuff.
Connections:
- net +3.3V: now also C4.1
- net at J3.1 (A), U3.2 (VO), U6.5 (V_{OUT}): no longer C4.1
Other:
- moved on the sheet: C4
Changed lines of the file:
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@@
 	)
 	(junction
+		(at 185.42 222.25)
+		(diameter 0)
+		(color 0 0 0 0)
+	)
+	(junction
 		(at 109.22 203.2)
 		(diameter 0)
@@
 	(wire
 		(pts
-			(xy 153.67 222.25) (xy 153.67 226.06)
+			(xy 185.42 222.25) (xy 185.42 226.06)
 		)
 		(stroke
@@
 	(symbol
 		(lib_id "Device:C")
-		(at 153.67 229.87 0)
+		(at 185.42 229.87 0)
 		(unit 1)
 		(exclude_from_sim no)
@@
 		(fields_autoplaced yes)
 		(property "Reference" "C4"
-			(at 156.845 228.6 0)
+			(at 188.595 228.6 0)
 			(effects
 				(font
@@
 		)
 		(property "Value" "1u"
-			(at 156.845 231.14 0)
+			(at 188.595 231.14 0)
 			(effects
 				(font
@@
 		)
 		(property "Footprint" "Capacitor_SMD:C_0603_1608Metric"
-			(at 154.6352 233.68 0)
+			(at 186.3852 233.68 0)
 			(effects
 				(font
@@
 		)
 		(property "Datasheet" "~"
-			(at 153.67 229.87 0)
+			(at 185.42 229.87 0)
 			(effects
 				(font
@@
 		)
 		(property "Description" ""
-			(at 153.67 229.87 0)
+			(at 185.42 229.87 0)
 			(effects
 				(font
@@
 		(lib_name "GND_1")
 		(lib_id "power:GND")
-		(at 153.67 233.68 0)
+		(at 185.42 233.68 0)
 		(unit 1)
 		(exclude_from_sim no)
@@
 		(fields_autoplaced yes)
 		(property "Reference" "#PWR015"
-			(at 153.67 240.03 0)
+			(at 185.42 240.03 0)
 			(effects
 				(font
@@
 		)
 		(property "Value" "GND"
-			(at 153.67 238.76 0)
+			(at 185.42 238.76 0)
 			(effects
 				(font
@@
 		)
 		(property "Footprint" ""
-			(at 153.67 233.68 0)
+			(at 185.42 233.68 0)
 			(effects
 				(font
@@
 		)
 		(property "Datasheet" ""
-			(at 153.67 233.68 0)
+			(at 185.42 233.68 0)
 			(effects
 				(font
@@
 		)
 		(property "Description" "Power symbol creates a global label with name \"GND\" , ground"
-			(at 153.67 233.68 0)
+			(at 185.42 233.68 0)
 			(effects
 				(font
