File: Version1/IOT-Mess-ESP_P16/IOT-Mess-ESP_P16.kicad_pcb (KiCad board)
At the start: 2 copper layers, 29.4 x 32.4 mm, 24 parts, among them J1 Conn_01x10_Pin, J2 Conn_01x09_Pin, J3 Jumper_2, J4 Jumper_2, J5 Jumper_2, J6 Jumper_2, SW10 SW_Push, SW11 SW_Push, U1 ESP-12F, U10 USB_C_Receptacle_USB2.0_16P, U5 ESP32-C3-WROOM-02, U6 ME6211C33M5

Commit message: updated.
Parts:
- removed D2: 1N5819WS, Diode_SMD:D_SOD-323
- added U2: XC6206PxxxMR, Package_TO_SOT_SMD:SOT-23-3, B.Cu at (128.1, 103.4)
- J4: moved to F.Cu
- moved J3 12.2 mm to (128.0, 99.7), turned to 45 degrees
- moved J4 9.68 mm to (135.4, 98.7), turned to 180 degrees
- moved C4 2.57 mm to (131.4, 98.5), turned to 0 degrees
- moved C2 1.69 mm to (139.2, 103.2)
Connections:
- C4 pad 1: P1 -> Net-(J3-B)
- C5 pad 1: 5V -> Net-(J4-B)
- J4 pad 1: Net-(D2-A) -> 5V
- J4 pad 2: 5V -> Net-(J4-B)
- U10 pad A4: Net-(D2-A) -> 5V
- U10 pad A9: Net-(D2-A) -> 5V
- U10 pad B4: Net-(D2-A) -> 5V
- U10 pad B9: Net-(D2-A) -> 5V
- U6 pad 3: 5V -> Net-(J4-B)
Routing:
- net P1: track 81.2 -> 16.3 mm, vias 4 -> 5
- net Net-(D2-A): track 21.5 -> 0.00 mm, vias 3 -> 0
- net P6: track 18.0 -> 11.4 mm, vias 0 -> 1
- net Net-(J4-B): track 0.00 -> 6.17 mm
- net 5V: track 30.3 -> 35.9 mm, vias 1 -> 2
- net P12: track 18.6 -> 13.5 mm
- net P9: track 3.05 -> 6.52 mm, vias 1 -> 2
- net Net-(J3-B): track 8.13 -> 11.0 mm, vias 0 -> 1
- net D+: track 17.7 -> 15.7 mm
- net D-: track 18.2 -> 16.7 mm
- net P2: track 60.2 -> 59.2 mm
- net BOOT: track 40.8 -> 41.4 mm
- added copper zone on B.Cu, net P1
- removed copper zone on B.Cu, net P9

Commit message: update stuff.
Connections:
- C4 pad 1: Net-(J3-B) -> P1
Routing:
- net Net-(J3-B): track 11.0 -> 8.43 mm
- net P1: track 16.3 -> 17.7 mm, vias 5 -> 6
Other:
- board size 29.4 x 32.4 mm -> 29.4 x 32.2 mm
- board text added: "IOT_Mess ESP_P16 V2.0 8/19/25"
- board text removed: "IOT_Mess ESP_P16 V1.0 7/5/25"
