File: Version1/IOT-Mess-ESP_P16/IOT-Mess-ESP_P16.kicad_sch (KiCad schematic)
At the start: 23 parts, among them J1 Conn_01x10_Pin, J2 Conn_01x09_Pin, J3 Jumper_2, J4 Jumper_2, J5 Jumper_2, J6 Jumper_2, SW10 SW_Push, SW11 SW_Push, U1 ESP-12F, U10 USB_C_Receptacle_USB2.0_16P, U5 ESP32-C3-WROOM-02, U6 ME6211C33M5

Commit message: updated.
Parts:
- removed D2: 1N5819WS, Diode_SMD:D_SOD-323, symbol Diode:1N5819WS
- added U2: XC6206PxxxMR, Package_TO_SOT_SMD:SOT-23-3, symbol Regulator_Linear:XC6206PxxxMR
Connections:
- net +3.3V: no longer C4.1
- net 5V: now also J4.1 (A), U10.A4 (VBUS), U10.A9 (VBUS), U10.B4 (VBUS), U10.B9 (VBUS), U2.3 (VI); no longer C5.1, J4.2 (B), U6.3 (CE)
- net GND: now also U2.1 (GND)
- net at J3.2 (B), U6.5 (V_{OUT}): now also C4.1, U2.2 (VO)
- new net: C5.1, J4.2 (B), U6.3 (CE)
Other:
- moved on the sheet: C4, C5, D1, J1, J2, J3, R5, U6

Commit message: update stuff.
Connections:
- net +3.3V: now also C4.1
- net at J3.2 (B), U2.2 (VO), U6.5 (V_{OUT}): no longer C4.1
Other:
- moved on the sheet: C4
Changed lines of the file:
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@@
 	)
 	(junction
+		(at 181.61 214.63)
+		(diameter 0)
+		(color 0 0 0 0)
+	)
+	(junction
 		(at 111.76 226.06)
 		(diameter 0)
@@
 	(wire
 		(pts
-			(xy 147.32 214.63) (xy 147.32 218.44)
+			(xy 181.61 214.63) (xy 181.61 218.44)
 		)
 		(stroke
@@
 	(symbol
 		(lib_id "Device:C")
-		(at 147.32 222.25 0)
+		(at 181.61 222.25 0)
 		(unit 1)
 		(exclude_from_sim no)
@@
 		(fields_autoplaced yes)
 		(property "Reference" "C4"
-			(at 150.495 220.98 0)
+			(at 184.785 220.98 0)
 			(effects
 				(font
@@
 		)
 		(property "Value" "1u"
-			(at 150.495 223.52 0)
+			(at 184.785 223.52 0)
 			(effects
 				(font
@@
 		)
 		(property "Footprint" "Capacitor_SMD:C_0603_1608Metric"
-			(at 148.2852 226.06 0)
+			(at 182.5752 226.06 0)
 			(effects
 				(font
@@
 		)
 		(property "Datasheet" "~"
-			(at 147.32 222.25 0)
+			(at 181.61 222.25 0)
 			(effects
 				(font
@@
 		)
 		(property "Description" ""
-			(at 147.32 222.25 0)
+			(at 181.61 222.25 0)
 			(effects
 				(font
@@
 		(lib_name "GND_1")
 		(lib_id "power:GND")
-		(at 147.32 226.06 0)
+		(at 181.61 226.06 0)
 		(unit 1)
 		(exclude_from_sim no)
@@
 		(fields_autoplaced yes)
 		(property "Reference" "#PWR015"
-			(at 147.32 232.41 0)
+			(at 181.61 232.41 0)
 			(effects
 				(font
@@
 		)
 		(property "Value" "GND"
-			(at 147.32 231.14 0)
+			(at 181.61 231.14 0)
 			(effects
 				(font
@@
 		)
 		(property "Footprint" ""
-			(at 147.32 226.06 0)
+			(at 181.61 226.06 0)
 			(effects
 				(font
@@
 		)
 		(property "Datasheet" ""
-			(at 147.32 226.06 0)
+			(at 181.61 226.06 0)
 			(effects
 				(font
@@
 		)
 		(property "Description" "Power symbol creates a global label with name \"GND\" , ground"
-			(at 147.32 226.06 0)
+			(at 181.61 226.06 0)
 			(effects
 				(font
