File: Version2/Mess-CHP20/IOT-MESS-CHP20.kicad_pcb (KiCad board)
At the start: 2 copper layers, 24.5 x 47.5 mm, 26 parts, among them J1 Jumper_2, J2 Jumper_2, J3 Jumper, J4 Conn_01x15_Pin, J5 Conn_01x15_Pin, J6 Jumper, J7 Jumper_2, J9 Jumper_2, K1 Crystal, U4 USB_C_Receptacle_USB2.0_16P, U5 ME6211C33M5, U6 XC6206PxxxMR

Commit message: updated.
Parts:
- AE2: footprint RF_Antenna:Texas_SWRA117D_2.4GHz_Right -> RF_Antenna:Texas_SWRA117D_2.4GHz_Left
- moved AE2 9.27 mm to (181.6, 94.3)
- moved J3 8.49 mm to (179.0, 95.6), turned to 0 degrees
Connections:
- AE2 pad 2: P_0 -> unconnected-(AE2-Shield-Pad2)
Routing:
- net P_20: track 35.7 -> 26.6 mm
- net P_5: track 46.1 -> 55.1 mm
- net P_16: track 60.0 -> 65.3 mm
- net P_10: track 29.7 -> 31.0 mm
- net P_17: track 44.0 -> 43.0 mm
- net OSCO: track 17.6 -> 18.6 mm
- net ANT: track 4.44 -> 3.69 mm
- net OSCI: track 22.5 -> 21.9 mm
- net P_6: track 40.5 -> 40.0 mm
- net P_18: track 37.7 -> 37.1 mm

Commit message: update stuff.
Connections:
- C5 pad 1: Net-(J9-A) -> +3.3V
Routing:
- net +3.3V: track 18.5 -> 21.7 mm
- net Net-(J9-A): track 9.05 -> 8.70 mm, vias 1 -> 2
Other:
- board text added: "IOT_Mess P20 V2.0 8/19/25"
- board text removed: "IOT_Mess CH-P20 V1.2 8/12/25"
Changed lines of the file:
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@@
 			(layers "F.Cu" "F.Mask" "F.Paste")
 			(roundrect_rratio 0.25)
-			(net 32 "Net-(J9-A)")
+			(net 18 "+3.3V")
 			(pintype "passive")
 		)
@@
 		)
 	)
-	(gr_text "IOT_Mess CH-P20\nV1.2 8/12/25"
+	(gr_text "IOT_Mess P20\nV2.0 8/19/25"
 		(at 177 92.4 0)
 		(layer "B.SilkS")
@@
 	)
 	(segment
+		(start 179.650002 119.825)
+		(end 179.650002 121.000002)
+		(width 0.5)
+		(layer "F.Cu")
+		(net 18)
+	)
+	(segment
 		(start 170.2 120.95)
 		(end 170.2 119.8)
@@
 	)
 	(segment
+		(start 179.650002 121.000002)
+		(end 181.1 122.45)
+		(width 0.5)
+		(layer "F.Cu")
+		(net 18)
+	)
+	(segment
 		(start 178.801002 118.651)
 		(end 179.650002 119.5)
@@
 	)
 	(segment
-		(start 181.1 122.45)
-		(end 181.1 120.025)
-		(width 0.5)
-		(layer "F.Cu")
-		(net 32)
-	)
-	(segment
-		(start 180.75 122.1)
-		(end 181.1 122.45)
+		(start 178.6 121.2)
+		(end 178.6 121.8)
 		(width 0.5)
 		(layer "F.Cu")
@@
 	)
 	(segment
-		(start 178.3 122.1)
-		(end 180.75 122.1)
+		(start 178.6 121.8)
+		(end 178.3 122.1)
 		(width 0.5)
 		(layer "F.Cu")
@@
 	)
 	(via
+		(at 178.6 121.2)
+		(size 0.6)
+		(drill 0.3)
+		(layers "F.Cu" "B.Cu")
+		(net 32)
+	)
+	(via
 		(at 182.1 120)
 		(size 0.6)
@@
 	)
 	(segment
+		(start 182.1 120)
+		(end 179.8 120)
+		(width 0.5)
+		(layer "B.Cu")
+		(net 32)
+	)
+	(segment
 		(start 182.1 122.074999)
 		(end 181.749999 122.425)
@@
 	)
 	(segment
+		(start 179.8 120)
+		(end 178.6 121.2)
+		(width 0.5)
+		(layer "B.Cu")
+		(net 32)
+	)
+	(segment
 		(start 170.2 122.6)
 		(end 170.2 124.312499)
@@
 		(polygon
 			(pts
-				(xy 160.8 93.1) (xy 193.1 93.1) (xy 193.1 135.8) (xy 160.8 135.8)
+				(xy 164.6 93.1) (xy 189.1 93.1) (xy 189.1 135.8) (xy 164.6 135.8)
 			)
 		)

Commit message: updates.
Parts:
- moved AE2 1.50 mm to (181.6, 92.8)
Routing:
- net ANT: track 3.69 -> 5.19 mm
Other:
- board size 24.5 x 47.5 mm -> 24.5 x 48.9 mm
Changed lines of the file:
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@@
 	(footprint "RF_Antenna:Texas_SWRA117D_2.4GHz_Left"
 		(layer "F.Cu")
-		(at 181.6 94.3)
+		(at 181.6 92.8)
 		(descr "http://www.ti.com/lit/an/swra117d/swra117d.pdf")
 		(tags "PCB antenna")
@@
 	)
 	(gr_rect
-		(start 164.6 88.3)
+		(start 164.6 86.9)
 		(end 189.1 135.8)
 		(stroke
@@
 		(layer "Dwgs.User")
 		(pts
-			(xy 164.6 88.3) (xy 164.6 135.8)
+			(xy 164.7 86.8) (xy 164.6 135.8)
 		)
 		(height -6.5)
@@
 			(keep_text_aligned yes)
 		)
-		(gr_text "47.5"
-			(at 156.95 112.05 90)
+		(gr_text "49"
+			(at 157.05 111.3 90)
 			(layer "Dwgs.User")
 			(effects
@@
 	)
 	(segment
+		(start 181.6 94.3)
+		(end 181.6 92.8)
+		(width 0.4)
+		(layer "F.Cu")
+		(net 31)
+	)
+	(segment
