File: Version2/Mess-P48/Mess-P48.kicad_pcb (KiCad board)
At the start: 2 copper layers, 29.8 x 49.4 mm, 38 parts, among them J1 Jumper_2, J10 Conn_01x19_Pin, J11 Conn_01x19_Pin, J2 Conn_01x06_Pin, J3 Conn_01x08_Pin, J4 Conn_01x08_Pin, K1 Crystal, K2 Crystal, SW1 SW_Push, U1 USB_C_Receptacle_USB2.0_16P, U3 XC6206PxxxMR, U4 ME6211C33M5, U5 CH32L103C8T6

Commit message: update stuff.
Other:
- board text added: "IOT_Mess P48 V2.0 8/19/25"
- board text removed: "IOT_Mess P48 V1.1 8/15/25"
Changed lines of the file:
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@@
 		)
 		(property "Datasheet" "~"
-			(at 0 0 -90)
+			(at 0 0 270)
 			(unlocked yes)
 			(layer "B.Fab")
@@
 		)
 		(property "Description" "Jumper, 2-pole, small symbol, open"
-			(at 0 0 -90)
+			(at 0 0 270)
 			(unlocked yes)
 			(layer "B.Fab")
@@
 			(fill yes)
 			(layer "B.SilkS")
-			(net 128259028)
 		)
 		(fp_poly
@@
 			(fill yes)
 			(layer "B.SilkS")
-			(net 128259028)
 		)
 		(fp_poly
@@
 			(fill yes)
 			(layer "B.SilkS")
-			(net 128259028)
 		)
 		(embedded_fonts no)
@@
 		)
 	)
-	(gr_text "IOT_Mess P48 V1.1\n8/15/25"
+	(gr_text "IOT_Mess P48 V2.0\n8/19/25"
 		(at 134.2 114.8 0)
 		(layer "B.SilkS")
