File: Version2/Mess-Perfboard/IOT-Mess-BaseSmall.kicad_pcb (KiCad board)
At the start: 2 copper layers, 49.6 x 100 mm, 12 parts, among them J1 Conn_02x34_Odd_Even, J15 Conn_02x19_Odd_Even, J18 Conn_02x19_Odd_Even, J2 Conn_02x34_Odd_Even, J20 Conn_01x34_Pin, J3 Conn_01x34_Pin, J4 Conn_01x34_Pin, J5 Conn_02x34_Odd_Even, J6 Conn_02x34_Odd_Even, J7 Conn_02x34_Odd_Even, J8 Conn_02x34_Odd_Even, J9 Conn_02x34_Odd_Even

Commit message: update stuff.
Other:
- board size 49.6 x 100 mm -> 49.2 x 99.6 mm
- board text added: "IOT_Mess Perfboard V2.0 8/19/25"
