File: Version2/Mess-Perfboard/IOT-Mess-BaseSmall.kicad_sch (KiCad schematic)
At the start: 19 parts, among them J1 Conn_02x34_Odd_Even, J10 ESP_P40, J11 Milk-V Duo, J12 ESP_P16 / ESP12, J13 SuperMini_ESP32-H2, J14 Lolin32-Lite, J15 Conn_02x19_Odd_Even, J16 CH582, J17 CH_P20, J18 Conn_02x19_Odd_Even, J2 Conn_02x34_Odd_Even, J20 Conn_01x34_Pin, J3 Conn_01x34_Pin, J4 Conn_01x34_Pin, J5 Conn_02x34_Odd_Even, J6 Conn_02x34_Odd_Even, J7 Conn_02x34_Odd_Even, J8 Conn_02x34_Odd_Even, J9 Conn_02x34_Odd_Even

Commit message: update stuff.
Parts:
- removed J10: ESP_P40, IOT-Mess-Footprints:ESP_P40, symbol Connector_Generic_Shielded:Conn_02x19_Top_Bottom_Shielded
- removed J11: Milk-V Duo, IOT-Mess-Footprints:Milk-V Duo, symbol Connector_Generic:Conn_02x20_Counter_Clockwise
- removed J12: ESP_P16 / ESP12, IOT-Mess-Footprints:ESP_P16, symbol IOT-Mess:ESP_P16
- removed J13: SuperMini_ESP32-H2, IOT-Mess-Footprints:SuperMiniH2, symbol IOT-Mess:SuperMini_ESP32-H2
- removed J14: Lolin32-Lite, IOT-Mess-Footprints:Lolin32-Lite, symbol IOT-Mess:Lolin32-Lite
- removed J16: CH582, IOT-Mess-Footprints:CH582_Base, symbol Connector_Generic:Conn_02x12_Top_Bottom
- removed J17: CH_P20, IOT-Mess-Footprints:CH_P20, symbol IOT-Mess:CH_P20
