File: Version2/PWR-Sleep/PWR-Sleep.kicad_pcb (KiCad board)
At the start: 2 copper layers, 19.6 x 49.6 mm, 37 parts, among them J1 Conn_01x18_Pin, J2 SN74LVC1 (AND Gate), Q1 BM8205 PFETs, Q2 AO3401A, SW1 SW_Push, SW2 SW_Push, U1 XC6206PxxxMR, U10 INA219AxD, U2 ME6211C33M5, U3 TPL5110, U4 INA219AxDCN, U5 INA219AxDCN, U6 INA219AxDCN, U7 INA219AxDCN, U8 INA219AxD, U9 INA219AxD

Commit message: hardware updates.
Parts:
- added EN4: Jumper_2, IOT-Mess-Footprints:Jumpper-triangle, B.Cu at (114.9, 109.3)
- added Q3: AO3401A, Package_TO_SOT_SMD:SOT-23, B.Cu at (107.9, 104.1)
- added Q4: AO3400A, Package_TO_SOT_SMD:SOT-23, B.Cu at (113.0, 106.5)
- added R19: R, Resistor_SMD:R_0603_1608Metric, B.Cu at (109.5, 107.9)
- moved G*** 3.07 mm to (109.9, 98.3)
- moved EN2 2.79 mm to (103.1, 105.3), turned to 90 degrees
Connections:
- net Net-(J2-Pin_4) renamed PWR_G
Routing:
- net PWR_G: track 8.73 -> 15.5 mm, vias 0 -> 1
- net PWR: track 37.5 -> 42.3 mm
- net EN: track 16.1 -> 19.7 mm, vias 0 -> 1
- net DRV: track 21.1 -> 24.6 mm
- net GND: track 36.1 -> 39.4 mm, vias 8 -> 9
- net V4b: track 69.7 -> 71.8 mm, vias 2 -> 3
- net Net-(EN4-A): track 14.7 -> 15.7 mm, vias 0 -> 1
