File: Version2/PWR-Sleep/PWR-Sleep.kicad_sch (KiCad schematic)
At the start: 36 parts, among them J1 Conn_01x18_Pin, J2 SN74LVC1 (AND Gate), Q1 BM8205 PFETs, Q2 AO3401A, SW1 SW_Push, SW2 SW_Push, U1 XC6206PxxxMR, U10 INA219AxD, U2 ME6211C33M5, U3 TPL5110, U4 INA219AxDCN, U5 INA219AxDCN, U6 INA219AxDCN, U7 INA219AxDCN, U8 INA219AxD, U9 INA219AxD

Commit message: hardware updates.
Parts:
- added EN4: Jumper_2, IOT-Mess-Footprints:Jumpper-triangle, symbol Jumper:Jumper_2_Small_Open
- added Q3: AO3401A, Package_TO_SOT_SMD:SOT-23, symbol Transistor_FET:AO3401A
- added Q4: AO3400A, Package_TO_SOT_SMD:SOT-23, symbol Transistor_FET:AO3400A
- added R19: R, Resistor_SMD:R_0603_1608Metric, symbol Device:R
Connections:
- net DRV: now also Q3.1 (G)
- net EN: now also Q4.1 (G), R19.2
- net GND: now also Q4.2 (S), R19.1
- net PWR: now also Q3.3 (D)
- net V4b: now also Q3.2 (S)
- net PWR_G: now reaches J2.4 (Pin_4), Q2.1 (G)
- net PWR_G: now also EN4.2 (B), Q4.3 (D)
- net at J2.1 (Pin_1), Q1.2 (S1/D2), Q1.5 (S1/D2)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: now also EN4.1 (A)
Other:
- moved on the sheet: C1, C2, C3, C4, EN1, EN2, EN3, J1, J2, Q1, Q2, R1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
