File: PowerCircuit/PowerCircuit/PowerCircuit.kicad_sch (KiCad schematic)
At the start: 44 parts, among them J1 Jumper_2, J3 Jumper_2, J4 Jumper_2, J5 Jumper_2, J6 Jumper_2, J7 Conn_01x04_Pin, J8 Conn_01x02_Pin, J9 Conn_01x12_Pin, Q1 AO3400A, Q10 AO3401A (P-Fet), Q11 AO3400A, Q12 AO3401A (P-Fet), Q2 AO3401A (P-Fet), Q3 AO3401A (P-Fet), Q4 AO3400A, Q5 AO3401A (P-Fet), Q6 AO3400A, Q7 AO3400A, Q8 AO3401A (P-Fet), Q9 AO3401A (P-Fet), U1 XC6206PxxxMR

Commit message: update schematic.
Parts:
- removed Q7: AO3400A, Package_TO_SOT_SMD:SOT-23, symbol Transistor_FET:AO3400A
- removed Q9: AO3401A (P-Fet), Package_TO_SOT_SMD:SOT-23, symbol Transistor_FET:AO3401A
- removed TP4: TestPoint, Connector_PinHeader_1.00mm:PinHeader_1x01_P1.00mm_Vertical, symbol Connector:TestPoint
- added C1: C, symbol Device:C
- added J10, J11, J12, J13, J14, J15, J16, J2: Jumper_2, IOT-Mess-Footprints:Jumpper-triangle, symbol Jumper:Jumper_2_Small_Open
- added R16, R19: R_Variable, symbol Device:R_Variable
- added R17, R18, R6: 10K, Resistor_SMD:R_0805_2012Metric, symbol Device:R
- added U2, U5: LT431 (Voltage Ref), Package_TO_SOT_SMD:SOT-23, symbol Power_Management:BD48LxxG
- added U3: 74LV1T08GW, Package_TO_SOT_SMD:SOT-353_SC-70-5, symbol 74xx:74LV1T08GW
- added U4: MT9700, Package_TO_SOT_SMD:SOT-23-5, symbol Power_Management:AAT4616IGV-1-T1
- R12: value 100K -> 10K
Connections:
- net GND: now also R12.1, C1.2, R16.2, R17.1, R19.2, U2.3 (GND), U3.3 (GND), U4.2 (GND), U5.3 (GND)
- net IN-: no longer J3.2 (B)
- net SOLAR/IN+: no longer J1.2 (B)
- net SW_CHARGER: now also J16.1 (A)
- net SW_PWR1: now also J14.1 (A)
- net SW_PWR2: now also J13.1 (A), U3.2 (A)
- net VCC/BATT: now also U3.1 (B), U3.5 (VCC), U4.5 (IN); no longer R12.2
- net at J5.2 (B), Q10.1 (G), R13.2: now also J10.2 (B), J2.1 (A); no longer J4.2 (B), Q11.1 (G)
- net at Q10.3 (D), Q12.3 (D), U1.3 (VI): now also C1.1
- net at J5.1 (A): now also U3.4 (Y)
- net at D3.1 (K), D4.1 (K), Q12.2 (S)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: now also J1.2 (B), J3.2 (B), J11.1 (A), J15.1 (A)
- new net: J16.2 (B), R18.1, R19.1, U5.1 (VOUT)
- new net: J15.2 (B), R18.2, U5.2 (VDD)
- new net: J12.2 (B), J13.2 (B), J14.2 (B), R16.1, R6.1, U2.1 (VOUT)
- new net: J2.2 (B), J4.2 (B), Q11.1 (G)
- new net: J11.2 (B), R6.2, U2.2 (VDD)
- new net: J10.1 (A), U4.1 (OUT)
- new net: R12.2, U4.3 (SET)
- new net SW_PWR3: J12.1 (A), R17.2, U4.4 (ON)
Other:
- note added: "A |B |Y H |H |H L |X |L X |L |L"
- note added: "Drivers Gate Switch"
- note added: "Q12 ON, Q10 OFF -> Battery to Load Q12 OFF, Q10 ON -> Solar to Load"
- note removed: "Q2 & Q4 Gates Switch"
- note removed: "Q2 ON, Q4 OFF -> Battery to Load Q2 OFF, Q4 ON -> Solar to Load"
- moved on the sheet: D1, D2, D3, D4, D5, J1, J3, J4, J6, J7, J8, J9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
