File: Panelized/Mess-Breakout+Perf/Mess-Breakout+Perf.kicad_pcb (KiCad board)
At the start: 2 copper layers, 98 x 108.8 mm, 105 parts, among them J10 Conn_01x30_Pin, J11 Conn_02x38_Odd_Even, J12 Conn_01x38_Pin, J13 Conn_02x30_Odd_Even, J2 Conn_01x30_Pin, J3 Conn_02x38_Odd_Even, J4 Conn_01x38_Pin, J5 Conn_02x30_Odd_Even, J6 Conn_01x30_Pin, J7 Conn_02x38_Odd_Even, J8 Conn_01x38_Pin, J9 Conn_02x30_Odd_Even, P1 Jumper4x1, P10 Jumper4x1, P11 Jumper4x1, P12 Jumper4x1, P13 Jumper4x1, P14 Jumper4x1, P15 Jumper4x1, P16 Jumper4x1, P17 Jumper4x1, P18 Jumper4x1, P19 Jumper4x1, P2 Jumper4x1, P20 Jumper4x1, P21 Jumper4x1, P22 Jumper4x1, P23 Jumper4x1, P24 Jumper4x1, P25 Jumper4x1, P26 Jumper4x1, P27 Jumper4x1, P28 Jumper4x1, P29 Jumper4x1, P3 Jumper4x1, P30 Jumper4x1, P31 Jumper4x1, P32 Jumper4x1, P33 Jumper4x1, P34 Jumper4x1, P35 Jumper4x1, P36 Jumper4x1, P37 Jumper4x1, P38 Jumper4x1, P39 Jumper4x1, P4 Jumper4x1, P40 Jumper4x1, P41 Jumper4x1, P42 Jumper4x1, P43 Jumper4x1, P44 Jumper4x1, P45 Jumper4x1, P46 Jumper4x1, P47 Jumper4x1, P48 Jumper4x1, P49 Jumper4x1, P5 Jumper4x1, P50 Jumper4x1, P51 Jumper4x1, P52 Jumper4x1, P53 Jumper4x1, P54 Jumper4x1, P55 Jumper4x1, P56 Jumper4x1, P57 Jumper4x1, P58 Jumper4x1, P59 Jumper4x1, P6 Jumper4x1, P60 Jumper4x1, P61 Jumper4x1, P62 Jumper4x1, P63 Jumper4x1, P64 Jumper4x1, P65 Jumper4x1, P66 Jumper4x1, P67 Jumper4x1, P68 Jumper4x1, P69 Jumper4x1, P7 Jumper4x1, P70 Jumper4x1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

Commit message: updates.
Parts:
- moved G*** 37.1 mm to (141.1, 80.9)
- moved G***2 37.1 mm to (108.1, 80.9)
- moved J3 37.1 mm to (122.5, 44.9)
- moved P10 37.1 mm to (138.1, 69.3)
- moved P11 37.1 mm to (138.1, 73.2)
- moved P12 37.1 mm to (138.1, 77.2)
- moved P13 37.1 mm to (138.1, 81.0)
- moved P14 37.1 mm to (138.1, 85.0)
- moved P15 37.1 mm to (138.1, 89.0)
- moved P16 37.1 mm to (138.1, 92.8)
- moved P17 37.1 mm to (138.1, 96.8)
- moved P18 37.1 mm to (138.1, 100.8)
- moved P19 37.1 mm to (138.1, 104.7)
- moved P20 37.1 mm to (138.1, 108.5)
- moved P21 37.1 mm to (138.1, 112.5)
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Other:
- board size 98 x 108.8 mm -> 98.1 x 99.8 mm
- board text added: "1"
- board text added: "10"
- board text added: "11"
- board text added: "12"
- board text added: "13"
- board text added: "14"
- board text added: "15"
- board text added: "16"
- board text added: "17"
- board text added: "18"
- board text added: "19"
- board text added: "2"
- board text added: "20"
- board text added: "21"
- board text added: "22"
- board text added: "23"
- board text added: "24"
- board text added: "25"
- board text added: "26"
- board text added: "27"
- board text added: "28"
- board text added: "29"
- board text added: "3"
- board text added: "30"
- board text added: "31"
- board text added: "32"
- board text added: "33"
- board text added: "34"
- board text added: "35"
- board text added: "36"
- board text added: "37"
- board text added: "38"
- board text added: "4"
- board text added: "5"
- board text added: "6"
- board text added: "7"
- board text added: "8"
- board text added: "9"
