File: Panelized/Mess-P20+PowerCircuit/Mess-P20+PowerCircuit.kicad_pcb (KiCad board)
At the start: 2 copper layers, 99 x 100 mm, 380 parts, among them J100 Jumper_2, J101 Jumper, J102 Jumper_2, J103 Conn_01x04_Pin, J104 Conn_01x02_Pin, J105 Jumper_2, J106 Conn_01x12_Pin, J107 Jumper_2, J108 Jumper_2, J109 Jumper_2, J110 Jumper_2, J111 Jumper_2, J112 Jumper_2, J113 Jumper_2, J114 Conn_01x01_Pin, J115 Jumper_2, J116 Jumper_2, J117 Jumper_2, J118 Jumper, J119 Jumper_2, J120 Jumper_2, J121 Conn_01x15_Pin, J122 Jumper_2, J123 Conn_01x15_Pin, J124 Jumper_2, J125 Jumper, J126 Jumper_2, J127 Conn_01x04_Pin, J128 Conn_01x02_Pin, J129 Jumper_2, J13 Jumper_2, J130 Conn_01x12_Pin, J131 Jumper_2, J132 Jumper_2, J133 Jumper_2, J134 Jumper_2, J135 Jumper_2, J136 Jumper_2, J137 Jumper_2, J138 Conn_01x01_Pin, J14 Jumper_2, J15 Jumper_2, J16 Jumper_2, J43 Jumper_2, J44 Jumper_2, J45 Jumper_2, J46 Jumper, J47 Jumper_2, J48 Jumper_2, J49 Conn_01x15_Pin, J50 Jumper_2, J51 Conn_01x15_Pin, J52 Jumper_2, J53 Jumper, J54 Jumper_2, J55 Conn_01x04_Pin, J56 Conn_01x02_Pin, J57 Jumper_2, J58 Conn_01x12_Pin, J59 Jumper_2, J60 Jumper_2, J61 Jumper_2, J62 Jumper_2, J63 Jumper_2, J64 Jumper_2, J65 Jumper_2, J66 Conn_01x01_Pin, J67 Jumper_2, J68 Jumper_2, J69 Jumper_2, J70 Jumper, J71 Jumper_2, J72 Jumper_2, J73 Conn_01x15_Pin, J74 Jumper_2, J75 Conn_01x15_Pin, J76 Jumper_2, J77 Jumper, J78 Jumper_2, J79 Conn_01x04_Pin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

Commit message: update.
Parts:
- removed G***10, G***4, G***6, G***8: LOGO, IOT-Mess-Footprints:catIcon8x8
Other:
- outline, holes or cut-outs redrawn
- board text removed: "IOT_Mess Power V1.0 12/18/25"
