File: Panelized/Mess-Sense+USBC/Mess-Sense+USBC.kicad_pcb (KiCad board)
At the start: 2 copper layers, 109.7 x 108.8 mm, 430 parts, among them IC1 SHT40I-AD1F-R2, IC10 SHT40I-AD1F-R2, IC2 SHT40I-AD1F-R2, IC3 SHT40I-AD1F-R2, IC4 SHT40I-AD1F-R2, IC5 SHT40I-AD1F-R2, IC6 SHT40I-AD1F-R2, IC7 SHT40I-AD1F-R2, IC8 SHT40I-AD1F-R2, IC9 SHT40I-AD1F-R2, J1 Conn_01x06_Pin, J10 Conn_01x04_Pin, J11 Jumper_2, J12 Conn_01x04_Pin, J13 Jumper_2, J14 Conn_01x02_Pin, J15 Jumper_2, J16 Conn_01x02_Pin, J17 Conn_01x06_Pin, J18 Conn_01x04_Pin, J19 Jumper_2, J2 Conn_01x04_Pin, J20 Conn_01x04_Pin, J21 Jumper_2, J22 Conn_01x02_Pin, J23 Jumper_2, J24 Conn_01x02_Pin, J25 Conn_01x06_Pin, J26 Conn_01x04_Pin, J27 Jumper_2, J28 Conn_01x04_Pin, J29 Jumper_2, J3 Jumper_2, J30 Conn_01x02_Pin, J31 Jumper_2, J32 Conn_01x02_Pin, J33 Conn_01x06_Pin, J34 Conn_01x04_Pin, J35 Jumper_2, J36 Conn_01x04_Pin, J37 Jumper_2, J38 Conn_01x02_Pin, J39 Jumper_2, J4 Conn_01x04_Pin, J40 Conn_01x02_Pin, J41 Conn_01x06_Pin, J42 Conn_01x04_Pin, J43 Jumper_2, J44 Conn_01x04_Pin, J45 Jumper_2, J46 Conn_01x02_Pin, J47 Jumper_2, J48 Conn_01x02_Pin, J49 Conn_01x06_Pin, J5 Jumper_2, J50 Conn_01x04_Pin, J51 Jumper_2, J52 Conn_01x04_Pin, J53 Jumper_2, J54 Conn_01x02_Pin, J55 Jumper_2, J56 Conn_01x02_Pin, J57 Conn_01x06_Pin, J58 Conn_01x04_Pin, J59 Jumper_2, J6 Conn_01x02_Pin, J60 Conn_01x04_Pin, J61 Jumper_2, J62 Conn_01x02_Pin, J63 Jumper_2, J64 Conn_01x02_Pin, J65 Conn_01x06_Pin, J66 Conn_01x04_Pin, J67 Jumper_2, J68 Conn_01x04_Pin, J69 Jumper_2, J7 Jumper_2, J70 Conn_01x02_Pin, J71 Jumper_2, J72 Conn_01x02_Pin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

Commit message: updates.
Parts:
- moved C42 18.8 mm to (117.8, 96.7)
- moved C49 18.8 mm to (167.8, 96.7)
- moved C56 18.8 mm to (117.8, 116.7)
- moved C63 18.8 mm to (167.8, 116.7)
- moved C7 18.8 mm to (167.8, 136.7)
- moved C70 18.8 mm to (117.8, 136.7)
- moved J4 18.8 mm to (181.3, 137.6)
- moved J6 18.8 mm to (147.8, 139.7)
- moved J76 18.8 mm to (131.3, 137.6)
- moved R1 18.8 mm to (156.4, 142.7)
- moved R2 18.8 mm to (156.4, 142.7)
- moved R4 18.8 mm to (140.4, 135.5)
- moved R76 18.8 mm to (90.4, 135.5)
- moved U100 18.8 mm to (172.4, 104.2)
- moved U132 18.8 mm to (172.4, 124.2)
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Other:
- board size 109.7 x 108.8 mm -> 99.1 x 99.1 mm

Commit message: update.
Parts:
- added J81: Conn_01x07_Pin, Connector_PinHeader_2.54mm:PinHeader_1x07_P2.54mm_Vertical, F.Cu at (145.9, 109.4)
- added J82: Conn_01x06_Pin, Connector_PinHeader_2.54mm:PinHeader_1x06_P2.54mm_Vertical, F.Cu at (72.3, 131.2)
- added J83: Conn_01x04_Pin, Connector_PinHeader_2.54mm:PinHeader_1x04_P2.54mm_Vertical, F.Cu at (99.1, 137.0)
- added J84: Jumper_2, IOT-Mess-Footprints:Jumpper-triangle, F.Cu at (112.7, 130.0)
- added J85: Conn_01x04_Pin, Connector_PinHeader_2.54mm:PinHeader_1x04_P2.54mm_Vertical, F.Cu at (116.9, 137.0)
- added J86: Jumper_2, IOT-Mess-Footprints:Jumpper-triangle, F.Cu at (98.9, 130.0)
- added J87: Conn_01x02_Pin, Connector_PinHeader_1.27mm:PinHeader_1x02_P1.27mm_Vertical, F.Cu at (83.3, 139.1)
- added J88: Jumper_2, IOT-Mess-Footprints:Jumpper-triangle, F.Cu at (102.3, 130.0)
- added J89: Conn_01x02_Pin, Connector_PinHeader_2.54mm:PinHeader_1x02_P2.54mm_Vertical, F.Cu at (92.9, 130.5)
- added J90: Conn_01x07_Pin, Connector_PinHeader_2.54mm:PinHeader_1x07_P2.54mm_Vertical, F.Cu at (95.9, 129.4)
- J10, J28: value Conn_01x04_Pin -> Conn_01x06_Pin; footprint Connector_PinHeader_2.54mm:PinHeader_1x04_P2.54mm_Vertical -> Connector_PinHeader_2.54mm:PinHeader_1x06_P2.54mm_Vertical
- J11, J13, J29, J31, J47, J67: value Jumper_2 -> Conn_01x04_Pin; footprint IOT-Mess-Footprints:Jumpper-triangle -> Connector_PinHeader_2.54mm:PinHeader_1x04_P2.54mm_Vertical
- J12, J34, J50, J52, J66, J68: value Conn_01x04_Pin -> Jumper_2; footprint Connector_PinHeader_2.54mm:PinHeader_1x04_P2.54mm_Vertical -> IOT-Mess-Footprints:Jumpper-triangle
- J14, J30, J70: value Conn_01x02_Pin -> Jumper_2; footprint Connector_PinHeader_1.27mm:PinHeader_1x02_P1.27mm_Vertical -> IOT-Mess-Footprints:Jumpper-triangle
- J15, J51, J69: value Jumper_2 -> Conn_01x02_Pin; footprint IOT-Mess-Footprints:Jumpper-triangle -> Connector_PinHeader_1.27mm:PinHeader_1x02_P1.27mm_Vertical
- J16, J32, J48: value Conn_01x02_Pin -> Jumper_2; footprint Connector_PinHeader_2.54mm:PinHeader_1x02_P2.54mm_Vertical -> IOT-Mess-Footprints:Jumpper-triangle
- J17: value Conn_01x06_Pin -> Conn_01x02_Pin; footprint Connector_PinHeader_2.54mm:PinHeader_1x06_P2.54mm_Vertical -> Connector_PinHeader_2.54mm:PinHeader_1x02_P2.54mm_Vertical
- J18, J36: value Conn_01x04_Pin -> Conn_01x07_Pin; footprint Connector_PinHeader_2.54mm:PinHeader_1x04_P2.54mm_Vertical -> Connector_PinHeader_2.54mm:PinHeader_1x07_P2.54mm_Vertical
- J19, J37, J55: value Jumper_2 -> Conn_01x06_Pin; footprint IOT-Mess-Footprints:Jumpper-triangle -> Connector_PinHeader_2.54mm:PinHeader_1x06_P2.54mm_Vertical
- J22, J38: value Conn_01x02_Pin -> Conn_01x04_Pin; footprint Connector_PinHeader_1.27mm:PinHeader_1x02_P1.27mm_Vertical -> Connector_PinHeader_2.54mm:PinHeader_1x04_P2.54mm_Vertical
- J24: footprint Connector_PinHeader_2.54mm:PinHeader_1x02_P2.54mm_Vertical -> Connector_PinHeader_1.27mm:PinHeader_1x02_P1.27mm_Vertical
- J25, J41, J57: value Conn_01x06_Pin -> Jumper_2; footprint Connector_PinHeader_2.54mm:PinHeader_1x06_P2.54mm_Vertical -> IOT-Mess-Footprints:Jumpper-triangle
- J26, J44: value Conn_01x04_Pin -> Conn_01x02_Pin; footprint Connector_PinHeader_2.54mm:PinHeader_1x04_P2.54mm_Vertical -> Connector_PinHeader_2.54mm:PinHeader_1x02_P2.54mm_Vertical
- J27, J45, J63: value Jumper_2 -> Conn_01x07_Pin; footprint IOT-Mess-Footprints:Jumpper-triangle -> Connector_PinHeader_2.54mm:PinHeader_1x07_P2.54mm_Vertical
- J33: value Conn_01x06_Pin -> Conn_01x02_Pin; footprint Connector_PinHeader_2.54mm:PinHeader_1x06_P2.54mm_Vertical -> Connector_PinHeader_1.27mm:PinHeader_1x02_P1.27mm_Vertical
- J35, J53, J71: value Jumper_2 -> Conn_01x02_Pin; footprint IOT-Mess-Footprints:Jumpper-triangle -> Connector_PinHeader_2.54mm:PinHeader_1x02_P2.54mm_Vertical
- J40, J56: value Conn_01x02_Pin -> Conn_01x04_Pin; footprint Connector_PinHeader_2.54mm:PinHeader_1x02_P2.54mm_Vertical -> Connector_PinHeader_2.54mm:PinHeader_1x04_P2.54mm_Vertical
- J42, J60: value Conn_01x04_Pin -> Conn_01x02_Pin; footprint Connector_PinHeader_2.54mm:PinHeader_1x04_P2.54mm_Vertical -> Connector_PinHeader_1.27mm:PinHeader_1x02_P1.27mm_Vertical
- J46: value Conn_01x02_Pin -> Conn_01x06_Pin; footprint Connector_PinHeader_1.27mm:PinHeader_1x02_P1.27mm_Vertical -> Connector_PinHeader_2.54mm:PinHeader_1x06_P2.54mm_Vertical
- J49, J65: value Conn_01x06_Pin -> Conn_01x04_Pin; footprint Connector_PinHeader_2.54mm:PinHeader_1x06_P2.54mm_Vertical -> Connector_PinHeader_2.54mm:PinHeader_1x04_P2.54mm_Vertical
- J54: value Conn_01x02_Pin -> Conn_01x07_Pin; footprint Connector_PinHeader_1.27mm:PinHeader_1x02_P1.27mm_Vertical -> Connector_PinHeader_2.54mm:PinHeader_1x07_P2.54mm_Vertical
- J62: footprint Connector_PinHeader_1.27mm:PinHeader_1x02_P1.27mm_Vertical -> Connector_PinHeader_2.54mm:PinHeader_1x02_P2.54mm_Vertical
- J64: value Conn_01x02_Pin -> Conn_01x06_Pin; footprint Connector_PinHeader_2.54mm:PinHeader_1x02_P2.54mm_Vertical -> Connector_PinHeader_2.54mm:PinHeader_1x06_P2.54mm_Vertical
- J72: value Conn_01x02_Pin -> Conn_01x07_Pin; footprint Connector_PinHeader_2.54mm:PinHeader_1x02_P2.54mm_Vertical -> Connector_PinHeader_2.54mm:PinHeader_1x07_P2.54mm_Vertical
- J9: value Conn_01x06_Pin -> Conn_01x07_Pin; footprint Connector_PinHeader_2.54mm:PinHeader_1x06_P2.54mm_Vertical -> Connector_PinHeader_2.54mm:PinHeader_1x07_P2.54mm_Vertical
- moved J9 97.6 mm to (145.9, 129.4)
- moved J51 94.1 mm to (83.3, 99.1), turned to 180 degrees
- moved J36 85.8 mm to (95.9, 69.4)
- moved J35 84.3 mm to (92.9, 70.5), turned to -90 degrees
- moved J68 82.8 mm to (98.9, 110.0)
- moved J69 80.4 mm to (83.3, 119.1), turned to 180 degrees
- moved J52 79.3 mm to (102.3, 90.0)
- moved J57 78.9 mm to (162.7, 90.0)
- moved J71 73.9 mm to (92.9, 110.5), turned to -90 degrees
- moved J53 70.5 mm to (92.9, 90.5), turned to -90 degrees
- moved J25 69.0 mm to (152.3, 50.0)
- moved J18 68.1 mm to (95.9, 49.4)
- moved J41 65.8 mm to (148.9, 70.0)
- moved J50 65.1 mm to (98.9, 90.0)
- moved J34 61.6 mm to (102.3, 70.0)
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Connections:
- J10 pad 2: 5V -> GND
- J10 pad 3: CE -> SDA_0
- J10 pad 4: GND -> SCL_0
- J11 pad 1: Net-(D1-K) -> +3.3V
- J12 pad 1: CC1 -> Net-(D1-K)
- J12 pad 2: CC2 -> 5V
- J13 pad 1: Net-(J5-A) -> CC1
- J13 pad 2: +3.3V -> CC2
- J14 pad 1: Net-(J6-Pin_1) -> Net-(J5-A)
- J14 pad 2: Net-(J6-Pin_2) -> +3.3V
- J15 pad 1: +3.3V -> Net-(J6-Pin_1)
- J15 pad 2: Net-(J7-B) -> Net-(J6-Pin_2)
- J16 pad 1: Net-(J8-Pin_1) -> +3.3V
- J16 pad 2: Net-(J8-Pin_2) -> Net-(J7-B)
- J17 pad 1: +3.3V -> Net-(J8-Pin_1)
- J17 pad 2: GND -> Net-(J8-Pin_2)
- J18 pad 2: 5V -> +3.3V
- J18 pad 3: CE -> 5V
- J18 pad 4: GND -> 5V
- J19 pad 1: Net-(D1-K) -> +3.3V
- J19 pad 2: 5V -> GND
- J20 pad 1: CC1 -> +3.3V
- J20 pad 2: CC2 -> 5V
- J20 pad 3: D+ -> CE
- J20 pad 4: D- -> GND
- J21 pad 1: Net-(J5-A) -> Net-(D1-K)
- J21 pad 2: +3.3V -> 5V
- J22 pad 1: Net-(J6-Pin_1) -> CC1
- J22 pad 2: Net-(J6-Pin_2) -> CC2
- J23 pad 1: +3.3V -> Net-(J5-A)
- J23 pad 2: Net-(J7-B) -> +3.3V
- J24 pad 1: Net-(J8-Pin_1) -> Net-(J6-Pin_1)
- J24 pad 2: Net-(J8-Pin_2) -> Net-(J6-Pin_2)
- J25 pad 2: GND -> Net-(J7-B)
- J26 pad 1: +3.3V -> Net-(J8-Pin_1)
- J26 pad 2: 5V -> Net-(J8-Pin_2)
- J27 pad 1: Net-(D1-K) -> +3.3V
- J27 pad 2: 5V -> +3.3V
- J28 pad 1: CC1 -> +3.3V
- J28 pad 2: CC2 -> GND
- J28 pad 3: D+ -> SDA_0
- J28 pad 4: D- -> SCL_0
- J29 pad 1: Net-(J5-A) -> +3.3V
- J29 pad 2: +3.3V -> 5V
- J30 pad 1: Net-(J6-Pin_1) -> Net-(D1-K)
- J30 pad 2: Net-(J6-Pin_2) -> 5V
- J31 pad 1: +3.3V -> CC1
- J31 pad 2: Net-(J7-B) -> CC2
- J32 pad 1: Net-(J8-Pin_1) -> Net-(J5-A)
- J32 pad 2: Net-(J8-Pin_2) -> +3.3V
- J33 pad 1: +3.3V -> Net-(J6-Pin_1)
- J33 pad 2: GND -> Net-(J6-Pin_2)
- J34 pad 2: 5V -> Net-(J7-B)
- J35 pad 1: Net-(D1-K) -> Net-(J8-Pin_1)
- J35 pad 2: 5V -> Net-(J8-Pin_2)
- J36 pad 1: CC1 -> +3.3V
- J36 pad 2: CC2 -> +3.3V
- J36 pad 3: D+ -> 5V
- J36 pad 4: D- -> 5V
- J37 pad 1: Net-(J5-A) -> +3.3V
- J37 pad 2: +3.3V -> GND
- J38 pad 1: Net-(J6-Pin_1) -> +3.3V
- J38 pad 2: Net-(J6-Pin_2) -> 5V
- J39 pad 1: +3.3V -> Net-(D1-K)
- J39 pad 2: Net-(J7-B) -> 5V
- J40 pad 1: Net-(J8-Pin_1) -> CC1
- J40 pad 2: Net-(J8-Pin_2) -> CC2
- J41 pad 1: +3.3V -> Net-(J5-A)
- J41 pad 2: GND -> +3.3V
- J42 pad 1: +3.3V -> Net-(J6-Pin_1)
- J42 pad 2: 5V -> Net-(J6-Pin_2)
- J43 pad 1: Net-(D1-K) -> +3.3V
- J43 pad 2: 5V -> Net-(J7-B)
- J44 pad 1: CC1 -> Net-(J8-Pin_1)
- J44 pad 2: CC2 -> Net-(J8-Pin_2)
- J45 pad 1: Net-(J5-A) -> +3.3V
- J46 pad 1: Net-(J6-Pin_1) -> +3.3V
- J46 pad 2: Net-(J6-Pin_2) -> GND
- J47 pad 2: Net-(J7-B) -> 5V
- J48 pad 1: Net-(J8-Pin_1) -> Net-(D1-K)
- J48 pad 2: Net-(J8-Pin_2) -> 5V
- J49 pad 1: +3.3V -> CC1
- J49 pad 2: GND -> CC2
- J49 pad 3: SDA_0 -> D+
- J49 pad 4: SCL_0 -> D-
- J50 pad 1: +3.3V -> Net-(J5-A)
- J50 pad 2: 5V -> +3.3V
- J51 pad 1: Net-(D1-K) -> Net-(J6-Pin_1)
- J51 pad 2: 5V -> Net-(J6-Pin_2)
- J52 pad 1: CC1 -> +3.3V
- J52 pad 2: CC2 -> Net-(J7-B)
- J53 pad 1: Net-(J5-A) -> Net-(J8-Pin_1)
- J53 pad 2: +3.3V -> Net-(J8-Pin_2)
- J54 pad 1: Net-(J6-Pin_1) -> +3.3V
- J54 pad 2: Net-(J6-Pin_2) -> +3.3V
- J55 pad 2: Net-(J7-B) -> GND
- J56 pad 1: Net-(J8-Pin_1) -> +3.3V
- J56 pad 2: Net-(J8-Pin_2) -> 5V
- J57 pad 1: +3.3V -> Net-(D1-K)
- J57 pad 2: GND -> 5V
- J58 pad 1: +3.3V -> CC1
- J58 pad 2: 5V -> CC2
- J58 pad 3: CE -> D+
- J58 pad 4: GND -> D-
- J59 pad 1: Net-(D1-K) -> Net-(J5-A)
- J59 pad 2: 5V -> +3.3V
- J60 pad 1: CC1 -> Net-(J6-Pin_1)
- J60 pad 2: CC2 -> Net-(J6-Pin_2)
- J61 pad 1: Net-(J5-A) -> +3.3V
- J61 pad 2: +3.3V -> Net-(J7-B)
- J62 pad 1: Net-(J6-Pin_1) -> Net-(J8-Pin_1)
- J62 pad 2: Net-(J6-Pin_2) -> Net-(J8-Pin_2)
- J63 pad 2: Net-(J7-B) -> +3.3V
- J64 pad 1: Net-(J8-Pin_1) -> +3.3V
- J64 pad 2: Net-(J8-Pin_2) -> GND
- J65 pad 2: GND -> 5V
- J65 pad 3: SDA_0 -> CE
- J65 pad 4: SCL_0 -> GND
- J66 pad 1: +3.3V -> Net-(D1-K)
- J67 pad 1: Net-(D1-K) -> CC1
- J67 pad 2: 5V -> CC2
- J68 pad 1: CC1 -> Net-(J5-A)
- J68 pad 2: CC2 -> +3.3V
- J69 pad 1: Net-(J5-A) -> Net-(J6-Pin_1)
- J69 pad 2: +3.3V -> Net-(J6-Pin_2)
- J70 pad 1: Net-(J6-Pin_1) -> +3.3V
- J70 pad 2: Net-(J6-Pin_2) -> Net-(J7-B)
- J71 pad 1: +3.3V -> Net-(J8-Pin_1)
- J71 pad 2: Net-(J7-B) -> Net-(J8-Pin_2)
- J72 pad 1: Net-(J8-Pin_1) -> +3.3V
- J72 pad 2: Net-(J8-Pin_2) -> +3.3V
- J9 pad 2: GND -> +3.3V
- J9 pad 3: SDA_0 -> 5V
- J9 pad 4: SCL_0 -> 5V
- J9 pad 5: ADDR -> Net-(J8-Pin_1)
- J9 pad 6: unconnected-(J1-Pin_6-Pad6) -> GND
Routing:
- net +3.3V: track 458.9 -> 517.0 mm
- net 5V: track 277.1 -> 311.5 mm
- net GND: track 297.6 -> 324.5 mm
- net Net-(J8-Pin_1): track 177.0 -> 196.2 mm
Other:
- outline, holes or cut-outs redrawn
