File: Version2/Bus-Breakout/RAIL-Devices.kicad_pcb (KiCad board)
At the start: 2 copper layers, 99.8 x 19.5 mm, 33 parts, among them J2 Conn_01x30_Pin, J5 Conn_02x30_Odd_Even, P1 Jumper4x1, P10 Jumper4x1, P11 Jumper4x1, P12 Jumper4x1, P13 Jumper4x1, P14 Jumper4x1, P15 Jumper4x1, P16 Jumper4x1, P17 Jumper4x1, P18 Jumper4x1, P19 Jumper4x1, P2 Jumper4x1, P20 Jumper4x1, P21 Jumper4x1, P22 Jumper4x1, P23 Jumper4x1, P24 Jumper4x1, P25 Jumper4x1, P26 Jumper4x1, P27 Jumper4x1, P28 Jumper4x1, P29 Jumper4x1, P3 Jumper4x1, P30 Jumper4x1, P4 Jumper4x1, P5 Jumper4x1, P6 Jumper4x1, P7 Jumper4x1, P8 Jumper4x1, P9 Jumper4x1

Commit message: update stuff.
Parts:
- moved G*** 8.33 mm to (153.4, 106.0)
Routing:
- net /JA1: track 138.2 -> 171.2 mm
- net /JA2: track 135.6 -> 163.0 mm
- net /JA4: track 134.0 -> 159.8 mm, vias 30 -> 31
- net /JA3: track 133.8 -> 157.7 mm
- net P30: track 19.1 -> 20.2 mm
Other:
- board text added: "IOT_Mess Bus-Breakout V2.0 8/19/25"
- board text removed: "IOT_Mess Bus-Breakout V1.2 8/12/25"

Commit message: updates.
Parts:
- added J3: Conn_02x38_Odd_Even, Connector_PinSocket_2.54mm:PinSocket_2x38_P2.54mm_Vertical, F.Cu at (110.5, 44.9)
- added J4: Conn_01x38_Pin, Connector_PinSocket_2.54mm:PinSocket_1x38_P2.54mm_Vertical, F.Cu at (104.0, 44.9)
- moved P3 87.5 mm to (115.8, 45.1), turned to 90 degrees
- moved P4 85.3 mm to (126.1, 45.3), turned to 90 degrees
- moved P2 81.9 mm to (115.8, 49.1), turned to 90 degrees
- moved P5 79.7 mm to (126.1, 49.3), turned to 90 degrees
- moved P1 76.4 mm to (115.8, 53.1), turned to 90 degrees
- moved P6 74.0 mm to (126.1, 53.3), turned to 90 degrees
- moved J2 71.6 mm to (116.4, 56.5), turned to 0 degrees
- moved J5 70.1 mm to (121.5, 56.5), turned to 0 degrees
- moved P7 68.4 mm to (126.1, 57.3), turned to 90 degrees
- moved P8 62.7 mm to (126.1, 61.3), turned to 90 degrees
- moved P9 57.1 mm to (126.1, 65.3), turned to 90 degrees
- moved P30 51.5 mm to (115.9, 139.7), turned to 90 degrees
- moved P10 51.4 mm to (126.1, 69.3), turned to 90 degrees
- moved P28 48.8 mm to (126.1, 140.0), turned to 90 degrees
- moved P29 46.4 mm to (115.8, 135.8), turned to 90 degrees
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Routing:
- net /B9: track 0.00 -> 6.54 mm
- net /B8: track 0.00 -> 6.54 mm
- net /B7: track 0.00 -> 6.54 mm
- net /B6: track 0.00 -> 6.54 mm
- net /B5: track 0.00 -> 6.54 mm
- net /B4: track 0.00 -> 6.54 mm
- net /B38: track 0.00 -> 6.54 mm
- net /B37: track 0.00 -> 6.54 mm
- net /B36: track 0.00 -> 6.54 mm
- net /B35: track 0.00 -> 6.54 mm
- net /B34: track 0.00 -> 6.54 mm
- net /B33: track 0.00 -> 6.54 mm
- net /B32: track 0.00 -> 6.54 mm
- net /B31: track 0.00 -> 6.54 mm
- net /B30: track 0.00 -> 6.54 mm
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Other:
- board size 99.8 x 19.5 mm -> 31.9 x 99.8 mm

Commit message: updates.
Other:
- outline, holes or cut-outs redrawn
- board text added: "1"
- board text added: "10"
- board text added: "11"
- board text added: "12"
- board text added: "13"
- board text added: "14"
- board text added: "15"
- board text added: "16"
- board text added: "17"
- board text added: "18"
- board text added: "19"
- board text added: "2"
- board text added: "20"
- board text added: "21"
- board text added: "22"
- board text added: "23"
- board text added: "24"
- board text added: "25"
- board text added: "26"
- board text added: "27"
- board text added: "28"
- board text added: "29"
- board text added: "3"
- board text added: "30"
- board text added: "31"
- board text added: "32"
- board text added: "33"
- board text added: "34"
- board text added: "35"
- board text added: "36"
- board text added: "37"
- board text added: "38"
- board text added: "4"
- board text added: "5"
- board text added: "6"
- board text added: "7"
- board text added: "8"
- board text added: "9"

Commit message: update.
Parts:
- added J1: Conn_01x38_Pin, Connector_PinSocket_2.54mm:PinSocket_1x38_P2.54mm_Vertical, F.Cu at (113.1, 44.9)
- moved J3 0.50 mm to (110.0, 44.9)
- moved J4 0.50 mm to (103.5, 44.9)
Connections:
- J3 pad 11: /B6 -> P2
- J3 pad 12: /B6 -> P2
- J3 pad 13: /B7 -> P3
- J3 pad 14: /B7 -> P3
- J3 pad 15: /B8 -> P4
- J3 pad 16: /B8 -> P4
- J3 pad 17: /B9 -> P5
- J3 pad 18: /B9 -> P5
- J3 pad 19: /B10 -> P6
- J3 pad 20: /B10 -> P6
- J3 pad 21: /B11 -> P7
- J3 pad 22: /B11 -> P7
- J3 pad 23: /B12 -> P8
- J3 pad 24: /B12 -> P8
- J3 pad 25: /B13 -> P9
- J3 pad 26: /B13 -> P9
- J3 pad 27: /B14 -> P10
- J3 pad 28: /B14 -> P10
- J3 pad 29: /B15 -> P11
- J3 pad 30: /B15 -> P11
- J3 pad 31: /B16 -> P12
- J3 pad 32: /B16 -> P12
- J3 pad 33: /B17 -> P13
- J3 pad 34: /B17 -> P13
- J3 pad 35: /B18 -> P14
- J3 pad 36: /B18 -> P14
- J3 pad 37: /B19 -> P15
- J3 pad 38: /B19 -> P15
- J3 pad 39: /B20 -> P16
- J3 pad 40: /B20 -> P16
- J3 pad 41: /B21 -> P17
- J3 pad 42: /B21 -> P17
- J3 pad 43: /B22 -> P18
- J3 pad 44: /B22 -> P18
- J3 pad 45: /B23 -> P19
- J3 pad 46: /B23 -> P19
- J3 pad 47: /B24 -> P20
- J3 pad 48: /B24 -> P20
- J3 pad 49: /B25 -> P21
- J3 pad 50: /B25 -> P21
- J3 pad 51: /B26 -> P22
- J3 pad 52: /B26 -> P22
- J3 pad 53: /B27 -> P23
- J3 pad 54: /B27 -> P23
- J3 pad 55: /B28 -> P24
- J3 pad 56: /B28 -> P24
- J3 pad 57: /B29 -> P25
- J3 pad 58: /B29 -> P25
- J3 pad 59: /B30 -> P26
- J3 pad 60: /B30 -> P26
- J3 pad 61: /B31 -> P27
- J3 pad 62: /B31 -> P27
- J3 pad 63: /B32 -> P28
- J3 pad 64: /B32 -> P28
- J3 pad 65: /B33 -> P29
- J3 pad 66: /B33 -> P29
- J3 pad 67: /B34 -> P30
- J3 pad 68: /B34 -> P30
- J4 pad 10: /B10 -> P6
- J4 pad 11: /B11 -> P7
- J4 pad 12: /B12 -> P8
- J4 pad 13: /B13 -> P9
- J4 pad 14: /B14 -> P10
- J4 pad 15: /B15 -> P11
- J4 pad 16: /B16 -> P12
- J4 pad 17: /B17 -> P13
- J4 pad 18: /B18 -> P14
- J4 pad 19: /B19 -> P15
- J4 pad 20: /B20 -> P16
- J4 pad 21: /B21 -> P17
- J4 pad 22: /B22 -> P18
- J4 pad 23: /B23 -> P19
- J4 pad 24: /B24 -> P20
- J4 pad 25: /B25 -> P21
- J4 pad 26: /B26 -> P22
- J4 pad 27: /B27 -> P23
- J4 pad 28: /B28 -> P24
- J4 pad 29: /B29 -> P25
- J4 pad 30: /B30 -> P26
- J4 pad 31: /B31 -> P27
- J4 pad 32: /B32 -> P28
- J4 pad 33: /B33 -> P29
- J4 pad 34: /B34 -> P30
- J4 pad 6: /B6 -> P2
- J4 pad 7: /B7 -> P3
- J4 pad 8: /B8 -> P4
- J4 pad 9: /B9 -> P5
Routing:
- net P30: track 20.2 -> 33.9 mm
- net P8: track 22.2 -> 35.8 mm
- net P17: track 11.9 -> 25.5 mm
- net P26: track 22.4 -> 36.0 mm
- net P29: track 17.7 -> 31.3 mm
- net P6: track 26.6 -> 40.2 mm
- net P4: track 29.5 -> 43.1 mm
- net P22: track 16.9 -> 30.5 mm
- net P2: track 19.2 -> 32.8 mm
- net P15: track 14.0 -> 27.6 mm
- net P13: track 16.6 -> 30.2 mm
- net P7: track 25.2 -> 38.8 mm
- net P24: track 20.1 -> 33.7 mm
- net P27: track 23.9 -> 37.5 mm
- net P23: track 20.2 -> 33.8 mm
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Other:
- outline, holes or cut-outs redrawn
