File: Version2/LED-74HC595/LED-74HC595.kicad_pcb (KiCad board)
At the start: 2 copper layers, 29.5 x 49.5 mm, 5 parts, among them J1 Conn_01x08_Pin, J2 Conn_01x08_Pin, J3 Conn_02x08_Odd_Even, U2 74HC595, U3 74HC595

Commit message: update.
Parts:
- removed the J3 at (136.5, 63.1)
- added C1: .1u, Capacitor_SMD:C_0603_1608Metric, F.Cu at (143.0, 91.3)
- added D1: LED, LED_SMD:LED_0603_1608Metric, F.Cu at (143.3, 106.9)
- added G***: LOGO, IOT-Mess-Footprints:catIcon8x8, B.Cu at (151.1, 95.5)
- added J2: Conn_02x19_Odd_Even, Connector_PinHeader_2.54mm:PinHeader_2x19_P2.54mm_Vertical, F.Cu at (136.5, 62.5)
- added R1: R, Resistor_SMD:R_0603_1608Metric, F.Cu at (143.3, 103.9)
- added SW1: SW_Push, Button_Switch_SMD:SW_SPST_PTS810, F.Cu at (143.3, 96.4)
- added U1: ~, Package_SO:TSSOP-20_4.4x6.5mm_P0.65mm, F.Cu at (150.2, 79.5)
- added U4: 74HC595, Package_SO:SOP-16_3.9x9.9mm_P1.27mm, F.Cu at (150.2, 67.6)
- J1: value Conn_01x08_Pin -> Conn_01x10_Pin; footprint Connector_PinHeader_2.54mm:PinHeader_1x08_P2.54mm_Vertical -> Connector_PinHeader_2.54mm:PinHeader_1x10_P2.54mm_Vertical
- moved J1 35.9 mm to (159.3, 62.5)
- moved U2 12.4 mm to (150.2, 91.2), turned to 0 degrees
- moved U3 11.9 mm to (150.1, 103.6), turned to 0 degrees
- moved J3 0.16 mm to (161.0, 90.4)
- renumbered J2 to J3
Connections:
- J1 pad 1: C7 -> GND
- J1 pad 2: C6 -> VCC
- J1 pad 3: R1 -> CLCK
- J1 pad 4: C0 -> LATCH
- J1 pad 5: R3 -> Net-(J1-Pin_5)
- J1 pad 6: C5 -> VCC
- J1 pad 7: C3 -> GND
- J1 pad 8: R0 -> SWIO
- J3 pad 1: R4 -> R0
- J3 pad 2: R6 -> R1
- J3 pad 3: C1 -> R2
- J3 pad 4: C2 -> R3
- J3 pad 5: R7 -> R4
- J3 pad 6: C4 -> R5
- J3 pad 7: R5 -> R6
- J3 pad 8: R2 -> R7
- U2 pad 10: unconnected-(U2-~{SRCLR}-Pad10) -> VCC
- U2 pad 13: EN_B -> EN_R
- U2 pad 9: unconnected-(U2-QH&apos;-Pad9) -> Net-(U2-QH')
- U3 pad 10: unconnected-(U3-~{SRCLR}-Pad10) -> VCC
- U3 pad 14: DATA -> Net-(U2-QH')
- U3 pad 9: unconnected-(U3-QH&apos;-Pad9) -> Net-(U3-QH')
Routing:
- net CLCK: track 0.00 -> 56.1 mm, vias 0 -> 6
- net LATCH: track 0.00 -> 53.1 mm, vias 0 -> 5
- net EN_C: track 0.00 -> 50.9 mm, vias 0 -> 1
- net EN_R: track 0.00 -> 50.1 mm, vias 0 -> 3
- net C1: track 63.4 -> 13.7 mm
- net Net-(U3-QH'): track 0.00 -> 49.6 mm
- net C2: track 59.0 -> 13.2 mm, vias 2 -> 1
- net C3: track 57.8 -> 12.7 mm, vias 3 -> 1
- net C4: track 55.1 -> 12.1 mm, vias 2 -> 1
- net C5: track 48.7 -> 11.6 mm, vias 3 -> 1
- net EN_A: track 0.00 -> 31.8 mm, vias 0 -> 3
- net C0: track 48.0 -> 22.0 mm
- net Net-(U1-PD7/RST): track 0.00 -> 23.9 mm, vias 0 -> 2
- net C6: track 34.8 -> 11.2 mm, vias 0 -> 1
- net R2: track 68.4 -> 46.6 mm
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- added copper zone on B.Cu, net VCC
Other:
- board text added: "A0"
- board text added: "A1"
- board text added: "A2"
- board text added: "A3"
- board text added: "A4"
- board text added: "A5"
- board text added: "A6"
- board text added: "A7"
- board text added: "C0"
- board text added: "C1"
- board text added: "C2"
- board text added: "C3"
- board text added: "C4"
- board text added: "C5"
- board text added: "C6"
- board text added: "C7"
- board text added: "EA"
- board text added: "EC"
- board text added: "ER"
- board text added: "G"
- board text added: "IOT_Mess LED595 V2.0 8/19/25"
- board text added: "R0"
- board text added: "R1"
- board text added: "R2"
- board text added: "R3"
- board text added: "R4"
- board text added: "R5"
- board text added: "R6"
- board text added: "R7"
- board text added: "SA"
- board text added: "SL"
- board text added: "SW"
- board text added: "V"
