File: Version2/LED-CharliePlexing1/LED-CharliePlexing1.kicad_pcb (KiCad board)
At the start: 2 copper layers, 32.6 x 49.6 mm, 139 parts, among them J1 Conn_02x19_Odd_Even, J12 Jumper, J2 Jumper, J3 Jumper, J4 Jumper, J5 Jumper, J6 Jumper, J7 Jumper, J8 Jumper

Commit message: update stuff.
Parts:
- added G***: LOGO, IOT-Mess-Footprints:catIcon8x8, B.Cu at (144.2, 109.4)
Other:
- board text added: "IOT_Mess Charlieplexing V2.0 8/19/25"

Commit message: update.
Parts:
- added J9: Conn_01x19_Pin, Connector_PinHeader_2.54mm:PinHeader_1x19_P2.54mm_Vertical, F.Cu at (120.6, 71.2)
Connections:
- net /P10 renamed /A_4
- net /P12 renamed /A_5
- net /P14 renamed /A_6
- net /P16 renamed /A_7
- net /P2 renamed /A_0
- net /P24 renamed /C0
- net /P26 renamed /C1
- net /P28 renamed /C2
- net /P30 renamed /C3
- net /P32 renamed /C4
- net /P34 renamed /C5
- net /P36 renamed /C6
- net /P38 renamed /C7
- net /P4 renamed /A_1
- net /P6 renamed /A_2
- net /P8 renamed /A_3
Routing:
- net /C0: track 18.7 -> 21.6 mm
- net /P22: track 12.5 -> 15.3 mm
- net /P20: track 18.4 -> 21.3 mm
- net /P18: track 12.2 -> 15.1 mm
- net /C7: track 33.5 -> 36.3 mm
- net /C6: track 20.2 -> 23.1 mm
- net /C4: track 19.4 -> 22.2 mm
- net /C2: track 18.7 -> 21.6 mm
- net /C1: track 13.0 -> 15.8 mm
- net /A_7: track 20.6 -> 23.5 mm
- net /A_6: track 9.93 -> 12.8 mm
- net /A_3: track 14.8 -> 17.6 mm
- net /A_2: track 8.67 -> 11.5 mm
- net /A_1: track 15.3 -> 18.2 mm
- net /A_0: track 9.74 -> 12.6 mm
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Other:
- board size 32.6 x 49.6 mm -> 35.1 x 49.6 mm
