File: Version2/LED-CharliePlexing1/LED-CharliePlexing1.kicad_sch (KiCad schematic)
At the start: 139 parts, among them J1 Conn_02x19_Odd_Even, J12 Jumper, J2 Jumper, J3 Jumper, J4 Jumper, J5 Jumper, J6 Jumper, J7 Jumper, J8 Jumper

Commit message: update.
Parts:
- added J9: Conn_01x19_Pin, Connector_PinHeader_2.54mm:PinHeader_1x19_P2.54mm_Vertical, symbol Connector:Conn_01x19_Pin
Connections:
- net P18: now also J9.9 (Pin_9)
- net P20: now also J9.10 (Pin_10)
- net P22: now also J9.11 (Pin_11)
- net P10 renamed A_4
- net A_4: now also J9.5 (Pin_5)
- net P12 renamed A_5
- net A_5: now also J9.6 (Pin_6)
- net P14 renamed A_6
- net A_6: now also J9.7 (Pin_7)
- net P16 renamed A_7
- net A_7: now also J9.8 (Pin_8)
- net P2 renamed A_0
- net A_0: now also J9.1 (Pin_1)
- net P24 renamed C0
- net C0: now also J9.12 (Pin_12)
- net P26 renamed C1
- net C1: now also J9.13 (Pin_13)
- net P28 renamed C2
- net C2: now also J9.14 (Pin_14)
- net P30 renamed C3
- net C3: now also J9.15 (Pin_15)
- net P32 renamed C4
- net C4: now also J9.16 (Pin_16)
- net P34 renamed C5
- net C5: now also J9.17 (Pin_17)
- net P36 renamed C6
- net C6: now also J9.18 (Pin_18)
- net P38 renamed C7
- net C7: now also J9.19 (Pin_19)
- net P4 renamed A_1
- net A_1: now also J9.2 (Pin_2)
- net P6 renamed A_2
- net A_2: now also J9.3 (Pin_3)
- net P8 renamed A_3
- net A_3: now also J9.4 (Pin_4)
