File: Version2/Mess-Sens/IOT-Mess-Base.kicad_sch (KiCad schematic)
At the start: 45 parts, among them IC1 SHT40I-AD1F-R2, J1 Conn_01x02_Pin, J2 TP_4056, J4 Conn_01x12_Pin, Q1 NM8205 PFETs, Q5 AO3401A, SW4 SW_Push, SW5 SW_Push, U1 TPL5110, U10 OPT3001DNPR, U11 HDC2010/DSBGA-6, U12 MMC5633NJL/WLP-4, U13 BH1750FVI-TR, U14 T117W, U15 DS1307Z+, U16 ENS210, U17 LIS2MDL, U19 MTS4, U2 INA219AxDCN, U3 TLV493D, U4 INA219AxD, U5 SHT31-DIS, U6 APDS-9960, U7 QMC6309/WLCSP-4, U8 AND_Gate, U9 LTR-303ALS-01

Commit message: updated.
Parts:
- removed C10, C11: .1u, Capacitor_SMD:C_0603_1608Metric, symbol Device:C
- removed C8: .22u, Capacitor_SMD:C_0603_1608Metric, symbol Device:C
- removed C9: 10u, Capacitor_SMD:C_0603_1608Metric, symbol Device:C
- removed U17: LIS2MDL, Package_LGA:LGA-12_2x2mm_P0.5mm, symbol Sensor_Magnetic:LIS2MDL
- U8: value AND_Gate -> SN74LVC1 (AND GATE)
Connections:
- no-connect marks 11 -> 10
Other:
- moved on the sheet: C3, C4, C5, J1, J2, J4, R10, R11, R9, U10, U11, U12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

Commit message: did some works.
Parts:
- removed C6, C7: 0.1u, Capacitor_SMD:C_0603_1608Metric, symbol Device:C
- removed J2: TP_4056, IOT-Mess-Footprints:TP_Charger, symbol Connector:Conn_01x04_Pin
- removed J4: Conn_01x12_Pin, Connector_PinHeader_2.54mm:PinHeader_1x12_P2.54mm_Vertical, symbol Connector:Conn_01x12_Pin
- removed Q1: NM8205 PFETs, Package_TO_SOT_SMD:SOT-23-6, symbol Transistor_FET:DMG9926UDM
- removed Q5: AO3401A, Package_TO_SOT_SMD:SOT-23, symbol Transistor_FET:AO3401A
- removed R19, R2, R20, R21, R7: R, Resistor_SMD:R_0603_1608Metric, symbol Device:R
- removed R4: 0.1R, Resistor_SMD:R_2512_6332Metric, symbol Device:R
- removed SW4, SW5: SW_Push, Button_Switch_SMD:SW_SPST_PTS810, symbol Switch:SW_Push
- removed U1: TPL5110, Package_TO_SOT_SMD:SOT-23-6, symbol Timer:TPL5110
- removed U2: INA219AxDCN, Package_TO_SOT_SMD:SOT-23-8, symbol Sensor_Energy:INA219AxDCN
- removed U4: INA219AxD, Package_SO:SOIC-8_3.9x4.9mm_P1.27mm, symbol Sensor_Energy:INA219AxD
- removed U8: SN74LVC1 (AND GATE), Sensor:Avago_APDS-9960, symbol IOT-Mess:AND_Gate
- added J2: Conn_01x06_Pin, Connector_PinHeader_2.54mm:PinHeader_1x06_P2.54mm_Vertical, symbol Connector:Conn_01x06_Pin
- added U1: TMP102xxDRL, Package_TO_SOT_SMD:SOT-563, symbol Sensor_Temperature:TMP102xxDRL
- added U4: TMP1075DGK, Package_SO:VSSOP-8_3x3mm_P0.65mm, symbol Sensor_Temperature:TMP1075DGK
- C3: value 0.1u -> 0.1uF
- C4: value 1u -> 1uF
- J1: footprint (none) -> Connector_PinHeader_1.27mm:PinHeader_1x02_P1.27mm_Vertical
- R1: value R -> 10K
Connections:
- net +3.3V: now also J2.1 (Pin_1), U1.5 (V+), U4.8 (V+)
- net ADDR: now also J2.5 (Pin_5), U1.4 (ADD0)
- net GND: now also U14.7 (GND), J2.2 (Pin_2), U1.2 (GND), U4.3 (ALERT), U4.4 (GND); no longer R1.1
- net SCL_0: now also R10.1, J2.4 (Pin_4), U1.1 (SCL), U4.1 (SDA); no longer R11.2
- net SDA_0: now also R11.2, J2.3 (Pin_3), U1.6 (SDA), U4.2 (SCL); no longer R10.1
- net DONE: no longer names the net of R1.2
- net DONE: now also U4.5 (A2), U4.6 (A1), U4.7 (A0)
- no-connect marks 10 -> 11
Other:
- moved on the sheet: C3, C4, C5, IC1, J1, R10, R11, R9, U10, U11, U12, U13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

Commit message: update stuff.
Changed lines of the file:
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@@
 	(wire
 		(pts
-			(xy 80.01 146.05) (xy 80.01 149.86)
+			(xy 78.74 142.24) (xy 78.74 149.86)
 		)
 		(stroke
@@
 	(wire
 		(pts
-			(xy 69.85 149.86) (xy 80.01 149.86)
+			(xy 69.85 149.86) (xy 78.74 149.86)
 		)
 		(stroke
@@
 	(wire
 		(pts
-			(xy 69.85 147.32) (xy 69.85 149.86)
+			(xy 69.85 142.24) (xy 69.85 149.86)
 		)
 		(stroke
@@
 	(symbol
 		(lib_id "power:+3.3V")
-		(at 69.85 147.32 0)
+		(at 69.85 142.24 0)
 		(unit 1)
 		(exclude_from_sim no)
@@
 		(dnp no)
 		(property "Reference" "#PWR015"
-			(at 69.85 151.13 0)
+			(at 69.85 146.05 0)
 			(effects
 				(font
@@
 		)
 		(property "Value" "+3.3V"
-			(at 69.596 143.256 0)
+			(at 69.596 138.176 0)
 			(effects
 				(font
@@
 		)
 		(property "Footprint" ""
-			(at 69.85 147.32 0)
+			(at 69.85 142.24 0)
 			(effects
 				(font
@@
 		)
 		(property "Datasheet" ""
-			(at 69.85 147.32 0)
+			(at 69.85 142.24 0)
 			(effects
 				(font
@@
 		)
 		(property "Description" ""
-			(at 69.85 147.32 0)
+			(at 69.85 142.24 0)
 			(effects
 				(font
@@
 	(symbol
 		(lib_id "power:PWR_FLAG")
-		(at 80.01 146.05 0)
+		(at 78.74 142.24 0)
 		(unit 1)
 		(exclude_from_sim no)
@@
 		(dnp no)
 		(property "Reference" "#FLG02"
-			(at 80.01 144.145 0)
+			(at 78.74 140.335 0)
 			(effects
 				(font
@@
 		)
 		(property "Value" "PWR_FLAG"
-			(at 80.01 140.97 0)
+			(at 78.74 137.16 0)
 			(effects
 				(font
@@
 		)
 		(property "Footprint" ""
-			(at 80.01 146.05 0)
+			(at 78.74 142.24 0)
 			(effects
 				(font
@@
 		)
 		(property "Datasheet" "~"
-			(at 80.01 146.05 0)
+			(at 78.74 142.24 0)
 			(effects
 				(font
@@
 		)
 		(property "Description" "Special symbol for telling ERC where power comes from"
-			(at 80.01 146.05 0)
+			(at 78.74 142.24 0)
 			(effects
 				(font

Commit message: updates.
Parts:
- removed U10: OPT3001DNPR, OPT3001DNPR:SON65P200X200X65-7N, symbol OPT300x:OPT3001DNPR
- removed U3: TLV493D, Package_SO:TSOP-6_1.65x3.05mm_P0.95mm, symbol Sensor_Magnetic:TLV493D
- removed U4: TMP1075DGK, Package_SO:VSSOP-8_3x3mm_P0.65mm, symbol Sensor_Temperature:TMP1075DGK
- added C3: 10u, Capacitor_SMD:C_0603_1608Metric, symbol Device:C
- added C4, C7: 1u, Capacitor_SMD:C_0603_1608Metric, symbol Device:C
- added C6: 22nF, Capacitor_SMD:C_0603_1608Metric, symbol Device:C
- added D1: 1N5819WS, Diode_SMD:D_SOD-323, symbol Diode:1N5819WS
- added D2: LED, LED_SMD:LED_0603_1608Metric, symbol Device:LED
- added J2, J4: Conn_01x04_Pin, Connector_PinHeader_2.54mm:PinHeader_1x04_P2.54mm_Vertical, symbol Connector:Conn_01x04_Pin
- added J3, J5, J7: Jumper_2, IOT-Mess-Footprints:Jumpper-triangle, symbol Jumper:Jumper_2_Small_Open
- added J8: Conn_01x02_Pin, Connector_PinHeader_2.54mm:PinHeader_1x02_P2.54mm_Vertical, symbol Connector:Conn_01x02_Pin
- added R2: 0.1, Resistor_SMD:R_1206_3216Metric, symbol Device:R
- added R5, R7: 5.1K, Resistor_SMD:R_0603_1608Metric, symbol Device:R
- added R8: R, Resistor_SMD:R_0603_1608Metric, symbol Device:R
- added TP1: TestPoint, Connector_PinHeader_1.00mm:PinHeader_1x01_P1.00mm_Vertical, symbol Connector:TestPoint
- added U2: LTR-507ALS, IOT-Mess-Footprints:LTR-507ALS, symbol IOT-Mess:LTR-507ALS
- added U3: INA219AxDCN, Package_TO_SOT_SMD:SOT-23-8, symbol Sensor_Energy:INA219AxDCN
- added U4: USB_C_Receptacle_USB2.0_16P, Connector_USB:USB_C_Receptacle_HRO_TYPE-C-31-M-12, symbol Connector:USB_C_Receptacle_USB2.0_16P
- added U8: ME6211C33M5, Package_TO_SOT_SMD:SOT-23-5, symbol Regulator_Linear:ME6211C33M5
- R1: value 10K -> 0.1; footprint Resistor_SMD:R_0603_1608Metric -> Resistor_SMD:R_2512_6332Metric
- U1: renamed from U9; value LTR-303ALS-01 -> LTR-303/308
- U11: renamed from U19; value MTS4 -> MTS4 0.1C DFN-4L
- U12: renamed from U14; value T117W -> T117W 0.1C DFN-6L
- U15: renamed from U1; value TMP102xxDRL -> TMP102xxDRL 0.5C SOT-563
- renumbered C3 to C1, C4 to C2, J2 to J1, J1 to J6, R10 to R3, R11 to R4, R9 to R6, U16 to U10, U7 to U13, U5 to U14, U15 to U16, U13 to U5, U12 to U7, U11 to U9
Connections:
- net +3.3V: now also C7.1, J2.1 (Pin_1), J5.2 (B), J7.1 (A), U2.1 (VCC), U3.4 (VS)
- net ADDR: now also U2.4 (ADDR), U3.7 (A0), U3.8 (A1)
- net GND: now also C3.2, C4.2, C6.2, C7.2, D2.1 (K), J2.4 (Pin_4), R5.2, R7.2, U2.2 (GND), U2.3 (GND_LED), U3.3 (GND), U4.A1 (GND), U4.A12 (GND), U4.B1 (GND), U4.B12 (GND), U4.S1 (SHIELD), U8.2 (V_{SS})
- net SCL_0: now also U2.7 (SCL), U3.5 (SCL)
- net SDA_0: now also U2.8 (SDA), U3.6 (SDA)
- net at R1.1: now also J8.1 (Pin_1), R2.1, U3.1 (IN+)
- net at R1.2: now also J8.2 (Pin_2), R2.2, U3.2 (IN-)
- new net: C6.1, U8.4 (NC)
- new net: D1.1 (K), J3.1 (A), U4.A4 (VBUS), U4.A9 (VBUS), U4.B4 (VBUS), U4.B9 (VBUS)
- new net: J5.1 (A), U8.5 (V_{OUT})
- new net: J7.2 (B), R8.2
- new net: TP1.1, U2.5 (VLED)
- new net: D2.2 (A), R8.1
- new net 5V: C3.1, C4.1, D1.2 (A), J2.2 (Pin_2), J3.2 (B), U8.1 (V_{IN})
- new net CC1: J4.1 (Pin_1), R7.1, U4.A5 (CC1)
- new net CC2: J4.2 (Pin_2), R5.1, U4.B5 (CC2)
- new net CE: J2.3 (Pin_3), U8.3 (CE)
- new net D+: J4.3 (Pin_3), U4.A6 (D+), U4.B6 (D+)
- new net D-: J4.4 (Pin_4), U4.A7 (D-), U4.B7 (D-)
- no-connect marks 11 -> 12
Other:
- note added: "Light Sens."
- note added: "Magnetic Sens."
- note added: "RTC"
- note added: "Temp Sens."
- note added: "Temp/Hum Sens."
- note added: "USB-C POWER"
- moved on the sheet: C1, C2, C5, IC1, J1, J6, R3, R4, R6, U1, U10, U11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

Commit message: update.
Parts:
- added J9: Conn_01x07_Pin, Connector_PinHeader_2.54mm:PinHeader_1x07_P2.54mm_Vertical, symbol Connector:Conn_01x07_Pin
Connections:
- net +3.3V: now also J9.1 (Pin_1), J9.2 (Pin_2)
- net 5V: now also J9.3 (Pin_3), J9.4 (Pin_4)
- net GND: now also J9.6 (Pin_6), J9.7 (Pin_7)
- net at J8.1 (Pin_1), R1.1, R2.1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: now also J9.5 (Pin_5)

Commit message: update.
Other:
- note added: "ADDR->0X41"
- note added: "ADDR->0x30?"
- note added: "ADDR->0x39"
- note added: "ADDR->0x40-0x4F"
- note added: "ADDR->0x7C"
- note added: "ADDR->0xA6"
- note added: "ADDR->GND 0x23 ADDR->VDD 0x5C"
- note added: "ADDR->GND 0x40 ADDR->VDD 0x41"
- note added: "ADDR->GND 0x40 ADDR->VDD 0x41 ADDR->SDA 0x42 ADDR->SCL 0x43"
- note added: "ADDR->GND 0x44 ADDR->VDD 0x45"
- note added: "ADDR->GND 0x48 ADDR->VDD 0x49 ADDR->SDA 0x4A ADDR->SCL 0x4B"
- note added: "ADDR->GND 0x74 ADDR->VDD 0x76 ADDR->Float 0x46"
Changed lines of the file:
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@@
 		)
 	)
+	(text "ADDR->0x40-0x4F"
+		(exclude_from_sim no)
+		(at 278.892 183.896 0)
+		(effects
+			(font
+				(size 1.27 1.27)
+			)
+		)
+	)
 	(text "USB-C POWER"
 		(exclude_from_sim no)
@@
 		)
 	)
+	(text "ADDR->GND 0x40\nADDR->VDD 0x41"
+		(exclude_from_sim no)
+		(at 358.648 73.152 0)
+		(effects
+			(font
+				(size 1.27 1.27)
+			)
+		)
+	)
+	(text "ADDR->GND 0x48\nADDR->VDD 0x49\nADDR->SDA 0x4A\nADDR->SCL 0x4B"
+		(exclude_from_sim no)
+		(at 394.97 156.464 0)
+		(effects
+			(font
+				(size 1.27 1.27)
+			)
+		)
+	)
+	(text "ADDR->0x39"
+		(exclude_from_sim no)
+		(at 277.876 143.002 0)
+		(effects
+			(font
+				(size 1.27 1.27)
+			)
+		)
+	)
+	(text "ADDR->GND 0x44\nADDR->VDD 0x45"
+		(exclude_from_sim no)
+		(at 398.78 72.644 0)
+		(effects
+			(font
+				(size 1.27 1.27)
+			)
+		)
+	)
+	(text "ADDR->0x7C"
+		(exclude_from_sim no)
+		(at 356.362 244.856 0)
+		(effects
+			(font
+				(size 1.27 1.27)
+			)
+		)
+	)
 	(text "Temp Sens."
 		(exclude_from_sim no)
@@
 		)
 	)
+	(text "ADDR->0X41\n"
+		(exclude_from_sim no)
+		(at 321.818 150.368 0)
+		(effects
+			(font
+				(size 1.27 1.27)
+			)
+		)
+	)
+	(text "ADDR->GND 0x44\nADDR->VDD 0x45"
+		(exclude_from_sim no)
+		(at 389.382 105.918 0)
+		(effects
+			(font
+				(size 1.27 1.27)
+			)
+		)
+	)
+	(text "ADDR->GND 0x40\nADDR->VDD 0x41\nADDR->SDA 0x42\nADDR->SCL 0x43"
+		(exclude_from_sim no)
+		(at 317.5 183.134 0)
+		(effects
+			(font
+				(size 1.27 1.27)
+			)
+		)
+	)
+	(text "ADDR->0xA6"
+		(exclude_from_sim no)
+		(at 174.498 90.678 0)
+		(effects
+			(font
+				(size 1.27 1.27)
+			)
+		)
+	)
 	(text "Magnetic Sens."
 		(exclude_from_sim no)
@@
 		)
 	)
+	(text "ADDR->0x30?"
+		(exclude_from_sim no)
+		(at 276.86 242.824 0)
+		(effects
+			(font
+				(size 1.27 1.27)
+			)
+		)
+	)
 	(text "Temp/Hum Sens."
 		(exclude_from_sim no)
@@
 		)
 	)
+	(text "ADDR->GND 0x23\nADDR->VDD 0x5C"
+		(exclude_from_sim no)
+		(at 232.41 90.424 0)
+		(effects
+			(font
+				(size 1.27 1.27)
+			)
+		)
+	)
+	(text "ADDR->GND 0x74\nADDR->VDD 0x76\nADDR->Float 0x46"
+		(exclude_from_sim no)
+		(at 168.656 140.97 0)
+		(effects
+			(font
+				(size 1.27 1.27)
+			)
+		)
+	)
 	(junction
 		(at 185.42 242.57)
@@
 			)
 		)
-		(property "Datasheet" ""
+		(property "Datasheet" "https://optoelectronics.liteon.com/upload/download/DS86-2013-0014/LTR-507ALS-01_FINAL%20DS.pdf"
 			(at 191.77 116.84 0)
 			(effects
@@
 			)
 		)
-		(property "Datasheet" "https://www.sensirion.com/fileadmin/user_upload/customers/sensirion/Dokumente/2_Humidity_Sensors/Datasheets/Sensirion_Humidity_Sensors_SHT3x_Datasheet_digital.pdf"
+		(property "Datasheet" "https://sensirion.com/media/documents/213E6A3B/63A5A569/Datasheet_SHT3x_DIS.pdf"
 			(at 410.21 55.88 0)
 			(effects
