File: Version3/Mess-CHP10/IOT-MESS-CHP20.kicad_sch (KiCad schematic)
At the start: 21 parts, among them J1 Jumper_2, J2 Jumper_2, J3 Conn_01x09_Pin, J4 Conn_01x09_Pin, J9 Jumper_2, U2 CH57xQ_QFN10x3, U4 USB_C_Receptacle_USB2.0_16P, U5 ME6211C33M5, U6 XC6206PxxxMR, Y1 XO32

Commit message: update.
Connections:
- net +3.3V: now also J3.8 (Pin_8); no longer R4.1
- net P_1: now also R1.1
- net P_5: now also R4.1
Other:
- moved on the sheet: D1, D2, R1, R4
Changed lines of the file:
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@@
 	)
 	(junction
-		(at 242.57 204.47)
-		(diameter 0)
-		(color 0 0 0 0)
-	)
-	(junction
 		(at 201.93 204.47)
 		(diameter 0)
@@
 	)
 	(junction
-		(at 187.96 217.17)
+		(at 252.73 125.73)
 		(diameter 0)
 		(color 0 0 0 0)
 	)
 	(junction
-		(at 201.93 185.42)
+		(at 187.96 217.17)
 		(diameter 0)
 		(color 0 0 0 0)
@@
 	(wire
 		(pts
+			(xy 234.95 140.97) (xy 252.73 140.97)
+		)
+		(stroke
+			(width 0)
+			(type default)
+		)
+	)
+	(wire
+		(pts
 			(xy 279.4 143.51) (xy 273.05 143.51)
 		)
@@
 	(wire
 		(pts
-			(xy 242.57 204.47) (xy 242.57 208.28)
+			(xy 267.97 204.47) (xy 267.97 209.55)
 		)
 		(stroke
@@
 	(wire
 		(pts
-			(xy 242.57 223.52) (xy 242.57 227.33)
-		)
-		(stroke
-			(width 0)
-			(type default)
-		)
-	)
-	(wire
-		(pts
 			(xy 135.89 224.79) (xy 142.24 224.79)
 		)
@@
 	(wire
 		(pts
-			(xy 201.93 180.34) (xy 201.93 185.42)
+			(xy 148.59 180.34) (xy 148.59 185.42)
 		)
 		(stroke
@@
 	(wire
 		(pts
-			(xy 325.12 88.9) (xy 325.12 92.71)
+			(xy 167.64 219.71) (xy 172.72 219.71)
 		)
 		(stroke
@@
 	(wire
 		(pts
-			(xy 167.64 219.71) (xy 172.72 219.71)
+			(xy 121.92 144.78) (xy 121.92 143.51)
 		)
 		(stroke
@@
 	(wire
 		(pts
-			(xy 121.92 144.78) (xy 121.92 143.51)
+			(xy 252.73 140.97) (xy 252.73 125.73)
 		)
 		(stroke
@@
 	(wire
 		(pts
+			(xy 251.46 209.55) (xy 251.46 204.47)
+		)
+		(stroke
+			(width 0)
+			(type default)
+		)
+	)
+	(wire
+		(pts
 			(xy 242.57 196.85) (xy 242.57 204.47)
 		)
@@
 		)
 	)
+	(global_label "P_1"
+		(shape input)
+		(at 251.46 204.47 0)
+		(fields_autoplaced yes)
+		(effects
+			(font
+				(size 1.27 1.27)
+				(thickness 0.254)
+				(bold yes)
+				(color 255 0 0 1)
+			)
+			(justify left)
+		)
+		(property "Intersheetrefs" "${INTERSHEET_REFS}"
+			(at 258.3683 204.47 0)
+			(effects
+				(font
+					(size 1.27 1.27)
+				)
+				(justify left)
+				(hide yes)
+			)
+		)
+	)
+	(global_label "P_5"
+		(shape input)
+		(at 267.97 204.47 0)
+		(fields_autoplaced yes)
+		(effects
+			(font
+				(size 1.27 1.27)
+			)
+			(justify left)
+		)
+		(property "Intersheetrefs" "${INTERSHEET_REFS}"
+			(at 274.4023 204.47 0)
+			(effects
+				(font
+					(size 1.27 1.27)
+				)
+				(justify left)
+				(hide yes)
+			)
+		)
+	)
 	(global_label "P_9"
 		(shape input)
@@
 	(symbol
 		(lib_id "Device:R")
-		(at 325.12 77.47 0)
+		(at 251.46 213.36 0)
 		(unit 1)
 		(exclude_from_sim no)
@@
 		(dnp no)
 		(property "Reference" "R1"
-			(at 325.12 80.01 90)
+			(at 251.46 215.9 90)
 			(effects
 				(font
@@
 		)
 		(property "Value" "R"
-			(at 325.12 76.835 90)
+			(at 251.46 212.725 90)
 			(effects
 				(font
@@
 		)
 		(property "Footprint" "Resistor_SMD:R_0603_1608Metric"
-			(at 323.342 77.47 90)
+			(at 249.682 213.36 90)
 			(effects
 				(font
@@
 		)
 		(property "Datasheet" "~"
-			(at 325.12 77.47 0)
+			(at 251.46 213.36 0)
 			(effects
 				(font
@@
 		)
 		(property "Description" ""
-			(at 325.12 77.47 0)
+			(at 251.46 213.36 0)
 			(effects
 				(font
@@
 	(symbol
 		(lib_id "Device:LED")
-		(at 325.12 85.09 270)
+		(at 251.46 220.98 270)
 		(mirror x)
 		(unit 1)
@@
 		(dnp no)
 		(property "Reference" "D2"
-			(at 328.295 87.3125 0)
+			(at 254.635 223.2025 0)
 			(effects
 				(font
@@
 		)
 		(property "Value" "LED"
-			(at 328.295 83.82 0)
+			(at 254.635 219.71 0)
 			(effects
 				(font
@@
 		)
 		(property "Footprint" "LED_SMD:LED_0603_1608Metric"
-			(at 325.12 85.09 0)
+			(at 251.46 220.98 0)
 			(effects
 				(font
@@
 		)
 		(property "Datasheet" "~"
-			(at 325.12 85.09 0)
+			(at 251.46 220.98 0)
 			(effects
 				(font
@@
 		)
 		(property "Description" "Light emitting diode"
-			(at 325.12 85.09 0)
+			(at 251.46 220.98 0)
 			(effects
 				(font
@@
 		)
 		(property "Sim.Pins" "1=K 2=A"
-			(at 325.12 85.09 0)
+			(at 251.46 220.98 0)
 			(effects
 				(font
@@
 	(symbol
 		(lib_id "power:GND")
-		(at 242.57 227.33 0)
+		(at 267.97 224.79 0)
 		(mirror y)
 		(unit 1)
@@
 		(dnp no)
 		(property "Reference" "#PWR017"
-			(at 242.57 233.68 0)
+			(at 267.97 231.14 0)
 			(effects
 				(font
@@
 		)
 		(property "Value" "GND"
-			(at 242.57 231.775 0)
+			(at 267.97 229.235 0)
 			(effects
 				(font
@@
 		)
 		(property "Footprint" ""
-			(at 242.57 227.33 0)
+			(at 267.97 224.79 0)
 			(effects
 				(font
@@
 		)
 		(property "Datasheet" ""
-			(at 242.57 227.33 0)
+			(at 267.97 224.79 0)
 			(effects
 				(font
@@
 		)
 		(property "Description" "Power symbol creates a global label with name \"GND\" , ground"
-			(at 242.57 227.33 0)
+			(at 267.97 224.79 0)
 			(effects
 				(font
@@
 	(symbol
 		(lib_id "power:GND")
-		(at 325.12 92.71 0)
+		(at 251.46 224.79 0)
 		(mirror y)
 		(unit 1)
@@
 		(dnp no)
 		(property "Reference" "#PWR018"
-			(at 325.12 99.06 0)
+			(at 251.46 231.14 0)
 			(effects
 				(font
@@
 		)
 		(property "Value" "GND"
-			(at 325.12 97.155 0)
+			(at 251.46 229.235 0)
 			(effects
 				(font
@@
 		)
 		(property "Footprint" ""
-			(at 325.12 92.71 0)
+			(at 251.46 224.79 0)
 			(effects
 				(font
@@
 		)
 		(property "Datasheet" ""
-			(at 325.12 92.71 0)
+			(at 251.46 224.79 0)
 			(effects
 				(font
@@
 		)
 		(property "Description" "Power symbol creates a global label with name \"GND\" , ground"
-			(at 325.12 92.71 0)
+			(at 251.46 224.79 0)
 			(effects
 				(font
@@
 	(symbol
 		(lib_id "Device:LED")
-		(at 242.57 219.71 270)
+		(at 267.97 220.98 270)
 		(mirror x)
 		(unit 1)
@@
 		(dnp no)
 		(property "Reference" "D1"
-			(at 245.745 221.9325 0)
+			(at 271.145 223.2025 0)
 			(effects
 				(font
@@
 		)
 		(property "Value" "LED"
-			(at 245.745 218.44 0)
+			(at 271.145 219.71 0)
 			(effects
 				(font
@@
 		)
 		(property "Footprint" "LED_SMD:LED_0603_1608Metric"
-			(at 242.57 219.71 0)
+			(at 267.97 220.98 0)
 			(effects
 				(font
@@
 		)
 		(property "Datasheet" "~"
-			(at 242.57 219.71 0)
+			(at 267.97 220.98 0)
 			(effects
 				(font
@@
 		)
 		(property "Description" "Light emitting diode"
-			(at 242.57 219.71 0)
+			(at 267.97 220.98 0)
 			(effects
 				(font
@@
 		)
 		(property "Sim.Pins" "1=K 2=A"
-			(at 242.57 219.71 0)
+			(at 267.97 220.98 0)
 			(effects
 				(font
@@
 	(symbol
 		(lib_id "power:PWR_FLAG")
-		(at 201.93 180.34 0)
+		(at 148.59 180.34 0)
 		(unit 1)
 		(exclude_from_sim no)
@@
 		(fields_autoplaced yes)
 		(property "Reference" "#FLG03"
-			(at 201.93 178.435 0)
+			(at 148.59 178.435 0)
 			(effects
 				(font
@@
 		)
 		(property "Value" "PWR_FLAG"
-			(at 201.93 175.26 0)
+			(at 148.59 175.26 0)
 			(effects
 				(font
@@
 		)
 		(property "Footprint" ""
-			(at 201.93 180.34 0)
+			(at 148.59 180.34 0)
 			(effects
 				(font
@@
 		)
 		(property "Datasheet" "~"
-			(at 201.93 180.34 0)
+			(at 148.59 180.34 0)
 			(effects
 				(font
@@
 		)
 		(property "Description" "Special symbol for telling ERC where power comes from"
-			(at 201.93 180.34 0)
+			(at 148.59 180.34 0)
 			(effects
 				(font
@@
 	(symbol
 		(lib_id "Device:R")
-		(at 242.57 212.09 0)
+		(at 267.97 213.36 0)
 		(unit 1)
 		(exclude_from_sim no)
@@
 		(dnp no)
 		(property "Reference" "R4"
-			(at 242.57 214.63 90)
+			(at 267.97 215.9 90)
 			(effects
 				(font
@@
 		)
 		(property "Value" "R"
-			(at 242.57 211.455 90)
+			(at 267.97 212.725 90)
 			(effects
 				(font
@@
 		)
 		(property "Footprint" "Resistor_SMD:R_0603_1608Metric"
-			(at 240.792 212.09 90)
+			(at 266.192 213.36 90)
 			(effects
 				(font
@@
 		)
 		(property "Datasheet" "~"
-			(at 242.57 212.09 0)
+			(at 267.97 213.36 0)
 			(effects
 				(font
@@
 		)
 		(property "Description" ""
-			(at 242.57 212.09 0)
+			(at 267.97 213.36 0)
 			(effects
 				(font
