File: Version3/Mess-CHP10/IOT-MESS-CHP20.kicad_sch (KiCad schematic)
At the start: 21 parts, among them J1 Jumper_2, J2 Jumper_2, J3 Conn_01x09_Pin, J4 Conn_01x09_Pin, J9 Jumper_2, U2 CH57xQ_QFN10x3, U4 USB_C_Receptacle_USB2.0_16P, U5 ME6211C33M5, U6 XC6206PxxxMR, Y1 XO32

Commit message: update.
Parts:
- U2: value CH57xQ_QFN10x3 -> CH57xQ_DFN10x3
Changed lines of the file:
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@@
 			)
 		)
-		(property "Value" "CH57xQ_QFN10x3"
+		(property "Value" "CH57xQ_DFN10x3"
 			(at 271.3833 60.96 0)
 			(effects
