File: Version3/CH-NFC/CH-NFC.kicad_pcb (KiCad board)
At the start: 2 copper layers, 100 x 100 mm, 50 parts, among them J1 Conn_01x16_Pin, J10 Conn_01x05_Pin, J12 Conn_01x05_Pin, J13 Conn_01x05_Pin, J14 RJ45_Kycon_G7LX-A88S7-BP-GY, J15 Conn_01x05_Pin, J16 RJ45_Kycon_G7LX-A88S7-BP-GY, J17 Conn_01x05_Pin, J18 RJ45_Kycon_G7LX-A88S7-BP-GY, J19 Conn_01x05_Pin, J2 Conn_01x02_Pin, J20 Conn_01x05_Pin, J21 Conn_01x05_Pin, J22 Conn_01x05_Pin, J23 RJ45_Kycon_G7LX-A88S7-BP-GY, J24 RJ45_Kycon_G7LX-A88S7-BP-GY, J25 RJ45_Kycon_G7LX-A88S7-BP-GY, J26 RJ45_Kycon_G7LX-A88S7-BP-GY, J27 Conn_01x05_Pin, J28 Conn_01x05_Pin, J29 RJ45_Kycon_G7LX-A88S7-BP-GY, J3 RJ45_Kycon_G7LX-A88S7-BP-GY, J30 RJ45_Kycon_G7LX-A88S7-BP-GY, J31 Conn_01x39_Pin, J32 Conn_01x39_Pin, J33 Conn_01x08_Pin, J34 Conn_01x39_Pin, J35 Conn_01x08_Pin, J36 Conn_01x08_Pin, J37 Conn_01x08_Pin, J38 Conn_01x08_Pin, J4 Conn_01x16_Pin, J5 Conn_01x16_Pin, J7 Conn_01x16_Pin, U1 NFC_ANTENNA, U4 USB_C_Receptacle_USB2.0_16P, U5 ME6211C33M5, U6 XC6206PxxxMR, Y1 XO32

Commit message: update.
Parts:
- removed J7: Conn_01x16_Pin, Connector_PinHeader_2.54mm:PinHeader_1x16_P2.54mm_Vertical
- added J8: Conn_01x29_Pin, Connector_PinHeader_2.54mm:PinHeader_1x29_P2.54mm_Vertical, F.Cu at (113.8, 75.5)
- J1: value Conn_01x16_Pin -> Conn_01x29_Pin; footprint Connector_PinHeader_2.54mm:PinHeader_1x16_P2.54mm_Vertical -> Connector_PinHeader_2.54mm:PinHeader_1x29_P2.54mm_Vertical
- moved J1 41.2 mm to (139.0, 75.4)
- moved AE2 7.50 mm to (142.1, 107.0)
Connections:
- J1 pad 1: P_1 -> unconnected-(J1-Pin_1-Pad1)
- J1 pad 10: P_12 -> unconnected-(J1-Pin_10-Pad10)
- J1 pad 11: P_13 -> unconnected-(J1-Pin_11-Pad11)
- J1 pad 12: P_14 -> unconnected-(J1-Pin_12-Pad12)
- J1 pad 13: P_15 -> unconnected-(J1-Pin_13-Pad13)
- J1 pad 14: +3.3V -> P_32
- J1 pad 15: GND -> P_31
- J1 pad 16: 5V -> P_30
- J1 pad 2: P_2 -> unconnected-(J1-Pin_2-Pad2)
- J1 pad 3: P_3 -> unconnected-(J1-Pin_3-Pad3)
- J1 pad 4: P_4 -> unconnected-(J1-Pin_4-Pad4)
- J1 pad 5: P_5 -> unconnected-(J1-Pin_5-Pad5)
- J1 pad 6: P_6 -> unconnected-(J1-Pin_6-Pad6)
- J1 pad 7: P_7 -> unconnected-(J1-Pin_7-Pad7)
- J1 pad 8: P_8 -> unconnected-(J1-Pin_8-Pad8)
- J1 pad 9: P_11 -> unconnected-(J1-Pin_9-Pad9)
Routing:
- net +3.3V: track 163.9 -> 414.2 mm, vias 0 -> 1
- net E_TX-4: track 0.00 -> 8.59 mm
- net E_TX+8: track 0.00 -> 5.77 mm
- net LDO_EN: track 0.00 -> 5.71 mm
- net E_TX+5: track 0.00 -> 5.67 mm
- net 5V: track 38.3 -> 42.9 mm
- net Net-(J9-A): track 0.00 -> 3.24 mm, vias 0 -> 1
- net GND: track 11.7 -> 9.24 mm
- net P_24: track 36.7 -> 37.8 mm
- net Net-(J2-Pin_1): track 9.21 -> 9.99 mm, vias 0 -> 1
