File: Version3/CH-NFC/CH-NFC.kicad_sch (KiCad schematic)
At the start: 52 parts, among them J1 Conn_01x16_Pin, J10 Conn_01x05_Pin, J12 Conn_01x05_Pin, J13 Conn_01x05_Pin, J14 RJ45_Kycon_G7LX-A88S7-BP-GY, J15 Conn_01x05_Pin, J16 RJ45_Kycon_G7LX-A88S7-BP-GY, J17 Conn_01x05_Pin, J18 RJ45_Kycon_G7LX-A88S7-BP-GY, J19 Conn_01x05_Pin, J2 Conn_01x02_Pin, J20 Conn_01x05_Pin, J21 Conn_01x05_Pin, J22 Conn_01x05_Pin, J23 RJ45_Kycon_G7LX-A88S7-BP-GY, J24 RJ45_Kycon_G7LX-A88S7-BP-GY, J25 RJ45_Kycon_G7LX-A88S7-BP-GY, J26 RJ45_Kycon_G7LX-A88S7-BP-GY, J27 Conn_01x05_Pin, J28 Conn_01x05_Pin, J29 RJ45_Kycon_G7LX-A88S7-BP-GY, J3 RJ45_Kycon_G7LX-A88S7-BP-GY, J30 RJ45_Kycon_G7LX-A88S7-BP-GY, J31 Conn_01x39_Pin, J32 Conn_01x39_Pin, J33 Conn_01x08_Pin, J34 Conn_01x39_Pin, J35 Conn_01x08_Pin, J36 Conn_01x08_Pin, J37 Conn_01x08_Pin, J38 Conn_01x08_Pin, J4 Conn_01x16_Pin, J5 Conn_01x16_Pin, J6 Jumper, J7 Conn_01x16_Pin, J9 Jumper_2, U1 NFC_ANTENNA, U4 USB_C_Receptacle_USB2.0_16P, U5 ME6211C33M5, U6 XC6206PxxxMR, Y1 XO32

Commit message: update.
Parts:
- removed J1, J7: Conn_01x16_Pin, Connector_PinHeader_2.54mm:PinHeader_1x16_P2.54mm_Vertical, symbol Connector:Conn_01x16_Pin
- added J1, J8: Conn_01x29_Pin, Connector_PinHeader_2.54mm:PinHeader_1x29_P2.54mm_Vertical, symbol Connector:Conn_01x29_Pin
Connections:
- net +3.3V: now also J8.27 (Pin_27)
- net 5V: now also J8.29 (Pin_29)
- net GND: now also J8.28 (Pin_28)
- net P_1: now also J8.14 (Pin_14)
- net P_11: now also J8.22 (Pin_22)
- net P_12: now also J8.23 (Pin_23)
- net P_13: now also J8.24 (Pin_24)
- net P_14: now also J8.25 (Pin_25)
- net P_15: now also J8.26 (Pin_26)
- net P_16: now also J1.29 (Pin_29)
- net P_17: now also J1.28 (Pin_28)
- net P_18: now also J1.27 (Pin_27)
- net P_19: now also J1.26 (Pin_26)
- net P_2: now also J8.15 (Pin_15)
- net P_20: now also J1.25 (Pin_25)
- net P_21: now also J1.24 (Pin_24)
- net P_22: now also J1.23 (Pin_23)
- net P_23: now also J1.22 (Pin_22)
- net P_24: now also J1.21 (Pin_21)
- net P_25: now also J1.20 (Pin_20)
- net P_27: now also J1.19 (Pin_19)
- net P_28: now also J1.18 (Pin_18)
- net P_29: now also J1.17 (Pin_17)
- net P_3: now also J8.16 (Pin_16)
- net P_30: now also J1.16 (Pin_16)
- net P_31: now also J1.15 (Pin_15)
- net P_32: now also J1.14 (Pin_14)
- net P_4: now also J8.17 (Pin_17)
- net P_5: now also J8.18 (Pin_18)
- net P_6: now also J8.19 (Pin_19)
- net P_7: now also J8.20 (Pin_20)
- net P_8: now also J8.21 (Pin_21)
- no-connect marks 92 -> 275
Other:
- moved on the sheet: J34
